File: opm-high/source/Cheap FOCer 2 60mm.sch (KiCad schematic (older format))
At the start: 49 parts, among them J1 Conn_01x02, J2 Conn_01x07, J3 Conn_01x03, J6 Conn_01x03, P1 MOTOR1, P2 MOTOR1, P3 MOTOR1, P4 HALL/Encoder

Commit message: cleanup
Parts:
- removed C1: 100n, Capacitor_SMD:C_0603_1608Metric, symbol BLDC_4-rescue:C-RESCUE-BLDC_4
- removed C2, C3: 0.01uF, Capacitor_SMD:C_0603_1608Metric, symbol BLDC_4-rescue:C-RESCUE-BLDC_4
- removed D1, D2: SMF05CT1G, Package_TO_SOT_SMD:SOT-363_SC-70-6, symbol Power_Protection:SP0505BAHT
- removed D3: RED, LED_SMD:LED_0603_1608Metric, symbol Device:LED
- removed J1: Conn_01x02, Connector_JST:JST_PH_B2B-PH-K_1x02_P2.00mm_Vertical, symbol Connector_Generic:Conn_01x02
- removed J2: Conn_01x07, Connector_JST:JST_PH_B7B-PH-K_1x07_P2.00mm_Vertical, symbol Connector_Generic:Conn_01x07
- removed P4: HALL/Encoder, Connector_JST:JST_PH_B6B-PH-K_1x06_P2.00mm_Vertical, symbol Connector_Generic:Conn_01x06
- removed R1: 39k, Resistor_SMD:R_0603_1608Metric, symbol BLDC_4-rescue:R-RESCUE-BLDC_4
- removed R10, R5, R7, R8, R9: 100R, Resistor_SMD:R_0603_1608Metric, symbol BLDC_4-rescue:R-RESCUE-BLDC_4
- removed R2: 2k2, Resistor_SMD:R_0603_1608Metric, symbol BLDC_4-rescue:R-RESCUE-BLDC_4
- removed R3, R4: 22R, Resistor_SMD:R_0603_1608Metric, symbol BLDC_4-rescue:R-RESCUE-BLDC_4
- removed R40, R68, R71, R72: DNP, Resistor_SMD:R_0603_1608Metric, symbol BLDC_4-rescue:R-RESCUE-BLDC_4
- removed USB1: USB Micro U-D-M5DD-W-1, Connector_USB:USB_Micro-B_Wuerth_614105150721_Vertical, symbol Connector:USB_B_Micro
Connections:
- net MCU/LED_GREEN: no longer names the net of R11.2
- net MCU/SERVO: no longer names the net of C4.2, R6.1
- no-connect marks 2 -> 0
Other:
- note removed: "Cheap F Cer 2"
- note removed: "Pull up and Pull down \nresistors on ADC channels. \nDNP by default.\nUse 10k resistors if needed"
- moved on the sheet: C4, D4, D5, F1, F2, F3, H1, H13, H2, H5, H6, H7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
