File: opm-high/source/Cheap FOCer 2 60mm.sch (KiCad schematic (older format))
At the start: 26 parts, among them J3 Conn_01x03, J6 Conn_01x03, P1 MOTOR1, P2 MOTOR1, P3 MOTOR1

Commit message: cleanup
Parts:
- removed C4: .01uF, Capacitor_SMD:C_0603_1608Metric, symbol BLDC_4-rescue:C-RESCUE-BLDC_4
- removed D4: GRN, LED_SMD:LED_0603_1608Metric, symbol Device:LED
- removed D5: BLU, LED_SMD:LED_0603_1608Metric, symbol Device:LED
- removed J3: Conn_01x03, Connector_JST:JST_PH_B3B-PH-K_1x03_P2.00mm_Vertical, symbol Connector_Generic:Conn_01x03
- removed J6: Conn_01x03, Connector_PinHeader_2.54mm:PinHeader_1x02_P2.54mm_Vertical, symbol Connector_Generic:Conn_01x02
- removed R11, R6: 100R, Resistor_SMD:R_0603_1608Metric, symbol BLDC_4-rescue:R-RESCUE-BLDC_4
- removed R12: 2k2, Resistor_SMD:R_0603_1608Metric, symbol BLDC_4-rescue:R-RESCUE-BLDC_4
Other:
- note removed: "Pads for \nauxillary 5V out"
Changed lines of the file:
@@
 Comment4 "Top level"
 $EndDescr
-$Comp
-L BLDC_4-rescue:C-RESCUE-BLDC_4 C4
-U 1 1 522DA0A7
-P 5950 6950
-F 0 "C4" V 6000 6800 50  0000 L CNN
-F 1 ".01uF" V 6100 6850 50  0000 L CNN
-F 2 "Capacitor_SMD:C_0603_1608Metric" H 5950 6950 60  0001 C CNN
-F 3 "" H 5950 6950 60  0001 C CNN
-	1    5950 6950
-	0    1    1    0
-$EndComp
-$Comp
-L BLDC_4-rescue:R-RESCUE-BLDC_4 R6
-U 1 1 522DA0AD
-P 6000 6750
-F 0 "R6" V 6100 6750 50  0000 C CNN
-F 1 "100R" V 6000 6750 50  0000 C CNN
-F 2 "Resistor_SMD:R_0603_1608Metric" H 6000 6750 60  0001 C CNN
-F 3 "" H 6000 6750 60  0001 C CNN
-	1    6000 6750
-	0    -1   -1   0
-$EndComp
-$Comp
-L BLDC_4-rescue:+5V #PWR015
-U 1 1 522DA158
-P 6500 6850
-F 0 "#PWR015" H 6500 6940 20  0001 C CNN
-F 1 "+5V" H 6500 7000 30  0000 C CNN
-F 2 "" H 6500 6850 60  0001 C CNN
-F 3 "" H 6500 6850 60  0001 C CNN
-	1    6500 6850
-	0    -1   1    0
-$EndComp
 Text Notes 8150 3050 0    40   ~ 0
 Voltage supply (0 - 51v)
-$Comp
-L BLDC_4-rescue:R-RESCUE-BLDC_4 R11
-U 1 1 53FC130C
-P 5600 7600
-F 0 "R11" V 5500 7600 50  0000 C CNN
-F 1 "100R" V 5600 7600 50  0000 C CNN
-F 2 "Resistor_SMD:R_0603_1608Metric" H 5600 7600 60  0001 C CNN
-F 3 "" H 5600 7600 60  0001 C CNN
-	1    5600 7600
-	-1   0    0    1
-$EndComp
-$Comp
-L Device:LED D4
-U 1 1 53FC1313
-P 5600 8300
-F 0 "D4" V 5700 8350 50  0000 C CNN
-F 1 "GRN" V 5500 8400 50  0000 C CNN
-F 2 "LED_SMD:LED_0603_1608Metric" H 5600 8300 60  0001 C CNN
-F 3 "" H 5600 8300 60  0001 C CNN
-	1    5600 8300
-	0    -1   -1   0
-$EndComp
-$Comp
-L BLDC_4-rescue:GND-RESCUE-BLDC_4 #PWR019
-U 1 1 53FC131A
-P 5600 8500
-F 0 "#PWR019" H 5600 8500 30  0001 C CNN
-F 1 "GND-RESCUE-BLDC_4" H 5600 8430 30  0001 C CNN
-F 2 "LED_SMD:LED_0603_1608Metric" H 5600 8500 60  0001 C CNN
-F 3 "" H 5600 8500 60  0001 C CNN
-	1    5600 8500
-	1    0    0    -1
-$EndComp
-$Comp
-L BLDC_4-rescue:R-RESCUE-BLDC_4 R12
-U 1 1 53FC6A67
-P 5900 7600
-F 0 "R12" V 5800 7600 50  0000 C CNN
-F 1 "2k2" V 5900 7600 50  0000 C CNN
-F 2 "Resistor_SMD:R_0603_1608Metric" H 5900 7600 60  0001 C CNN
-F 3 "" H 5900 7600 60  0001 C CNN
-	1    5900 7600
-	-1   0    0    1
-$EndComp
-$Comp
-L BLDC_4-rescue:GND-RESCUE-BLDC_4 #PWR020
-U 1 1 53FC8AA4
-P 5900 8500
-F 0 "#PWR020" H 5900 8500 30  0001 C CNN
-F 1 "GND" H 5900 8430 30  0001 C CNN
-F 2 "" H 5900 8500 60  0001 C CNN
-F 3 "" H 5900 8500 60  0001 C CNN
-	1    5900 8500
-	1    0    0    -1
-$EndComp
-$Comp
-L BLDC_4-rescue:VCC #PWR017
-U 1 1 53FC98D2
-P 5900 7350
-F 0 "#PWR017" H 5900 7450 30  0001 C CNN
-F 1 "VCC" V 5900 7500 30  0000 C CNN
-F 2 "" H 5900 7350 60  0001 C CNN
-F 3 "" H 5900 7350 60  0001 C CNN
-	1    5900 7350
-	0    -1   -1   0
-$EndComp
-Wire Wire Line
-	6400 6950 6400 7050
-Wire Wire Line
-	6150 6950 6400 6950
-Connection ~ 6400 6950
-Wire Wire Line
-	5700 6950 5750 6950
-Wire Wire Line
-	5700 6750 5700 6950
 Wire Wire Line
 	7100 3850 8050 3850
@@
 	1    0    0    -1
 $EndComp
-Wire Wire Line
-	6400 6950 6550 6950
-Wire Wire Line
-	5700 6750 5750 6750
 Wire Wire Line
 	7100 5000 8050 5000
@@
 Text Notes 8550 6100 0    60   ~ 0
 Connect signal ground and\npower ground in one place only
-Wire Wire Line
-	5600 7850 5600 8150
 $Comp
 L BLDC_4-rescue:CONN_1 P3
@@
 	0    1    1    0
 $EndComp
-$Comp
-L Connector_Generic:Conn_01x03 J3
-U 1 1 5DA818C8
-P 6750 6850
-F 0 "J3" H 6668 6525 50  0000 C CNN
-F 1 "Conn_01x03" H 6668 6616 50  0000 C CNN
-F 2 "Connector_JST:JST_PH_B3B-PH-K_1x03_P2.00mm_Vertical" H 6750 6850 50  0001 C CNN
-F 3 "~" H 6750 6850 50  0001 C CNN
-	1    6750 6850
-	1    0    0    1
-$EndComp
-Wire Wire Line
-	6500 6850 6550 6850
 Connection ~ 8500 2800
-$Comp
-L BLDC_4-rescue:GND-RESCUE-BLDC_4 #PWR016
-U 1 1 522DA0BA
-P 6400 7050
-F 0 "#PWR016" H 6400 7050 30  0001 C CNN
-F 1 "GND" H 6400 6980 30  0001 C CNN
-F 2 "" H 6400 7050 60  0001 C CNN
-F 3 "" H 6400 7050 60  0001 C CNN
-	1    6400 7050
-	1    0    0    -1
-$EndComp
-Wire Wire Line
-	5600 7000 5600 7350
-Wire Wire Line
-	6250 6750 6550 6750
-$Comp
-L Connector_Generic:Conn_01x02 J6
-U 1 1 5DD4EBB7
-P 8000 7250
-F 0 "J6" H 7918 6925 50  0000 C CNN
-F 1 "Conn_01x03" H 7918 7016 50  0000 C CNN
-F 2 "Connector_PinHeader_2.54mm:PinHeader_1x02_P2.54mm_Vertical" H 8000 7250 50  0001 C CNN
-F 3 "~" H 8000 7250 50  0001 C CNN
-	1    8000 7250
-	1    0    0    1
-$EndComp
-$Comp
-L BLDC_4-rescue:+5V #PWR087
-U 1 1 5DD56875
-P 7750 7150
-F 0 "#PWR087" H 7750 7240 20  0001 C CNN
-F 1 "+5V" H 7750 7300 30  0000 C CNN
-F 2 "" H 7750 7150 60  0001 C CNN
-F 3 "" H 7750 7150 60  0001 C CNN
-	1    7750 7150
-	0    -1   1    0
-$EndComp
-Wire Wire Line
-	7750 7150 7800 7150
-Wire Wire Line
-	7800 7250 7700 7250
-$Comp
-L BLDC_4-rescue:GND-RESCUE-BLDC_4 #PWR086
-U 1 1 5DD5E8F2
-P 7700 7250
-F 0 "#PWR086" H 7700 7250 30  0001 C CNN
-F 1 "GND" H 7700 7180 30  0001 C CNN
-F 2 "" H 7700 7250 60  0001 C CNN
-F 3 "" H 7700 7250 60  0001 C CNN
-	1    7700 7250
-	0    1    1    0
-$EndComp
-Wire Wire Line
-	5900 7850 5900 8150
-$Comp
-L Device:LED D5
-U 1 1 53FC6A60
-P 5900 8300
-F 0 "D5" V 6000 8350 50  0000 C CNN
-F 1 "BLU" V 5800 8400 50  0000 C CNN
-F 2 "LED_SMD:LED_0603_1608Metric" H 5900 8300 60  0001 C CNN
-F 3 "" H 5900 8300 60  0001 C CNN
-	1    5900 8300
-	0    -1   -1   0
-$EndComp
-Wire Wire Line
-	5900 8450 5900 8500
-Wire Wire Line
-	5600 8500 5600 8450
 $Comp
 L Mechanical:MountingHole H13
@@
 Text Notes 5900 2350 0    60   ~ 0
 Fiducials
-Wire Notes Line
-	8200 6600 8200 7400
-Wire Notes Line
-	8200 7400 7500 7400
-Wire Notes Line
-	7500 7400 7500 6600
-Wire Notes Line
-	7500 6600 8200 6600
-Text Notes 7650 6800 0    39   ~ 0
-Pads for \nauxillary 5V out
 $EndSCHEMATC
