File: opm-high/source/Cheap FOCer 2 60mm.kicad_pcb (KiCad board)
At the start: 2 copper layers, 59.1 x 99.9 mm, 193 parts, among them J1 Conn_01x02, J2 Conn_01x07, J3 Conn_01x03, J4 On/Off, J5 UNUSED MCU PINS, J6 Conn_01x03, P1 MOTOR1, P2 MOTOR1, P3 MOTOR1, P4 HALL/Encoder, P5 SWD, Q1 NCEP60T20, Q2 NCEP60T20, Q3 NCEP60T20, Q4 NCEP60T20, Q5 NCEP60T20, Q6 NCEP60T20, U1 AMS1117-3.3, U2 DRV8301, U3 TP2604-SR, U4 TJA1051T/3/1J, U5 STM32F405RGT6, U6 BMI160, X1 8MHz 10ppm (X50328MSB2GI)

Commit message: cleanup
Parts:
- C13: value 120p -> 150p
Connections:
- C16 pad 2: /MCU/BR_SO1 -> /Mosfet driver/BR_SO1
- C4 pad 2: /MCU/SERVO -> Net-(C4-Pad2)
- C57 pad 2: /MCU/BR_SO2 -> /Mosfet driver/BR_SO2
- C58 pad 2: /MCU/BR_SO3 -> /Mosfet driver/BR_SO3
- R11 pad 2: /MCU/LED_GREEN -> Net-(R11-Pad2)
- R22 pad 2: /MCU/FAULT -> /Mosfet driver/FAULT
- R24 pad 1: /MCU/SDO -> /Mosfet driver/SDO
- R25 pad 1: /MCU/EN_GATE -> /Mosfet driver/EN_GATE
- R26 pad 1: /MCU/BR_SO1 -> /Mosfet driver/BR_SO1
- R27 pad 2: /MCU/SENS1 -> /Mosfet driver/SENS1
- R28 pad 1: /MCU/BR_SO2 -> /Mosfet driver/BR_SO2
- R29 pad 2: /MCU/SENS1 -> /Mosfet driver/SENS1
- R30 pad 1: /MCU/BR_SO3 -> /Mosfet driver/BR_SO3
- R31 pad 2: /MCU/SENS2 -> /Mosfet driver/SENS2
- R32 pad 2: /MCU/SENS2 -> /Mosfet driver/SENS2
- R36 pad 2: /MCU/SENS3 -> /Mosfet driver/SENS3
- R38 pad 2: /MCU/SENS3 -> /Mosfet driver/SENS3
- R6 pad 1: /MCU/SERVO -> Net-(C4-Pad2)
- U2 pad 10: /MCU/SDO -> /Mosfet driver/SDO
- U2 pad 11: /MCU/SLCK -> /Mosfet driver/SLCK
- U2 pad 16: /MCU/EN_GATE -> /Mosfet driver/EN_GATE
- U2 pad 17: /MCU/H1 -> /Mosfet driver/H1
- U2 pad 18: /MCU/L1 -> /Mosfet driver/L1
- U2 pad 19: /MCU/H2 -> /Mosfet driver/H2
- U2 pad 20: /MCU/L2 -> /Mosfet driver/L2
- U2 pad 21: /MCU/H3 -> /Mosfet driver/H3
- U2 pad 22: /MCU/L3 -> /Mosfet driver/L3
- U2 pad 6: /MCU/FAULT -> /Mosfet driver/FAULT
- U2 pad 8: /MCU/CS -> /Mosfet driver/CS
- U2 pad 9: /MCU/SDI -> /Mosfet driver/SDI
