File: opm-high-inline/source/Connevtors.sch (KiCad schematic (older format))
At the start: 29 parts, among them J201 W+P_46-3492-44-3-00-10-PPTR, U201 Metz_31330102, U202 Metz_31349102, U203 Metz_31330103, U204 Metz_31349103

Commit message: rename files
Parts:
- removed J201: W+P_46-3492-44-3-00-10-PPTR, Connector_Samtec_HLE_SMD:Samtec_HLE-144-02-xxx-DV-BE-A_2x22_P2.54mm_Horizontal, symbol TMC6100-EVAL-v1.1-rescue:W+P_46-3492-44-3-00-10-PPTR_TMC-mod-SAMTEC-HLE-122-02-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
- removed R203: 10kΩ/1%, Resistor_SMD:R_0603_1608Metric, symbol Device:R
- removed TP201, TP202, TP203, TP204, TP205, TP206, TP207, TP208, TP209, TP210: TestPoint, TestPoint:TestPoint_Pad_D1.5mm, symbol Connector:TestPoint
- H201, H202, H203, H204: symbol TMC6100-EVAL-v1.2-rescue:MountingHole_Pad-Mechanical -> TMC6100-EVAL-v1.2-rescue:MountingHole_Pad-Mechanical-TMC6100-EVAL-v1.2-rescue
- U201: symbol TMC6100-EVAL-v1.2-rescue:Metz_31330102-Conector_library -> TMC6100-EVAL-v1.2-rescue:Metz_31330102-Conector_library-TMC6100-EVAL-v1.2-rescue
- U202: symbol TMC6100-EVAL-v1.2-rescue:Metz_31349102-Conector_library -> TMC6100-EVAL-v1.2-rescue:Metz_31349102-Conector_library-TMC6100-EVAL-v1.2-rescue
- U203: symbol TMC6100-EVAL-v1.2-rescue:Metz_31330103-Conector_library -> TMC6100-EVAL-v1.2-rescue:Metz_31330103-Conector_library-TMC6100-EVAL-v1.2-rescue
- U204: symbol TMC6100-EVAL-v1.2-rescue:Metz_31349103-Conector_library -> TMC6100-EVAL-v1.2-rescue:Metz_31349103-Conector_library-TMC6100-EVAL-v1.2-rescue
Connections:
- no-connect marks 27 -> 5
Other:
- note removed: "Testpads"
- moved on the sheet: C201, C202, C203, C204, C205, D402, H201, H202, H203, H204, U201, U202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
