File: opm-high-inline/source/Motor Driver.sch (KiCad schematic (older format))
At the start: 38 parts, among them IC301 TMC6100-LA, Q301 BSC026N08NS5, Q302 BSC026N08NS5, Q303 BSC026N08NS5, Q304 BSC026N08NS5, Q305 BSC026N08NS5, Q306 BSC026N08NS5, U301 AD8418, U303 AD8418

Commit message: update for current sense
Parts:
- removed C301, C316: 100nF/16V, Capacitor_SMD:C_0603_1608Metric, symbol Device:C
- removed C302, C317: 2,2nF/16V, Capacitor_SMD:C_0603_1608Metric, symbol Device:C
- removed R303, R317: 1kΩ/1%, Resistor_SMD:R_0603_1608Metric, symbol Device:R
- removed R305, R319: 3mΩ/1%/3W, Resistor_SMD:R_2512_6332Metric, symbol Device:R
- removed U301, U303: AD8418, Package_SO:MSOP-8_3x3mm_P0.65mm, symbol TMC6100-EVAL-v1.1-rescue:AD8418-Amplifier_Current-TMC6100-EVAL-v1.1-rescue
- added 1000pF (x3), 3300pF (x3): C, symbol Device:C
- added C? (x3): 0.1uF, symbol Device:C
- added R? (x6): .001Ω/1%, symbol Device:R
- added R? (x6): 10Ω/1%, symbol Device:R
- added R? (x3): 100, symbol Device:R
- added U? (x3): INA180A3IDBVR, SOT95P280X145-5N, symbol amplifier:INA180A3IDBVR
- IC301: symbol TMC6100-EVAL-v1.2-rescue:TMC6100-TA-Trinamic-TMC6100-EVAL-v1.2-rescue -> opm-high-inline-rescue:TMC6100-TA-Trinamic-TMC6100-EVAL-v1.2-rescue-TMC6100-EVAL-v1.2-rescue
- Q301, Q302, Q303, Q304, Q305, Q306: value BSC026N08NS5 -> YJG95G06A
Connections:
- net labels added: +5V, U-IA-IDC, V-IA-IDC, W-IA-IDC
- net labels removed: +5V_VM, ADC_I_u, ADC_I_w, U, V, W
- wire segments 183 -> 193
Other:
- moved on the sheet: C303, C304, C305, C306, C307, C310, C311, C312, C313, C314, C315, C318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

Commit message: annotate
Parts:
- R13, R14, R15: renamed from R?; value 100 -> 100Ω/5%
- gave numbers to parts that had none: 18
- renumbered 1000pF to 1000pF1, 1000pF to 1000pF2, 1000pF to 1000pF3, 3300pF to 3300pF1, 3300pF to 3300pF2, 3300pF to 3300pF3
Connections:
- net +5V: now also U3.2 (GND)
