File: tmc6100-eval/Connevtors.sch (KiCad schematic (older format))
At the start: 29 parts, among them J201 W+P_46-3492-44-3-00-10-PPTR, U201 Metz_31330102, U202 Metz_31349102, U203 Metz_31330103, U204 Metz_31349103

Commit message: add libs
Parts:
- U201: symbol Conector_library:Metz_31330102 -> TMC6100-EVAL-v1.2-rescue:Metz_31330102-Conector_library
- U202: symbol Conector_library:Metz_31349102 -> TMC6100-EVAL-v1.2-rescue:Metz_31349102-Conector_library
- U203: symbol Conector_library:Metz_31330103 -> TMC6100-EVAL-v1.2-rescue:Metz_31330103-Conector_library
- U204: symbol Conector_library:Metz_31349103 -> TMC6100-EVAL-v1.2-rescue:Metz_31349103-Conector_library
Changed lines of the file:
@@
 $EndDescr
 $Comp
-L Conector_library:Metz_31330102 U201
+L TMC6100-EVAL-v1.2-rescue:Metz_31330102-Conector_library U201
 U 1 1 5C0100EA
 P 1200 750
@@
 	1500 5300 500  5300
 $Comp
-L Conector_library:Metz_31349102 U202
+L TMC6100-EVAL-v1.2-rescue:Metz_31349102-Conector_library U202
 U 1 1 5C59EB06
 P 650 750
@@
 Connection ~ 2550 1200
 $Comp
-L Conector_library:Metz_31330103 U203
+L TMC6100-EVAL-v1.2-rescue:Metz_31330103-Conector_library U203
 U 1 1 5D65AFA7
 P 2100 1850
@@
 ~CS_EEPROM
 $Comp
-L Conector_library:Metz_31349103 U204
+L TMC6100-EVAL-v1.2-rescue:Metz_31349103-Conector_library U204
 U 1 1 5DA86CEE
 P 2650 1850

Commit message: update libs
Parts:
- H201, H202, H203, H204: symbol TMC6100-EVAL-v1.2-rescue:MountingHole_Pad-Mechanical -> TMC6100-EVAL-v1.2-rescue:MountingHole_Pad-Mechanical-TMC6100-EVAL-v1.2-rescue
- U201: symbol TMC6100-EVAL-v1.2-rescue:Metz_31330102-Conector_library -> TMC6100-EVAL-v1.2-rescue:Metz_31330102-Conector_library-TMC6100-EVAL-v1.2-rescue
- U202: symbol TMC6100-EVAL-v1.2-rescue:Metz_31349102-Conector_library -> TMC6100-EVAL-v1.2-rescue:Metz_31349102-Conector_library-TMC6100-EVAL-v1.2-rescue
- U203: symbol TMC6100-EVAL-v1.2-rescue:Metz_31330103-Conector_library -> TMC6100-EVAL-v1.2-rescue:Metz_31330103-Conector_library-TMC6100-EVAL-v1.2-rescue
- U204: symbol TMC6100-EVAL-v1.2-rescue:Metz_31349103-Conector_library -> TMC6100-EVAL-v1.2-rescue:Metz_31349103-Conector_library-TMC6100-EVAL-v1.2-rescue
Changed lines of the file:
@@
 $EndDescr
 $Comp
-L TMC6100-EVAL-v1.2-rescue:Metz_31330102-Conector_library U201
+L TMC6100-EVAL-v1.2-rescue:Metz_31330102-Conector_library-TMC6100-EVAL-v1.2-rescue U201
 U 1 1 5C0100EA
 P 1200 750
@@
 $EndComp
 $Comp
-L TMC6100-EVAL-v1.2-rescue:MountingHole_Pad-Mechanical H201
+L TMC6100-EVAL-v1.2-rescue:MountingHole_Pad-Mechanical-TMC6100-EVAL-v1.2-rescue H201
 U 1 1 5C33535A
 P 900 5650
@@
 $EndComp
 $Comp
-L TMC6100-EVAL-v1.2-rescue:MountingHole_Pad-Mechanical H202
+L TMC6100-EVAL-v1.2-rescue:MountingHole_Pad-Mechanical-TMC6100-EVAL-v1.2-rescue H202
 U 1 1 5C335D22
 P 900 5850
@@
 $EndComp
 $Comp
-L TMC6100-EVAL-v1.2-rescue:MountingHole_Pad-Mechanical H203
+L TMC6100-EVAL-v1.2-rescue:MountingHole_Pad-Mechanical-TMC6100-EVAL-v1.2-rescue H203
 U 1 1 5C335E56
 P 900 6050
@@
 $EndComp
 $Comp
-L TMC6100-EVAL-v1.2-rescue:MountingHole_Pad-Mechanical H204
+L TMC6100-EVAL-v1.2-rescue:MountingHole_Pad-Mechanical-TMC6100-EVAL-v1.2-rescue H204
 U 1 1 5C3360CB
 P 900 6250
@@
 	1500 5300 500  5300
 $Comp
-L TMC6100-EVAL-v1.2-rescue:Metz_31349102-Conector_library U202
+L TMC6100-EVAL-v1.2-rescue:Metz_31349102-Conector_library-TMC6100-EVAL-v1.2-rescue U202
 U 1 1 5C59EB06
 P 650 750
@@
 Connection ~ 2550 1200
 $Comp
-L TMC6100-EVAL-v1.2-rescue:Metz_31330103-Conector_library U203
+L TMC6100-EVAL-v1.2-rescue:Metz_31330103-Conector_library-TMC6100-EVAL-v1.2-rescue U203
 U 1 1 5D65AFA7
 P 2100 1850
@@
 ~CS_EEPROM
 $Comp
-L TMC6100-EVAL-v1.2-rescue:Metz_31349103-Conector_library U204
+L TMC6100-EVAL-v1.2-rescue:Metz_31349103-Conector_library-TMC6100-EVAL-v1.2-rescue U204
 U 1 1 5DA86CEE
 P 2650 1850
