File: tmc6100-eval/Motor Driver.sch (KiCad schematic (older format))
At the start: 38 parts, among them IC301 TMC6100-LA, Q301 BSC026N08NS5, Q302 BSC026N08NS5, Q303 BSC026N08NS5, Q304 BSC026N08NS5, Q305 BSC026N08NS5, Q306 BSC026N08NS5, U301 AD8418, U303 AD8418

Commit message: add libs
Parts:
- IC301: symbol Trinamic:TMC6100-TA -> TMC6100-EVAL-v1.2-rescue:TMC6100-TA-Trinamic
Changed lines of the file:
@@
 	5800 1800 6700 1800
 $Comp
-L Trinamic:TMC6100-TA IC301
+L TMC6100-EVAL-v1.2-rescue:TMC6100-TA-Trinamic IC301
 U 1 1 5D604226
 P 3750 4200

Commit message: update libs
Parts:
- IC301: symbol TMC6100-EVAL-v1.2-rescue:TMC6100-TA-Trinamic -> TMC6100-EVAL-v1.2-rescue:TMC6100-TA-Trinamic-TMC6100-EVAL-v1.2-rescue
Changed lines of the file:
@@
 	5800 1800 6700 1800
 $Comp
-L TMC6100-EVAL-v1.2-rescue:TMC6100-TA-Trinamic IC301
+L TMC6100-EVAL-v1.2-rescue:TMC6100-TA-Trinamic-TMC6100-EVAL-v1.2-rescue IC301
 U 1 1 5D604226
 P 3750 4200
