File: tmc6100-eval/Regulator and ID.sch (KiCad schematic (older format))
At the start: 11 parts, among them U401 LP2985-3.3, U402 AT25128B-SSHL-T8S1-L

Commit message: update libs
Parts:
- U402: symbol TMC6100-EVAL-v1.2-rescue:AT25xxx-Memory_EEPROM -> TMC6100-EVAL-v1.2-rescue:AT25xxx-Memory_EEPROM-TMC6100-EVAL-v1.2-rescue
Changed lines of the file:
@@
 	1950 2800 1450 2800
 $Comp
-L TMC6100-EVAL-v1.2-rescue:AT25xxx-Memory_EEPROM U402
+L TMC6100-EVAL-v1.2-rescue:AT25xxx-Memory_EEPROM-TMC6100-EVAL-v1.2-rescue U402
 U 1 1 5D6ABCD6
 P 1950 3200
