File: opm-inline/source/Connevtors.sch (KiCad schematic (older format))
At the start: 30 parts, among them J1 Conn_01x04_Female, J2 Conn_01x02_Female, J3 Conn_01x06_Female, J4 Conn_01x02_Female, J5 Conn_01x02_Female, J6 Conn_01x03_Female, U2 TerminalBlock_2_P5.08mm, U3 TerminalBlock_3_P5.08mm

Commit message: more layout
Parts:
- removed J1: Conn_01x04_Female, Connector_PinHeader_2.54mm:PinHeader_1x04_P2.54mm_Vertical, symbol Connector:Conn_01x04_Female
- removed J4: Conn_01x02_Female, Connector_PinHeader_2.54mm:PinHeader_1x02_P2.54mm_Vertical, symbol Connector:Conn_01x02_Female
- added J1: SPI/Info, Connector_JST:JST_PH_B6B-PH-K_1x06_P2.00mm_Vertical, symbol Connector:Conn_01x06_Female
- C15, C16: value 330μF/63V -> 330uF/63V
- H201, H202, fid201, fid202, fid203: JLCPCB BOM (none) -> No
- J2: value Conn_01x02_Female -> VCC_IO; footprint Connector_PinHeader_2.54mm:PinHeader_1x02_P2.54mm_Vertical -> Connector_JST:JST_PH_B2B-PH-K_1x02_P2.00mm_Vertical; LCSC (none) -> C131337; manf_num (none) -> B2B-PH-K-S(LF)(SN)
- J3: value Conn_01x06_Female -> PWMx6; footprint Connector_PinHeader_2.54mm:PinHeader_1x06_P2.54mm_Vertical -> Connector_JST:JST_PH_B6B-PH-K_1x06_P2.00mm_Vertical; LCSC (none) -> C265365; comment (none) -> copper when possible over brass; manf_num (none) -> B6B-PH-KL(LF)(SN)
- J5: value Conn_01x02_Female -> Temperature; footprint Connector_PinHeader_2.54mm:PinHeader_1x02_P2.54mm_Vertical -> Connector_JST:JST_PH_B2B-PH-K_1x02_P2.00mm_Vertical; LCSC (none) -> C131337; manf_num (none) -> B2B-PH-K-S(LF)(SN)
- J6: value Conn_01x03_Female -> Current Sensing; footprint Connector_PinHeader_2.54mm:PinHeader_1x03_P2.54mm_Vertical -> Connector_JST:JST_PH_B3B-PH-K_1x03_P2.00mm_Vertical; LCSC (none) -> C131339; manf_num (none) -> B3B-PH-K-S(LF)(SN)
- R16: value 10000Ω/1% -> 10000R/1%
- R17, R18, R24: value 4700Ω/1% -> 4700R/1%
- R19, R21: value 1000Ω/1% -> 1000R/1%
- R20: value 150Ω/1% -> 150R/1%
- R22: value 0Ω -> 0R; LCPCB BOM (none) -> No
- R23: value 1500Ω/1% -> 1500R/1%
Connections:
- net DRV_EN: now also J1.5 (Pin_5)
- net FAULT: now also J1.6 (Pin_6)
- net SPI1_MISO: now also J1.4 (Pin_4)
- net SPI1_MOSI: now also J1.3 (Pin_3)
- net SPI1_SCK: now also J1.2 (Pin_2)
- net ~CS_DRIVER: now also J1.1 (Pin_1)
Changed lines of the file:
@@
 F 2 "Fiducial:Fiducial_0.5mm_Mask1mm" H 7650 1050 39  0001 C CNN
 F 3 "" H 7650 1050 39  0001 C CNN
+F 4 "No" H 7650 1050 50  0001 C CNN "JLCPCB BOM"
 	1    7650 1050
 	1    0    0    -1
@@
 F 2 "Fiducial:Fiducial_0.5mm_Mask1mm" H 7650 1200 39  0001 C CNN
 F 3 "" H 7650 1200 39  0001 C CNN
+F 4 "No" H 7650 1200 50  0001 C CNN "JLCPCB BOM"
 	1    7650 1200
 	1    0    0    -1
@@
 F 2 "Fiducial:Fiducial_0.5mm_Mask1mm" H 7650 1350 39  0001 C CNN
 F 3 "" H 7650 1350 39  0001 C CNN
+F 4 "No" H 7650 1350 50  0001 C CNN "JLCPCB BOM"
 	1    7650 1350
 	1    0    0    -1
@@
 F 2 "MountingHole:MountingHole_3.2mm_M3_Pad" H 6800 1300 39  0001 C CNN
 F 3 "~" H 6800 1300 39  0001 C CNN
+F 4 "No" V 6800 1300 50  0001 C CNN "JLCPCB BOM"
 	1    6800 1300
 	0    1    1    0
@@
 F 2 "MountingHole:MountingHole_3.2mm_M3_Pad" H 6800 1100 39  0001 C CNN
 F 3 "~" H 6800 1100 39  0001 C CNN
+F 4 "No" V 6800 1100 50  0001 C CNN "JLCPCB BOM"
 	1    6800 1100
 	0    1    1    0
@@
 P 2350 1500
 F 0 "C15" V 2200 1500 39  0000 C CNN
-F 1 "330μF/63V" V 2500 1500 39  0000 C CNN
+F 1 "330uF/63V" V 2500 1500 39  0000 C CNN
 F 2 "Capacitor_THT:C_Radial_D10.0mm_H20.0mm_P5.00mm" V 2550 1500 39  0001 C CNN
 F 3 "~" H 2350 1500 39  0001 C CNN
@@
 P 2850 1500
 F 0 "C16" V 2700 1500 39  0000 C CNN
-F 1 "330μF/63V" V 3000 1500 39  0000 C CNN
+F 1 "330uF/63V" V 3000 1500 39  0000 C CNN
 F 2 "Capacitor_THT:C_Radial_D10.0mm_H20.0mm_P5.00mm" H 2850 1500 39  0001 C CNN
 F 3 "~" H 2850 1500 39  0001 C CNN
@@
 P 1700 4600
 F 0 "J2" H 1592 4275 50  0000 C CNN
-F 1 "Conn_01x02_Female" H 1592 4366 50  0000 C CNN
-F 2 "Connector_PinHeader_2.54mm:PinHeader_1x02_P2.54mm_Vertical" H 1700 4600 50  0001 C CNN
-F 3 "~" H 1700 4600 50  0001 C CNN
+F 1 "VCC_IO" H 1592 4366 50  0000 C CNN
+F 2 "Connector_JST:JST_PH_B2B-PH-K_1x02_P2.00mm_Vertical" H 1700 4600 50  0001 C CNN
+F 3 "https://datasheet.lcsc.com/lcsc/1811151524_JST-Sales-America-B2B-PH-K-S-LF-SN_C131337.pdf" H 1700 4600 50  0001 C CNN
+F 4 "C131337" H 1700 4600 50  0001 C CNN "LCSC"
+F 5 "B2B-PH-K-S(LF)(SN)" H 1700 4600 50  0001 C CNN "manf_num"
 	1    1700 4600
-	1    0    0    -1
-$EndComp
-$Comp
-L Connector:Conn_01x04_Female J1
-U 1 1 61C15E32
-P 1550 5500
-F 0 "J1" H 1442 5075 50  0000 C CNN
-F 1 "Conn_01x04_Female" H 1442 5166 50  0000 C CNN
-F 2 "Connector_PinHeader_2.54mm:PinHeader_1x04_P2.54mm_Vertical" H 1550 5500 50  0001 C CNN
-F 3 "~" H 1550 5500 50  0001 C CNN
-	1    1550 5500
 	1    0    0    -1
 $EndComp
@@
 P 4550 1500
 F 0 "R19" V 4343 1500 50  0000 C CNN
-F 1 "1000Ω/1%" V 4434 1500 50  0000 C CNN
+F 1 "1000R/1%" V 4434 1500 50  0000 C CNN
 F 2 "Resistor_SMD:R_0603_1608Metric" V 4480 1500 50  0001 C CNN
 F 3 "https://datasheet.lcsc.com/lcsc/2110252030_UNI-ROYAL-Uniroyal-Elec-0603WAF1001T5E_C21190.pdf" H 4550 1500 50  0001 C CNN
@@
 P 4550 3000
 F 0 "R20" V 4343 3000 50  0000 C CNN
-F 1 "150Ω/1%" V 4434 3000 50  0000 C CNN
+F 1 "150R/1%" V 4434 3000 50  0000 C CNN
 F 2 "Resistor_SMD:R_0603_1608Metric" V 4480 3000 50  0001 C CNN
 F 3 "https://datasheet.lcsc.com/lcsc/2110252030_UNI-ROYAL-Uniroyal-Elec-0603WAF1500T5E_C22808.pdf" H 4550 3000 50  0001 C CNN
@@
 P 3800 5400
 F 0 "R18" H 3870 5446 50  0000 L CNN
-F 1 "4700Ω/1%" H 3870 5355 50  0000 L CNN
+F 1 "4700R/1%" H 3870 5355 50  0000 L CNN
 F 2 "Resistor_SMD:R_0603_1608Metric" V 3730 5400 50  0001 C CNN
 F 3 "https://datasheet.lcsc.com/lcsc/2110252130_UNI-ROYAL-Uniroyal-Elec-0603WAF4701T5E_C23162.pdf" H 3800 5400 50  0001 C CNN
@@
 P 3800 4800
 F 0 "R17" H 3870 4846 50  0000 L CNN
-F 1 "4700Ω/1%" H 3870 4755 50  0000 L CNN
+F 1 "4700R/1%" H 3870 4755 50  0000 L CNN
 F 2 "Resistor_SMD:R_0603_1608Metric" V 3730 4800 50  0001 C CNN
 F 3 "https://datasheet.lcsc.com/lcsc/2110252130_UNI-ROYAL-Uniroyal-Elec-0603WAF4701T5E_C23162.pdf" H 3800 4800 50  0001 C CNN
@@
 P 3800 4250
 F 0 "R16" H 3870 4296 50  0000 L CNN
-F 1 "10000Ω/1%" H 3870 4205 50  0000 L CNN
+F 1 "10000R/1%" H 3870 4205 50  0000 L CNN
 F 2 "Resistor_SMD:R_0603_1608Metric" V 3730 4250 50  0001 C CNN
 F 3 "https://datasheet.lcsc.com/lcsc/1810311113_Murata-Electronics-NCP18XH103F03RB_C13564.pdf" H 3800 4250 50  0001 C CNN
@@
 U 1 1 61C07AC4
 P 5650 5150
-F 0 "J5" H 5678 5126 50  0000 L CNN
-F 1 "Conn_01x02_Female" H 5678 5035 50  0000 L CNN
-F 2 "Connector_PinHeader_2.54mm:PinHeader_1x02_P2.54mm_Vertical" H 5650 5150 50  0001 C CNN
-F 3 "~" H 5650 5150 50  0001 C CNN
+F 0 "J5" H 5400 5200 50  0000 L CNN
+F 1 "Temperature" H 5700 5150 50  0000 L CNN
+F 2 "Connector_JST:JST_PH_B2B-PH-K_1x02_P2.00mm_Vertical" H 5650 5150 50  0001 C CNN
+F 3 "https://datasheet.lcsc.com/lcsc/1811151524_JST-Sales-America-B2B-PH-K-S-LF-SN_C131337.pdf" H 5650 5150 50  0001 C CNN
+F 4 "C131337" H 5650 5150 50  0001 C CNN "LCSC"
+F 5 "B2B-PH-K-S(LF)(SN)" H 5650 5150 50  0001 C CNN "manf_num"
 	1    5650 5150
 	1    0    0    -1
@@
 P 2600 4700
 F 0 "J3" H 2492 4175 50  0000 C CNN
-F 1 "Conn_01x06_Female" H 2492 4266 50  0000 C CNN
-F 2 "Connector_PinHeader_2.54mm:PinHeader_1x06_P2.54mm_Vertical" H 2600 4700 50  0001 C CNN
-F 3 "~" H 2600 4700 50  0001 C CNN
+F 1 "PWMx6" H 2492 4266 50  0000 C CNN
+F 2 "Connector_JST:JST_PH_B6B-PH-K_1x06_P2.00mm_Vertical" H 2600 4700 50  0001 C CNN
+F 3 "https://datasheet.lcsc.com/lcsc/1912111437_JST-Sales-America-B6B-PH-KL-LF-SN_C265365.pdf" H 2600 4700 50  0001 C CNN
+F 4 "B6B-PH-KL(LF)(SN)" H 2600 4700 50  0001 C CNN "manf_num"
+F 5 "C265365" H 2600 4700 50  0001 C CNN "LCSC"
+F 6 "copper when possible over brass" H 2600 4700 50  0001 C CNN "comment"
 	1    2600 4700
-	1    0    0    -1
-$EndComp
-$Comp
-L Connector:Conn_01x02_Female J4
-U 1 1 61C1C6CB
-P 2600 5600
-F 0 "J4" H 2492 5275 50  0000 C CNN
-F 1 "Conn_01x02_Female" H 2492 5366 50  0000 C CNN
-F 2 "Connector_PinHeader_2.54mm:PinHeader_1x02_P2.54mm_Vertical" H 2600 5600 50  0001 C CNN
-F 3 "~" H 2600 5600 50  0001 C CNN
-	1    2600 5600
 	1    0    0    -1
 $EndComp
@@
 Wire Wire Line
 	1050 4700 1050 4750
-Text HLabel 1350 5700 0    50   Input ~ 0
-SPI1_MISO
 Text HLabel 2400 5000 0    50   Input ~ 0
 UH
@@
 Text HLabel 2400 4500 0    50   Input ~ 0
 WL
-Text HLabel 2400 5600 0    50   Input ~ 0
-DRV_EN
-Text HLabel 2400 5700 0    50   Input ~ 0
-FAULT
-Text HLabel 1350 5500 0    50   Input ~ 0
-SPI1_SCK
-Text HLabel 1350 5400 0    50   Input ~ 0
-~CS_DRIVER
-Text HLabel 1350 5600 0    50   Input ~ 0
-SPI1_MOSI
 $Comp
 L Device:R R21
@@
 P 6850 3050
 F 0 "R21" H 6920 3096 50  0000 L CNN
-F 1 "1000Ω/1%" H 6920 3005 50  0000 L CNN
+F 1 "1000R/1%" H 6920 3005 50  0000 L CNN
 F 2 "Resistor_SMD:R_0603_1608Metric" V 6780 3050 50  0001 C CNN
 F 3 "~" H 6850 3050 50  0001 C CNN
@@
 P 6850 3550
 F 0 "R22" H 6920 3596 50  0000 L CNN
-F 1 "0Ω" H 6920 3505 50  0000 L CNN
+F 1 "0R" H 6920 3505 50  0000 L CNN
 F 2 "Resistor_SMD:R_0603_1608Metric" V 6780 3550 50  0001 C CNN
 F 3 "~" H 6850 3550 50  0001 C CNN
+F 4 "No" H 6850 3550 50  0001 C CNN "LCPCB BOM"
 	1    6850 3550
 	1    0    0    -1
@@
 P 7950 3050
 F 0 "R23" H 8020 3096 50  0000 L CNN
-F 1 "1500Ω/1%" H 8020 3005 50  0000 L CNN
+F 1 "1500R/1%" H 8020 3005 50  0000 L CNN
 F 2 "Resistor_SMD:R_0603_1608Metric" V 7880 3050 50  0001 C CNN
 F 3 "~" H 7950 3050 50  0001 C CNN
@@
 P 7950 3550
 F 0 "R24" H 8020 3596 50  0000 L CNN
-F 1 "4700Ω/1%" H 8020 3505 50  0000 L CNN
+F 1 "4700R/1%" H 8020 3505 50  0000 L CNN
 F 2 "Resistor_SMD:R_0603_1608Metric" V 7880 3550 50  0001 C CNN
 F 3 "https://datasheet.lcsc.com/lcsc/2110252130_UNI-ROYAL-Uniroyal-Elec-0603WAF4701T5E_C23162.pdf" H 7950 3550 50  0001 C CNN
@@
 P 1550 6450
 F 0 "J6" H 1578 6476 50  0000 L CNN
-F 1 "Conn_01x03_Female" H 1578 6385 50  0000 L CNN
-F 2 "Connector_PinHeader_2.54mm:PinHeader_1x03_P2.54mm_Vertical" H 1550 6450 50  0001 C CNN
-F 3 "~" H 1550 6450 50  0001 C CNN
+F 1 "Current Sensing" H 1578 6385 50  0000 L CNN
+F 2 "Connector_JST:JST_PH_B3B-PH-K_1x03_P2.00mm_Vertical" H 1550 6450 50  0001 C CNN
+F 3 "https://datasheet.lcsc.com/lcsc/1811151524_JST-Sales-America-B3B-PH-K-S-LF-SN_C131339.pdf" H 1550 6450 50  0001 C CNN
+F 4 "C131339" H 1550 6450 50  0001 C CNN "LCSC"
+F 5 "B3B-PH-K-S(LF)(SN)" H 1550 6450 50  0001 C CNN "manf_num"
 	1    1550 6450
 	1    0    0    -1
@@
 Wire Wire Line
 	1700 1750 2350 1750
+$Comp
+L Connector:Conn_01x06_Female J1
+U 1 1 61C4DAFD
+P 1600 5500
+F 0 "J1" H 1700 5400 50  0000 C CNN
+F 1 "SPI/Info" H 1800 5500 50  0000 C CNN
+F 2 "Connector_JST:JST_PH_B6B-PH-K_1x06_P2.00mm_Vertical" H 1600 5500 50  0001 C CNN
+F 3 "https://datasheet.lcsc.com/lcsc/1912111437_JST-Sales-America-B6B-PH-KL-LF-SN_C265365.pdf" H 1600 5500 50  0001 C CNN
+F 4 "C265365" H 1600 5500 50  0001 C CNN "LCSC"
+F 5 "B6B-PH-KL(LF)(SN)" H 1600 5500 50  0001 C CNN "manf_num"
+F 6 "copper when possible over brass" H 1600 5500 50  0001 C CNN "comment"
+	1    1600 5500
+	1    0    0    -1
+$EndComp
+Text HLabel 1400 5600 0    50   Input ~ 0
+SPI1_MISO
+Text HLabel 1400 5700 0    50   Input ~ 0
+DRV_EN
+Text HLabel 1400 5800 0    50   Input ~ 0
+FAULT
+Text HLabel 1400 5400 0    50   Input ~ 0
+SPI1_SCK
+Text HLabel 1400 5300 0    50   Input ~ 0
+~CS_DRIVER
+Text HLabel 1400 5500 0    50   Input ~ 0
+SPI1_MOSI
 $EndSCHEMATC
