File: opm-inline/source/Connevtors.sch (KiCad schematic (older format))
At the start: 29 parts, among them J1 SPI/Info, J2 VCC_IO, J3 PWMx6, J5 Temperature, J6 Current Sensing, U2 TerminalBlock_2_P5.08mm, U3 TerminalBlock_3_P5.08mm

Commit message: update from latest
Parts:
- U2: footprint TerminalBlock:TerminalBlock_bornier-2_P5.08mm -> Libraries:TerminalBlock_bornier-2_P5.08mm
- U3: footprint TerminalBlock:TerminalBlock_bornier-3_P5.08mm -> Libraries:TerminalBlock_bornier-3_P5.08mm
Changed lines of the file:
@@
 F 0 "U3" H 2400 2950 39  0000 C CNN
 F 1 "TerminalBlock_3_P5.08mm" H 2400 2900 39  0000 C CNN
-F 2 "TerminalBlock:TerminalBlock_bornier-3_P5.08mm" H 2400 2350 39  0001 C CNN
+F 2 "Libraries:TerminalBlock_bornier-3_P5.08mm" H 2400 2350 39  0001 C CNN
 F 3 "http://www.farnell.com/datasheets/2336348.pdf" H 2450 2650 39  0001 C CNN
 	1    2400 2700
@@
 F 0 "U2" H 1500 1100 39  0000 C CNN
 F 1 "TerminalBlock_2_P5.08mm" H 1500 1150 39  0000 C CNN
-F 2 "TerminalBlock:TerminalBlock_bornier-2_P5.08mm" H 1500 1150 39  0001 C CNN
+F 2 "Libraries:TerminalBlock_bornier-2_P5.08mm" H 1500 1150 39  0001 C CNN
 F 3 "" H 1550 1300 39  0001 C CNN
 	1    1500 1300

Commit message: fix some parts
Parts:
- removed fid201, fid202, fid203: fiducial, Fiducial:Fiducial_0.5mm_Mask1mm, symbol fiducual:fiducial-markings
- R21: LCSC (none) -> C21190; manf_num (none) -> 0603WAF1001T5E
- R23: LCSC (none) -> C22843; manf_num (none) -> 0603WAF1501T5E
- U2: LCSC (none) -> C8465; manf_num (none) -> WJ500V-5.08-2P
- U3: LCSC (none) -> C72334; manf_num (none) -> WJ500V-5.08-3P
Other:
- note removed: "Fiducials"
Changed lines of the file:
@@
 Comment4 ""
 $EndDescr
-$Comp
-L fiducual:fiducial-markings fid201
-U 1 1 5C6BBB15
-P 7650 1050
-F 0 "fid201" H 7750 1100 39  0000 L CNN
-F 1 "fiducial" H 7750 1050 39  0000 L CNN
-F 2 "Fiducial:Fiducial_0.5mm_Mask1mm" H 7650 1050 39  0001 C CNN
-F 3 "" H 7650 1050 39  0001 C CNN
-F 4 "No" H 7650 1050 50  0001 C CNN "JLCPCB BOM"
-	1    7650 1050
-	1    0    0    -1
-$EndComp
-$Comp
-L fiducual:fiducial-markings fid202
-U 1 1 5C6BC61F
-P 7650 1200
-F 0 "fid202" H 7750 1250 39  0000 L CNN
-F 1 "fiducial" H 7750 1200 39  0000 L CNN
-F 2 "Fiducial:Fiducial_0.5mm_Mask1mm" H 7650 1200 39  0001 C CNN
-F 3 "" H 7650 1200 39  0001 C CNN
-F 4 "No" H 7650 1200 50  0001 C CNN "JLCPCB BOM"
-	1    7650 1200
-	1    0    0    -1
-$EndComp
-$Comp
-L fiducual:fiducial-markings fid203
-U 1 1 5C6BC9A9
-P 7650 1350
-F 0 "fid203" H 7750 1400 39  0000 L CNN
-F 1 "fiducial" H 7750 1350 39  0000 L CNN
-F 2 "Fiducial:Fiducial_0.5mm_Mask1mm" H 7650 1350 39  0001 C CNN
-F 3 "" H 7650 1350 39  0001 C CNN
-F 4 "No" H 7650 1350 50  0001 C CNN "JLCPCB BOM"
-	1    7650 1350
-	1    0    0    -1
-$EndComp
-Text Notes 7550 900  0    79   ~ 0
-Fiducials
-Wire Notes Line
-	8150 1450 8150 750
-Wire Notes Line
-	8150 750  7500 750
-Wire Notes Line
-	7500 1450 8150 1450
-Wire Notes Line
-	7500 750  7500 1450
 Wire Notes Line
 	7400 750  6400 750
@@
 F 1 "TerminalBlock_3_P5.08mm" H 2400 2900 39  0000 C CNN
 F 2 "Libraries:TerminalBlock_bornier-3_P5.08mm" H 2400 2350 39  0001 C CNN
-F 3 "http://www.farnell.com/datasheets/2336348.pdf" H 2450 2650 39  0001 C CNN
+F 3 "https://datasheet.lcsc.com/lcsc/1912251709_Ningbo-Kangnex-Elec-WJ500V-5-08-3P_C72334.pdf" H 2450 2650 39  0001 C CNN
+F 4 "C72334" H 2400 2700 50  0001 C CNN "LCSC"
+F 5 "WJ500V-5.08-3P" H 2400 2700 50  0001 C CNN "manf_num"
 	1    2400 2700
 	1    0    0    -1
@@
 F 1 "TerminalBlock_2_P5.08mm" H 1500 1150 39  0000 C CNN
 F 2 "Libraries:TerminalBlock_bornier-2_P5.08mm" H 1500 1150 39  0001 C CNN
-F 3 "" H 1550 1300 39  0001 C CNN
+F 3 "https://datasheet.lcsc.com/lcsc/1912251636_Ningbo-Kangnex-Elec-WJ500V-5-08-2P_C8465.pdf" H 1550 1300 39  0001 C CNN
+F 4 "C8465" H 1500 1300 50  0001 C CNN "LCSC"
+F 5 "WJ500V-5.08-2P" H 1500 1300 50  0001 C CNN "manf_num"
 	1    1500 1300
 	-1   0    0    1
@@
 F 1 "1000R/1%" H 6920 3005 50  0000 L CNN
 F 2 "Resistor_SMD:R_0603_1608Metric" V 6780 3050 50  0001 C CNN
-F 3 "~" H 6850 3050 50  0001 C CNN
+F 3 "https://datasheet.lcsc.com/lcsc/2110252030_UNI-ROYAL-Uniroyal-Elec-0603WAF1001T5E_C21190.pdf" H 6850 3050 50  0001 C CNN
+F 4 "C21190" H 6850 3050 50  0001 C CNN "LCSC"
+F 5 "0603WAF1001T5E" H 6850 3050 50  0001 C CNN "manf_num"
 	1    6850 3050
 	1    0    0    -1
@@
 F 1 "1500R/1%" H 8020 3005 50  0000 L CNN
 F 2 "Resistor_SMD:R_0603_1608Metric" V 7880 3050 50  0001 C CNN
-F 3 "~" H 7950 3050 50  0001 C CNN
+F 3 "https://datasheet.lcsc.com/lcsc/2110252030_UNI-ROYAL-Uniroyal-Elec-0603WAF1501T5E_C22843.pdf" H 7950 3050 50  0001 C CNN
+F 4 "C22843" H 7950 3050 50  0001 C CNN "LCSC"
+F 5 "0603WAF1501T5E" H 7950 3050 50  0001 C CNN "manf_num"
 	1    7950 3050
 	1    0    0    -1
