File: opm-inline/source/Motor Driver.sch (KiCad schematic (older format))
At the start: 55 parts, among them IC301 TMC6100-LA, Q301 YJG95G06A, Q302 YJG95G06A, Q303 YJG95G06A, Q304 YJG95G06A, Q305 YJG95G06A, Q306 YJG95G06A, U1 INA180A3IDBVR, U2 INA180A3IDBVR, U3 INA180A3IDBVR

Commit message: some work on inline
Parts:
- removed C303, C310, C318: 470nF/16V, Capacitor_SMD:C_0603_1608Metric, symbol Device:C
- removed C304, C314, C319: 2,2μF/100V, Capacitor_SMD:C_1210_3225Metric, symbol Device:C
- removed C305, C307: 100nF/100V, Capacitor_SMD:C_0805_2012Metric, symbol Device:C
- removed C306: 22nF/100V, Capacitor_SMD:C_0603_1608Metric, symbol Device:C
- removed IC301: TMC6100-LA, Trinamic:QFN-44-1EP_7x7mm_P0.5mm_EP4x4mm, symbol opm-lowside-rescue:TMC6100-LA-opm-v1.2-rescue
- removed Q301, Q302, Q303, Q304, Q305, Q306: YJG95G06A, Package_TO_SOT_SMD:TDSON-8-1, symbol opm-lowside-rescue:YJG95G06A-Transistor_FET-opm-v1.1-rescue
- removed R304, R306, R310, R313, R318, R320: 2,2Ω/1%, Resistor_SMD:R_0603_1608Metric, symbol Device:R
- removed U1, U2, U3: INA180A3IDBVR, SOT95P280X145-5N:SOT95P280X145-5N, symbol amplifier:INA180A3IDBVR
- added IC1: TMC6200-TA, Trinamic:QFN-44-1EP_7x7mm_P0.5mm_EP4x4mm, symbol opm-inline-rescue:TMC6200-TA-opm-inline-cache
- added Q1, Q2, Q3, Q4, Q5, Q6: YJG95G06A, Package_TO_SOT_SMD:TDSON-8-1, symbol opm-inline-cache:opm-inline-rescue_YJG95G06A-Transistor_FET-opm-v1.1-rescue-opm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
- C1, C2, C3: value 0.1uF -> C
- C4, C5, C6: value 3300pF -> C
- C7, C8, C9: value 1000pF -> C
- R1, R2, R3, R4, R5, R6: value .001Ω/1% -> R
- R10, R11, R12, R7, R8, R9: value 10Ω/1% -> R
- R13, R14, R15: value 100Ω/5% -> R
Connections:
- net labels removed: +5V, DRV_EN, FAULT, SPE, SPI2_MISO, SPI2_MOSI, SPI2_SCK, U-IA-IDC, UH, UL, V-IA-IDC, VCP, VH, VL, W-IA-IDC, WH, WL, ~CS_DRIVER
- wire segments 194 -> 148
Other:
- moved on the sheet: C311, C312, C313, C315, R311, R314

Commit message: add some values
Parts:
- C4, C5, C6: value C -> 470nF
- C7, C8, C9: value C -> 2.2uF/100V
- R1, R11, R13, R3, R4, R6: value R -> 2R2/1%
- R10, R14, R15, R7, R8, R9: value R -> 0R033/1%/2W
- R12, R2, R5: value R -> 10R/1%
Other:
- moved on the sheet: R10, R14, R15, R7, R8, R9
Changed lines of the file:
@@
 P 7050 5150
 F 0 "R4" V 6876 5150 35  0000 C CNN
-F 1 "R" V 6945 5150 35  0000 C CNN
+F 1 "2R2/1%" V 6945 5150 35  0000 C CNN
 F 2 "Resistor_SMD:R_0603_1608Metric" V 6980 5150 50  0001 C CNN
 F 3 "~" H 7050 5150 50  0001 C CNN
@@
 P 7050 5550
 F 0 "R5" V 6876 5550 35  0000 C CNN
-F 1 "R" V 6945 5550 35  0000 C CNN
+F 1 "10R/1%" V 6945 5550 35  0000 C CNN
 F 2 "Resistor_SMD:R_0603_1608Metric" V 6980 5550 50  0001 C CNN
 F 3 "~" H 7050 5550 50  0001 C CNN
@@
 P 7050 5950
 F 0 "R6" V 6876 5950 35  0000 C CNN
-F 1 "R" V 6945 5950 35  0000 C CNN
+F 1 "2R2/1%" V 6945 5950 35  0000 C CNN
 F 2 "Resistor_SMD:R_0603_1608Metric" V 6980 5950 50  0001 C CNN
 F 3 "~" H 7050 5950 50  0001 C CNN
@@
 L Device:R R9
 U 1 1 61C5CFCB
-P 8600 5400
-F 0 "R9" V 8426 5400 35  0000 C CNN
-F 1 "R" V 8495 5400 35  0000 C CNN
-F 2 "Resistor_SMD:R_0603_1608Metric" V 8530 5400 50  0001 C CNN
-F 3 "~" H 8600 5400 50  0001 C CNN
-	1    8600 5400
+P 8750 5400
+F 0 "R9" V 8576 5400 35  0000 C CNN
+F 1 "0R033/1%/2W" V 8645 5400 35  0000 C CNN
+F 2 "Resistor_SMD:R_0603_1608Metric" V 8680 5400 50  0001 C CNN
+F 3 "~" H 8750 5400 50  0001 C CNN
+	1    8750 5400
 	0    1    1    0
 $EndComp
@@
 L Device:R R10
 U 1 1 61C5DC5F
-P 8600 5700
-F 0 "R10" V 8426 5700 35  0000 C CNN
-F 1 "R" V 8495 5700 35  0000 C CNN
-F 2 "Resistor_SMD:R_0603_1608Metric" V 8530 5700 50  0001 C CNN
-F 3 "~" H 8600 5700 50  0001 C CNN
-	1    8600 5700
+P 8750 5700
+F 0 "R10" V 8576 5700 35  0000 C CNN
+F 1 "0R033/1%/2W" V 8645 5700 35  0000 C CNN
+F 2 "Resistor_SMD:R_0603_1608Metric" V 8680 5700 50  0001 C CNN
+F 3 "~" H 8750 5700 50  0001 C CNN
+	1    8750 5700
 	0    1    1    0
 $EndComp
@@
 $EndComp
 Wire Wire Line
-	7200 5550 9000 5550
-Wire Wire Line
-	9000 5700 8750 5700
+	9150 5700 8900 5700
 Wire Wire Line
 	7200 5950 7500 5950
@@
 Wire Wire Line
 	7500 5150 7200 5150
-Wire Wire Line
-	8450 5700 7800 5700
 Wire Wire Line
 	7800 5700 7800 5750
@@
 Connection ~ 7800 5700
 Wire Wire Line
-	8450 5400 7800 5400
-Wire Wire Line
 	7800 5350 7800 5400
 Connection ~ 7800 5400
@@
 	7800 5400 7800 5500
 Wire Wire Line
-	8750 5400 9000 5400
-Wire Wire Line
-	9000 5400 9000 5550
-Wire Wire Line
-	9000 5550 9000 5700
-Connection ~ 9000 5550
+	8900 5400 9150 5400
+Wire Wire Line
+	9150 5400 9150 5550
+Wire Wire Line
+	9150 5550 9150 5700
+Connection ~ 9150 5550
 Wire Wire Line
 	7800 6150 7800 6250
@@
 P 8350 4950
 F 0 "C8" H 8465 4985 35  0000 L CNN
-F 1 "C" H 8465 4916 35  0000 L CNN
+F 1 "2.2uF/100V" H 8465 4916 35  0000 L CNN
 F 2 "Capacitor_SMD:C_0603_1608Metric" H 8388 4800 50  0001 C CNN
 F 3 "~" H 8350 4950 50  0001 C CNN
@@
 U 1 1 61C4C1D6
 P 6600 4600
-F 0 "C5" V 6381 4600 35  0000 C CNN
-F 1 "C" V 6450 4600 35  0000 C CNN
+F 0 "C5" H 6715 4635 35  0000 L CNN
+F 1 "470nF" H 6715 4566 35  0000 L CNN
 F 2 "Capacitor_SMD:C_0603_1608Metric" H 6638 4450 50  0001 C CNN
 F 3 "~" H 6600 4600 50  0001 C CNN
@@
 P 8700 3650
 F 0 "R11" V 8526 3650 35  0000 C CNN
-F 1 "R" V 8595 3650 35  0000 C CNN
+F 1 "2R2/1%" V 8595 3650 35  0000 C CNN
 F 2 "Resistor_SMD:R_0603_1608Metric" V 8630 3650 50  0001 C CNN
 F 3 "~" H 8700 3650 50  0001 C CNN
@@
 P 8700 4050
 F 0 "R12" V 8526 4050 35  0000 C CNN
-F 1 "R" V 8595 4050 35  0000 C CNN
+F 1 "10R/1%" V 8595 4050 35  0000 C CNN
 F 2 "Resistor_SMD:R_0603_1608Metric" V 8630 4050 50  0001 C CNN
 F 3 "~" H 8700 4050 50  0001 C CNN
@@
 P 8700 4450
 F 0 "R13" V 8526 4450 35  0000 C CNN
-F 1 "R" V 8595 4450 35  0000 C CNN
+F 1 "2R2/1%" V 8595 4450 35  0000 C CNN
 F 2 "Resistor_SMD:R_0603_1608Metric" V 8630 4450 50  0001 C CNN
 F 3 "~" H 8700 4450 50  0001 C CNN
@@
 L Device:R R14
 U 1 1 61D8AF32
-P 10250 3900
-F 0 "R14" V 10076 3900 35  0000 C CNN
-F 1 "R" V 10145 3900 35  0000 C CNN
-F 2 "Resistor_SMD:R_0603_1608Metric" V 10180 3900 50  0001 C CNN
-F 3 "~" H 10250 3900 50  0001 C CNN
-	1    10250 3900
+P 10400 3900
+F 0 "R14" V 10226 3900 35  0000 C CNN
+F 1 "0R033/1%/2W" V 10295 3900 35  0000 C CNN
+F 2 "Resistor_SMD:R_0603_1608Metric" V 10330 3900 50  0001 C CNN
+F 3 "~" H 10400 3900 50  0001 C CNN
+	1    10400 3900
 	0    1    1    0
 $EndComp
@@
 L Device:R R15
 U 1 1 61D8AF3C
-P 10250 4200
-F 0 "R15" V 10076 4200 35  0000 C CNN
-F 1 "R" V 10145 4200 35  0000 C CNN
-F 2 "Resistor_SMD:R_0603_1608Metric" V 10180 4200 50  0001 C CNN
-F 3 "~" H 10250 4200 50  0001 C CNN
-	1    10250 4200
+P 10400 4200
+F 0 "R15" V 10226 4200 35  0000 C CNN
+F 1 "0R033/1%/2W" V 10295 4200 35  0000 C CNN
+F 2 "Resistor_SMD:R_0603_1608Metric" V 10330 4200 50  0001 C CNN
+F 3 "~" H 10400 4200 50  0001 C CNN
+	1    10400 4200
 	0    1    1    0
 $EndComp
@@
 $EndComp
 Wire Wire Line
-	8850 4050 10650 4050
-Wire Wire Line
-	10650 4200 10400 4200
+	10800 4200 10550 4200
 Wire Wire Line
 	8850 4450 9150 4450
@@
 Wire Wire Line
 	9150 3650 8850 3650
-Wire Wire Line
-	10100 4200 9450 4200
-Wire Wire Line
-	9450 4200 9450 4250
 Connection ~ 9450 4250
-Connection ~ 9450 4200
-Wire Wire Line
-	10100 3900 9450 3900
-Wire Wire Line
-	9450 3850 9450 3900
-Connection ~ 9450 3900
-Wire Wire Line
-	9450 3900 9450 4200
-Wire Wire Line
-	10400 3900 10650 3900
-Wire Wire Line
-	10650 3900 10650 4050
-Wire Wire Line
-	10650 4050 10650 4200
-Connection ~ 10650 4050
+Wire Wire Line
+	10550 3900 10800 3900
+Wire Wire Line
+	10800 3900 10800 4050
+Wire Wire Line
+	10800 4050 10800 4200
+Connection ~ 10800 4050
 Wire Wire Line
 	9450 4650 9450 4750
@@
 P 10000 3450
 F 0 "C9" H 10115 3485 35  0000 L CNN
-F 1 "C" H 10115 3416 35  0000 L CNN
+F 1 "2.2uF/100V" H 10115 3416 35  0000 L CNN
 F 2 "Capacitor_SMD:C_0603_1608Metric" H 10038 3300 50  0001 C CNN
 F 3 "~" H 10000 3450 50  0001 C CNN
@@
 P 7050 2350
 F 0 "R1" V 6876 2350 35  0000 C CNN
-F 1 "R" V 6945 2350 35  0000 C CNN
+F 1 "2R2/1%" V 6945 2350 35  0000 C CNN
 F 2 "Resistor_SMD:R_0603_1608Metric" V 6980 2350 50  0001 C CNN
 F 3 "~" H 7050 2350 50  0001 C CNN
@@
 P 7050 2750
 F 0 "R2" V 6876 2750 35  0000 C CNN
-F 1 "R" V 6945 2750 35  0000 C CNN
+F 1 "10R/1%" V 6945 2750 35  0000 C CNN
 F 2 "Resistor_SMD:R_0603_1608Metric" V 6980 2750 50  0001 C CNN
 F 3 "~" H 7050 2750 50  0001 C CNN
@@
 P 7050 3150
 F 0 "R3" V 6876 3150 35  0000 C CNN
-F 1 "R" V 6945 3150 35  0000 C CNN
+F 1 "2R2/1%" V 6945 3150 35  0000 C CNN
 F 2 "Resistor_SMD:R_0603_1608Metric" V 6980 3150 50  0001 C CNN
 F 3 "~" H 7050 3150 50  0001 C CNN
@@
 	7500 2350 7200 2350
 Wire Wire Line
-	8450 2900 7800 2900
-Wire Wire Line
 	7800 2900 7800 2950
 Connection ~ 7800 2950
 Connection ~ 7800 2900
-Wire Wire Line
-	8450 2600 7800 2600
 Wire Wire Line
 	7800 2550 7800 2600
@@
 P 8350 2150
 F 0 "C7" H 8465 2185 35  0000 L CNN
-F 1 "C" H 8465 2116 35  0000 L CNN
+F 1 "2.2uF/100V" H 8465 2116 35  0000 L CNN
 F 2 "Capacitor_SMD:C_0603_1608Metric" H 8388 2000 50  0001 C CNN
 F 3 "~" H 8350 2150 50  0001 C CNN
@@
 P 5650 3400
 F 0 "C4" V 5431 3400 35  0000 C CNN
-F 1 "C" V 5500 3400 35  0000 C CNN
+F 1 "470nF" V 5500 3400 35  0000 C CNN
 F 2 "Capacitor_SMD:C_0603_1608Metric" H 5688 3250 50  0001 C CNN
 F 3 "~" H 5650 3400 50  0001 C CNN
@@
 P 6750 3750
 F 0 "C6" V 6531 3750 35  0000 C CNN
-F 1 "C" V 6600 3750 35  0000 C CNN
+F 1 "470nF" V 6600 3750 35  0000 C CNN
 F 2 "Capacitor_SMD:C_0603_1608Metric" H 6788 3600 50  0001 C CNN
 F 3 "~" H 6750 3750 50  0001 C CNN
@@
 L Device:R R7
 U 1 1 61E48788
-P 8600 2600
-F 0 "R7" V 8426 2600 35  0000 C CNN
-F 1 "R" V 8495 2600 35  0000 C CNN
-F 2 "Resistor_SMD:R_0603_1608Metric" V 8530 2600 50  0001 C CNN
-F 3 "~" H 8600 2600 50  0001 C CNN
-	1    8600 2600
+P 8750 2600
+F 0 "R7" V 8576 2600 35  0000 C CNN
+F 1 "0R033/1%/2W" V 8645 2600 35  0000 C CNN
+F 2 "Resistor_SMD:R_0603_1608Metric" V 8680 2600 50  0001 C CNN
+F 3 "~" H 8750 2600 50  0001 C CNN
+	1    8750 2600
 	0    1    1    0
 $EndComp
@@
 L Device:R R8
 U 1 1 61E48BDE
-P 8600 2900
-F 0 "R8" V 8426 2900 35  0000 C CNN
-F 1 "R" V 8495 2900 35  0000 C CNN
-F 2 "Resistor_SMD:R_0603_1608Metric" V 8530 2900 50  0001 C CNN
-F 3 "~" H 8600 2900 50  0001 C CNN
-	1    8600 2900
-	0    1    1    0
-$EndComp
-Wire Wire Line
-	7200 2750 9000 2750
-Wire Wire Line
-	9000 2900 8750 2900
-Wire Wire Line
-	8750 2600 9000 2600
-Wire Wire Line
-	9000 2600 9000 2750
-Wire Wire Line
-	9000 2750 9000 2900
-Connection ~ 9000 2750
+P 8750 2900
+F 0 "R8" V 8576 2900 35  0000 C CNN
+F 1 "0R033/1%/2W" V 8645 2900 35  0000 C CNN
+F 2 "Resistor_SMD:R_0603_1608Metric" V 8680 2900 50  0001 C CNN
+F 3 "~" H 8750 2900 50  0001 C CNN
+	1    8750 2900
+	0    1    1    0
+$EndComp
+Wire Wire Line
+	9150 2900 8900 2900
+Wire Wire Line
+	8900 2600 9150 2600
+Wire Wire Line
+	9150 2600 9150 2750
+Wire Wire Line
+	9150 2750 9150 2900
+Connection ~ 9150 2750
 Wire Wire Line
 	4800 3200 4800 3400
@@
 Wire Wire Line
 	2500 3550 2500 3450
+Wire Wire Line
+	7200 5550 9150 5550
+Wire Wire Line
+	7800 5400 8600 5400
+Wire Wire Line
+	7800 5700 8600 5700
+Wire Wire Line
+	8850 4050 10800 4050
+Wire Wire Line
+	9450 3900 10250 3900
+Wire Wire Line
+	9450 3850 9450 3900
+Connection ~ 9450 3900
+Wire Wire Line
+	9450 3900 9450 4200
+Wire Wire Line
+	9450 4200 10250 4200
+Connection ~ 9450 4200
+Wire Wire Line
+	9450 4200 9450 4250
+Wire Wire Line
+	7800 2600 8600 2600
+Wire Wire Line
+	7800 2900 8600 2900
+Wire Wire Line
+	7200 2750 9150 2750
 $EndSCHEMATC

Commit message: more value updates
Parts:
- added C10: 100nF/50V, symbol Device:C
- C1: value C -> 22nF/100V
- C2, C3: value C -> 100nF/100V
- C5, C6: value 470nF -> 470nF/16V
- Q1, Q2, Q3, Q4, Q5, Q6: symbol opm-inline-cache:opm-inline-rescue_YJG95G06A-Transistor_FET-opm-v1.1-rescue-opm-lowside-rescue -> opm-inline-rescue:opm-inline-rescue_YJG95G06A-Transistor_FET-opm-v1.1-rescue-opm-lowside-rescue-opm-inline-cache
Connections:
- net labels added: VOFS
- wire segments 148 -> 152
Changed lines of the file:
@@
 Wire Wire Line
 	3450 4850 3450 4950
-Connection ~ 3450 4850
-Wire Wire Line
-	3450 4850 4400 4850
 $Comp
 L Device:C C315
@@
 	4900 5300 4900 5050
 $Comp
-L opm-inline-cache:opm-inline-rescue_YJG95G06A-Transistor_FET-opm-v1.1-rescue-opm-lowside-rescue Q3
+L opm-inline-rescue:opm-inline-rescue_YJG95G06A-Transistor_FET-opm-v1.1-rescue-opm-lowside-rescue-opm-inline-cache Q3
 U 1 1 61C4D7D0
 P 7700 5150
+AR Path="/61C4D7D0" Ref="Q3"  Part="1"
+AR Path="/5D5FDD98/61C4D7D0" Ref="Q3"  Part="1"
 F 0 "Q3" V 8031 5188 39  0000 R BNN
 F 1 "YJG95G06A" V 8031 5113 39  0000 C TNN
@@
 $EndComp
 $Comp
-L opm-inline-cache:opm-inline-rescue_YJG95G06A-Transistor_FET-opm-v1.1-rescue-opm-lowside-rescue Q4
+L opm-inline-rescue:opm-inline-rescue_YJG95G06A-Transistor_FET-opm-v1.1-rescue-opm-lowside-rescue-opm-inline-cache Q4
 U 1 1 61C4FD8F
 P 7700 5950
+AR Path="/61C4FD8F" Ref="Q4"  Part="1"
+AR Path="/5D5FDD98/61C4FD8F" Ref="Q4"  Part="1"
 F 0 "Q4" H 8031 5988 39  0000 L CNN
 F 1 "YJG95G06A" H 8031 5913 39  0000 L CNN
@@
 P 6600 4600
 F 0 "C5" H 6715 4635 35  0000 L CNN
-F 1 "470nF" H 6715 4566 35  0000 L CNN
+F 1 "470nF/16V" H 6715 4566 35  0000 L CNN
 F 2 "Capacitor_SMD:C_0603_1608Metric" H 6638 4450 50  0001 C CNN
 F 3 "~" H 6600 4600 50  0001 C CNN
@@
 $EndComp
 $Comp
-L opm-inline-cache:opm-inline-rescue_YJG95G06A-Transistor_FET-opm-v1.1-rescue-opm-lowside-rescue Q5
+L opm-inline-rescue:opm-inline-rescue_YJG95G06A-Transistor_FET-opm-v1.1-rescue-opm-lowside-rescue-opm-inline-cache Q5
 U 1 1 61D8AC5E
 P 9350 3650
+AR Path="/61D8AC5E" Ref="Q5"  Part="1"
+AR Path="/5D5FDD98/61D8AC5E" Ref="Q5"  Part="1"
 F 0 "Q5" V 9681 3688 39  0000 R BNN
 F 1 "YJG95G06A" V 9681 3613 39  0000 C TNN
@@
 $EndComp
 $Comp
-L opm-inline-cache:opm-inline-rescue_YJG95G06A-Transistor_FET-opm-v1.1-rescue-opm-lowside-rescue Q6
+L opm-inline-rescue:opm-inline-rescue_YJG95G06A-Transistor_FET-opm-v1.1-rescue-opm-lowside-rescue-opm-inline-cache Q6
 U 1 1 61D8AF0A
 P 9350 4450
+AR Path="/61D8AF0A" Ref="Q6"  Part="1"
+AR Path="/5D5FDD98/61D8AF0A" Ref="Q6"  Part="1"
 F 0 "Q6" H 9681 4488 39  0000 L CNN
 F 1 "YJG95G06A" H 9681 4413 39  0000 L CNN
@@
 Connection ~ 9450 3200
 $Comp
-L opm-inline-cache:opm-inline-rescue_YJG95G06A-Transistor_FET-opm-v1.1-rescue-opm-lowside-rescue Q1
+L opm-inline-rescue:opm-inline-rescue_YJG95G06A-Transistor_FET-opm-v1.1-rescue-opm-lowside-rescue-opm-inline-cache Q1
 U 1 1 61D9B312
 P 7700 2350
+AR Path="/61D9B312" Ref="Q1"  Part="1"
+AR Path="/5D5FDD98/61D9B312" Ref="Q1"  Part="1"
 F 0 "Q1" V 8031 2388 39  0000 R BNN
 F 1 "YJG95G06A" V 8031 2313 39  0000 C TNN
@@
 $EndComp
 $Comp
-L opm-inline-cache:opm-inline-rescue_YJG95G06A-Transistor_FET-opm-v1.1-rescue-opm-lowside-rescue Q2
+L opm-inline-rescue:opm-inline-rescue_YJG95G06A-Transistor_FET-opm-v1.1-rescue-opm-lowside-rescue-opm-inline-cache Q2
 U 1 1 61D9B6B4
 P 7700 3150
+AR Path="/61D9B6B4" Ref="Q2"  Part="1"
+AR Path="/5D5FDD98/61D9B6B4" Ref="Q2"  Part="1"
 F 0 "Q2" H 8031 3188 39  0000 L CNN
 F 1 "YJG95G06A" H 8031 3113 39  0000 L CNN
@@
 U 1 1 61DA87F1
 P 4650 3200
-F 0 "C1" V 4902 3200 50  0000 C CNN
-F 1 "C" V 4811 3200 50  0000 C CNN
+F 0 "C1" V 4902 3200 35  0000 C CNN
+F 1 "22nF/100V" V 4811 3200 35  0000 C CNN
 F 2 "Capacitor_SMD:C_0603_1608Metric" H 4688 3050 50  0001 C CNN
 F 3 "~" H 4650 3200 50  0001 C CNN
@@
 U 1 1 61DA9103
 P 5050 3200
-F 0 "C2" V 4798 3200 50  0000 C CNN
-F 1 "C" V 4889 3200 50  0000 C CNN
+F 0 "C2" V 4798 3200 35  0000 C CNN
+F 1 "100nF/100V" V 4889 3200 35  0000 C CNN
 F 2 "Capacitor_SMD:C_0603_1608Metric" H 5088 3050 50  0001 C CNN
 F 3 "~" H 5050 3200 50  0001 C CNN
@@
 U 1 1 61DABDB6
 P 5400 2800
-F 0 "C3" H 5515 2846 50  0000 L CNN
-F 1 "C" H 5515 2755 50  0000 L CNN
+F 0 "C3" H 5515 2846 35  0000 L CNN
+F 1 "100nF/100V" H 5515 2755 35  0000 L CNN
 F 2 "Capacitor_SMD:C_0603_1608Metric" H 5438 2650 50  0001 C CNN
 F 3 "~" H 5400 2800 50  0001 C CNN
@@
 P 6750 3750
 F 0 "C6" V 6531 3750 35  0000 C CNN
-F 1 "470nF" V 6600 3750 35  0000 C CNN
+F 1 "470nF/16V" V 6600 3750 35  0000 C CNN
 F 2 "Capacitor_SMD:C_0603_1608Metric" H 6788 3600 50  0001 C CNN
 F 3 "~" H 6750 3750 50  0001 C CNN
@@
 Wire Wire Line
 	7200 2750 9150 2750
+Connection ~ 3450 4850
+Wire Wire Line
+	3450 4850 4400 4850
+$Comp
+L Device:C C10
+U 1 1 61F37D7D
+P 5650 4950
+F 0 "C10" H 5765 4985 35  0000 L CNN
+F 1 "100nF/50V" H 5765 4916 35  0000 L CNN
+F 2 "" H 5688 4800 50  0001 C CNN
+F 3 "~" H 5650 4950 50  0001 C CNN
+	1    5650 4950
+	1    0    0    -1
+$EndComp
+Wire Wire Line
+	5650 4800 5650 4750
+Wire Wire Line
+	5650 4750 5400 4750
+$Comp
+L power:GND #PWR09
+U 1 1 61F3EA05
+P 5650 5200
+F 0 "#PWR09" H 5650 4950 50  0001 C CNN
+F 1 "GND" H 5655 5027 50  0000 C CNN
+F 2 "" H 5650 5200 50  0001 C CNN
+F 3 "" H 5650 5200 50  0001 C CNN
+	1    5650 5200
+	1    0    0    -1
+$EndComp
+Wire Wire Line
+	5650 5100 5650 5200
+Text HLabel 5850 4750 2    39   Input ~ 0
+VOFS
+Wire Wire Line
+	5650 4750 5850 4750
+Connection ~ 5650 4750
 $EndSCHEMATC

Commit message: update parts
Parts:
- C10: footprint (none) -> Capacitor_SMD:C_0603_1608Metric; LCSC (none) -> C14663; manf_num (none) -> CC0603KRX7R9BB104
- C2, C3: LCSC (none) -> C106243; manf_num (none) -> CC0805KKX7R0BB104
- C311: value 100nF/100V -> 2,2μF/50V; LCSC (none) -> C348735; manf_num (none) -> UMK212BB7225KG-T
- C312: value 2,2μF/50V -> 100nF/100V; LCSC (none) -> C106243; manf_num (none) -> CC0805KKX7R0BB104
- C313: LCSC (none) -> C348735; manf_num (none) -> UMK212BB7225KG-T
- C315: LCSC (none) -> C14663; manf_num (none) -> CC0603KRX7R9BB104
- C4, C5, C6: LCSC (none) -> C519409; alt (none) -> CC0603JRX7R7BB471; manf_num (none) -> CC0603KRX7R7BB471
- C7, C8, C9: LCSC (none) -> C92775; manf_num   (none) -> HMK325B7225KN-T
- R1, R11, R13, R3, R4, R6: LCSC (none) -> C112307; manf_num (none) -> RC0603FR-072R2L
- R10, R14, R15, R7, R8, R9: LCSC (none) -> C2688862; manf_num (none) -> BVS-I-R003-1.0
- R12, R2, R5: LCSC (none) -> C138286; manf_num (none) -> AC0603FR-0710RL
