File: opm-inline/source/Motor Driver.sch (KiCad schematic (older format))
At the start: 38 parts, among them IC1 TMC6200-TA, Q1 YJG95G06A, Q2 YJG95G06A, Q3 YJG95G06A, Q4 YJG95G06A, Q5 YJG95G06A, Q6 YJG95G06A

Commit message: add more lssc basic parts
Parts:
- C311, C313: LCSC C348735 -> C49217; alt (none) -> UMK212BB7225KG-T; manf_num UMK212BB7225KG-T -> 0805F225M500NT
- R1, R11, R13, R3, R6: LCSC C112307 -> C22977; alt (none) -> RC0603FR-072R2L; manf_num RC0603FR-072R2L -> 0603WAF200KT5E
- R12, R2, R5: LCSC C138286 -> C22859; alt (none) -> AC0603FR-0710RL; manf_num AC0603FR-0710RL -> 0603WAF100JT5E
- R311, R314: LCSC (none) -> C21189; alt (none) -> RC0603FR-070RL; manf_num (none) -> 0603WAF0000T5E
- R4: Field6 (none) -> RC0603FR-072R2L; LCSC C112307 -> C22977; manf_num RC0603FR-072R2L -> 0603WAF200KT5E
Changed lines of the file:
@@
 F 1 "0Ω" V 3450 4100 39  0000 C CNN
 F 2 "Resistor_SMD:R_0603_1608Metric" V 3280 4100 39  0001 C CNN
-F 3 "~" H 3350 4100 39  0001 C CNN
+F 3 "https://datasheet.lcsc.com/lcsc/2110252030_UNI-ROYAL-Uniroyal-Elec-0603WAF0000T5E_C21189.pdf" H 3350 4100 39  0001 C CNN
+F 4 "C21189" V 3350 4100 50  0001 C CNN "LCSC"
+F 5 "0603WAF0000T5E" V 3350 4100 50  0001 C CNN "manf_num"
+F 6 "RC0603FR-070RL" V 3350 4100 50  0001 C CNN "alt"
 	1    3350 4100
 	1    0    0    -1
@@
 F 1 "0Ω" V 1850 3650 39  0000 C CNN
 F 2 "Resistor_SMD:R_0603_1608Metric" V 1680 3650 39  0001 C CNN
-F 3 "~" H 1750 3650 39  0001 C CNN
+F 3 "https://datasheet.lcsc.com/lcsc/2110252030_UNI-ROYAL-Uniroyal-Elec-0603WAF0000T5E_C21189.pdf" H 1750 3650 39  0001 C CNN
+F 4 "C21189" V 1750 3650 50  0001 C CNN "LCSC"
+F 5 "0603WAF0000T5E" V 1750 3650 50  0001 C CNN "manf_num"
+F 6 "RC0603FR-070RL" V 1750 3650 50  0001 C CNN "alt"
 	1    1750 3650
 	0    1    1    0
@@
 F 1 "2,2μF/50V" V 2200 4050 39  0000 C CNN
 F 2 "Capacitor_SMD:C_0805_2012Metric" H 2088 3900 39  0001 C CNN
-F 3 "https://www.mouser.fi/datasheet/2/396/mlcc02_e-1307760.pdf" H 2050 4050 39  0001 C CNN
-F 4 "C348735" V 2050 4050 50  0001 C CNN "LCSC"
-F 5 "UMK212BB7225KG-T" V 2050 4050 50  0001 C CNN "manf_num"
+F 3 "https://datasheet.lcsc.com/lcsc/1811101411_FH-Guangdong-Fenghua-Advanced-Tech-0805F225M500NT_C49217.pdf" H 2050 4050 39  0001 C CNN
+F 4 "C49217" V 2050 4050 50  0001 C CNN "LCSC"
+F 5 "0805F225M500NT" V 2050 4050 50  0001 C CNN "manf_num"
+F 6 "UMK212BB7225KG-T" V 2050 4050 50  0001 C CNN "alt"
 	1    2050 4050
 	1    0    0    -1
@@
 F 1 "2,2μF/50V" V 3100 4050 39  0000 C CNN
 F 2 "Capacitor_SMD:C_0805_2012Metric" H 2988 3900 39  0001 C CNN
-F 3 "https://www.mouser.fi/datasheet/2/396/mlcc02_e-1307760.pdf" H 2950 4050 39  0001 C CNN
-F 4 "C348735" V 2950 4050 50  0001 C CNN "LCSC"
-F 5 "UMK212BB7225KG-T" V 2950 4050 50  0001 C CNN "manf_num"
+F 3 "https://datasheet.lcsc.com/lcsc/1811101411_FH-Guangdong-Fenghua-Advanced-Tech-0805F225M500NT_C49217.pdf" H 2950 4050 39  0001 C CNN
+F 4 "C49217" V 2950 4050 50  0001 C CNN "LCSC"
+F 5 "0805F225M500NT" V 2950 4050 50  0001 C CNN "manf_num"
+F 6 "UMK212BB7225KG-T" V 2950 4050 50  0001 C CNN "alt"
 	1    2950 4050
 	1    0    0    -1
@@
 F 1 "2R2/1%" V 6945 5150 35  0000 C CNN
 F 2 "Resistor_SMD:R_0603_1608Metric" V 6980 5150 50  0001 C CNN
-F 3 "https://www.mouser.fi/datasheet/2/447/Yageo_03_18_2021_PYu_RC_Group_51_RoHS_L_11-2199992.pdf" H 7050 5150 50  0001 C CNN
-F 4 "C112307" V 7050 5150 50  0001 C CNN "LCSC"
-F 5 "RC0603FR-072R2L" V 7050 5150 50  0001 C CNN "manf_num"
+F 3 "https://datasheet.lcsc.com/lcsc/2110252130_UNI-ROYAL-Uniroyal-Elec-0603WAF200KT5E_C22977.pdf" H 7050 5150 50  0001 C CNN
+F 4 "C22977" V 7050 5150 50  0001 C CNN "LCSC"
+F 5 "0603WAF200KT5E" V 7050 5150 50  0001 C CNN "manf_num"
+F 6 "RC0603FR-072R2L" V 7050 5150 50  0001 C CNN "Field6"
 	1    7050 5150
 	0    1    1    0
@@
 F 1 "10R/1%" V 6945 5550 35  0000 C CNN
 F 2 "Resistor_SMD:R_0603_1608Metric" V 6980 5550 50  0001 C CNN
-F 3 "https://www.mouser.fi/datasheet/2/447/Yageo_03_18_2021_PYu_RC_Group_51_RoHS_L_11-2199992.pdf" H 7050 5550 50  0001 C CNN
-F 4 "C138286" V 7050 5550 50  0001 C CNN "LCSC"
-F 5 "AC0603FR-0710RL" V 7050 5550 50  0001 C CNN "manf_num"
+F 3 "https://datasheet.lcsc.com/lcsc/2110252030_UNI-ROYAL-Uniroyal-Elec-0603WAF100JT5E_C22859.pdf" H 7050 5550 50  0001 C CNN
+F 4 "C22859" V 7050 5550 50  0001 C CNN "LCSC"
+F 5 "0603WAF100JT5E" V 7050 5550 50  0001 C CNN "manf_num"
+F 6 "AC0603FR-0710RL" V 7050 5550 50  0001 C CNN "alt"
 	1    7050 5550
 	0    1    1    0
@@
 F 1 "2R2/1%" V 6945 5950 35  0000 C CNN
 F 2 "Resistor_SMD:R_0603_1608Metric" V 6980 5950 50  0001 C CNN
-F 3 "https://www.mouser.fi/datasheet/2/447/Yageo_03_18_2021_PYu_RC_Group_51_RoHS_L_11-2199992.pdf" H 7050 5950 50  0001 C CNN
-F 4 "C112307" V 7050 5950 50  0001 C CNN "LCSC"
-F 5 "RC0603FR-072R2L" V 7050 5950 50  0001 C CNN "manf_num"
+F 3 "https://datasheet.lcsc.com/lcsc/2110252130_UNI-ROYAL-Uniroyal-Elec-0603WAF200KT5E_C22977.pdf" H 7050 5950 50  0001 C CNN
+F 4 "C22977" V 7050 5950 50  0001 C CNN "LCSC"
+F 5 "0603WAF200KT5E" V 7050 5950 50  0001 C CNN "manf_num"
+F 6 "RC0603FR-072R2L" V 7050 5950 50  0001 C CNN "alt"
 	1    7050 5950
 	0    1    1    0
@@
 F 1 "2R2/1%" V 8595 3650 35  0000 C CNN
 F 2 "Resistor_SMD:R_0603_1608Metric" V 8630 3650 50  0001 C CNN
-F 3 "https://www.mouser.fi/datasheet/2/447/Yageo_03_18_2021_PYu_RC_Group_51_RoHS_L_11-2199992.pdf" H 8700 3650 50  0001 C CNN
-F 4 "C112307" V 8700 3650 50  0001 C CNN "LCSC"
-F 5 "RC0603FR-072R2L" V 8700 3650 50  0001 C CNN "manf_num"
+F 3 "https://datasheet.lcsc.com/lcsc/2110252130_UNI-ROYAL-Uniroyal-Elec-0603WAF200KT5E_C22977.pdf" H 8700 3650 50  0001 C CNN
+F 4 "C22977" V 8700 3650 50  0001 C CNN "LCSC"
+F 5 "0603WAF200KT5E" V 8700 3650 50  0001 C CNN "manf_num"
+F 6 "RC0603FR-072R2L" V 8700 3650 50  0001 C CNN "alt"
 	1    8700 3650
 	0    1    1    0
@@
 F 1 "10R/1%" V 8595 4050 35  0000 C CNN
 F 2 "Resistor_SMD:R_0603_1608Metric" V 8630 4050 50  0001 C CNN
-F 3 "https://www.mouser.fi/datasheet/2/447/Yageo_03_18_2021_PYu_RC_Group_51_RoHS_L_11-2199992.pdf" H 8700 4050 50  0001 C CNN
-F 4 "C138286" V 8700 4050 50  0001 C CNN "LCSC"
-F 5 "AC0603FR-0710RL" V 8700 4050 50  0001 C CNN "manf_num"
+F 3 "https://datasheet.lcsc.com/lcsc/2110252030_UNI-ROYAL-Uniroyal-Elec-0603WAF100JT5E_C22859.pdf" H 8700 4050 50  0001 C CNN
+F 4 "C22859" V 8700 4050 50  0001 C CNN "LCSC"
+F 5 "0603WAF100JT5E" V 8700 4050 50  0001 C CNN "manf_num"
+F 6 "AC0603FR-0710RL" V 8700 4050 50  0001 C CNN "alt"
 	1    8700 4050
 	0    1    1    0
@@
 F 1 "2R2/1%" V 8595 4450 35  0000 C CNN
 F 2 "Resistor_SMD:R_0603_1608Metric" V 8630 4450 50  0001 C CNN
-F 3 "https://www.mouser.fi/datasheet/2/447/Yageo_03_18_2021_PYu_RC_Group_51_RoHS_L_11-2199992.pdf" H 8700 4450 50  0001 C CNN
-F 4 "C112307" V 8700 4450 50  0001 C CNN "LCSC"
-F 5 "RC0603FR-072R2L" V 8700 4450 50  0001 C CNN "manf_num"
+F 3 "https://datasheet.lcsc.com/lcsc/2110252130_UNI-ROYAL-Uniroyal-Elec-0603WAF200KT5E_C22977.pdf" H 8700 4450 50  0001 C CNN
+F 4 "C22977" V 8700 4450 50  0001 C CNN "LCSC"
+F 5 "0603WAF200KT5E" V 8700 4450 50  0001 C CNN "manf_num"
+F 6 "RC0603FR-072R2L" V 8700 4450 50  0001 C CNN "alt"
 	1    8700 4450
 	0    1    1    0
@@
 F 1 "2R2/1%" V 6945 2350 35  0000 C CNN
 F 2 "Resistor_SMD:R_0603_1608Metric" V 6980 2350 50  0001 C CNN
-F 3 "https://www.mouser.fi/datasheet/2/447/Yageo_03_18_2021_PYu_RC_Group_51_RoHS_L_11-2199992.pdf" H 7050 2350 50  0001 C CNN
-F 4 "C112307" V 7050 2350 50  0001 C CNN "LCSC"
-F 5 "RC0603FR-072R2L" V 7050 2350 50  0001 C CNN "manf_num"
+F 3 "https://datasheet.lcsc.com/lcsc/2110252130_UNI-ROYAL-Uniroyal-Elec-0603WAF200KT5E_C22977.pdf" H 7050 2350 50  0001 C CNN
+F 4 "C22977" V 7050 2350 50  0001 C CNN "LCSC"
+F 5 "0603WAF200KT5E" V 7050 2350 50  0001 C CNN "manf_num"
+F 6 "RC0603FR-072R2L" V 7050 2350 50  0001 C CNN "alt"
 	1    7050 2350
 	0    1    1    0
@@
 F 1 "10R/1%" V 6945 2750 35  0000 C CNN
 F 2 "Resistor_SMD:R_0603_1608Metric" V 6980 2750 50  0001 C CNN
-F 3 "https://www.mouser.fi/datasheet/2/447/Yageo_03_18_2021_PYu_RC_Group_51_RoHS_L_11-2199992.pdf" H 7050 2750 50  0001 C CNN
-F 4 "C138286" V 7050 2750 50  0001 C CNN "LCSC"
-F 5 "AC0603FR-0710RL" V 7050 2750 50  0001 C CNN "manf_num"
+F 3 "https://datasheet.lcsc.com/lcsc/2110252030_UNI-ROYAL-Uniroyal-Elec-0603WAF100JT5E_C22859.pdf" H 7050 2750 50  0001 C CNN
+F 4 "C22859" V 7050 2750 50  0001 C CNN "LCSC"
+F 5 "0603WAF100JT5E" V 7050 2750 50  0001 C CNN "manf_num"
+F 6 "AC0603FR-0710RL" V 7050 2750 50  0001 C CNN "alt"
 	1    7050 2750
 	0    1    1    0
@@
 F 1 "2R2/1%" V 6945 3150 35  0000 C CNN
 F 2 "Resistor_SMD:R_0603_1608Metric" V 6980 3150 50  0001 C CNN
-F 3 "https://www.mouser.fi/datasheet/2/447/Yageo_03_18_2021_PYu_RC_Group_51_RoHS_L_11-2199992.pdf" H 7050 3150 50  0001 C CNN
-F 4 "C112307" V 7050 3150 50  0001 C CNN "LCSC"
-F 5 "RC0603FR-072R2L" V 7050 3150 50  0001 C CNN "manf_num"
+F 3 "https://datasheet.lcsc.com/lcsc/2110252130_UNI-ROYAL-Uniroyal-Elec-0603WAF200KT5E_C22977.pdf" H 7050 3150 50  0001 C CNN
+F 4 "C22977" V 7050 3150 50  0001 C CNN "LCSC"
+F 5 "0603WAF200KT5E" V 7050 3150 50  0001 C CNN "manf_num"
+F 6 "RC0603FR-072R2L" V 7050 3150 50  0001 C CNN "alt"
 	1    7050 3150
 	0    1    1    0

Commit message: update libs
Parts:
- C1: LCSC (none) -> C313105; manf_num (none) -> CC0603KRX7R0BB223
Connections:
- wire segments 152 -> 154
Changed lines of the file:
@@
 F 1 "22nF/100V" V 4811 3200 35  0000 C CNN
 F 2 "Capacitor_SMD:C_0603_1608Metric" H 4688 3050 50  0001 C CNN
-F 3 "~" H 4650 3200 50  0001 C CNN
+F 3 "https://datasheet.lcsc.com/lcsc/1811082033_YAGEO-CC0603KRX7R0BB223_C313105.pdf" H 4650 3200 50  0001 C CNN
+F 4 "C313105" V 4650 3200 50  0001 C CNN "LCSC"
+F 5 "CC0603KRX7R0BB223" V 4650 3200 50  0001 C CNN "manf_num"
 	1    4650 3200
 	0    -1   -1   0
@@
 F 1 "0R033/1%/2W" V 8645 2900 35  0000 C CNN
 F 2 "Resistor_SMD:R_0603_1608Metric" V 8680 2900 50  0001 C CNN
-F 3 "~" H 8750 2900 50  0001 C CNN
+F 3 "https://www.isabellenhuette.de/fileadmin/Daten/Praezisionswiderstaende/Datenblaetter/BVT.PDF" H 8750 2900 50  0001 C CNN
 F 4 "C2688862" V 8750 2900 50  0001 C CNN "LCSC"
 F 5 "BVS-I-R003-1.0" V 8750 2900 50  0001 C CNN "manf_num"
@@
 	5650 4750 5850 4750
 Connection ~ 5650 4750
+Wire Wire Line
+	5050 3400 5200 3400
+Wire Wire Line
+	5200 3400 5200 3200
+Connection ~ 5200 3200
 $EndSCHEMATC

Commit message: cleanup
Parts:
- R10, R14, R15, R7, R8, R9: LCSC C2688862 -> C2838960; manf_num BVS-I-R003-1.0 -> LMP25NF2P0R033
Changed lines of the file:
@@
 AR Path="/61C4FD8F" Ref="Q4"  Part="1"
 AR Path="/5D5FDD98/61C4FD8F" Ref="Q4"  Part="1"
-F 0 "Q4" H 8031 5988 39  0000 L CNN
-F 1 "YJG95G06A" H 8031 5913 39  0000 L CNN
+F 0 "Q4" V 8031 5988 39  0000 R BNN
+F 1 "YJG95G06A" V 8031 5913 39  0000 C TNN
 F 2 "Package_TO_SOT_SMD:TDSON-8-1" H 7900 5875 39  0001 L CIN
 F 3 "" V 7700 5950 50  0001 L CNN
@@
 F 1 "0R033/1%/2W" V 8645 5400 35  0000 C CNN
 F 2 "Resistor_SMD:R_0603_1608Metric" V 8680 5400 50  0001 C CNN
-F 3 "https://www.isabellenhuette.de/fileadmin/Daten/Praezisionswiderstaende/Datenblaetter/BVT.PDF" H 8750 5400 50  0001 C CNN
-F 4 "C2688862" V 8750 5400 50  0001 C CNN "LCSC"
-F 5 "BVS-I-R003-1.0" V 8750 5400 50  0001 C CNN "manf_num"
+F 3 "https://datasheet.lcsc.com/lcsc/2108141930_prosemi-LMP25NF2P0R033_C2838960.pdf" H 8750 5400 50  0001 C CNN
+F 4 "C2838960" V 8750 5400 50  0001 C CNN "LCSC"
+F 5 "LMP25NF2P0R033" V 8750 5400 50  0001 C CNN "manf_num"
 	1    8750 5400
 	0    1    1    0
@@
 F 1 "0R033/1%/2W" V 8645 5700 35  0000 C CNN
 F 2 "Resistor_SMD:R_0603_1608Metric" V 8680 5700 50  0001 C CNN
-F 3 "https://www.isabellenhuette.de/fileadmin/Daten/Praezisionswiderstaende/Datenblaetter/BVT.PDF" H 8750 5700 50  0001 C CNN
-F 4 "C2688862" V 8750 5700 50  0001 C CNN "LCSC"
-F 5 "BVS-I-R003-1.0" V 8750 5700 50  0001 C CNN "manf_num"
+F 3 "https://datasheet.lcsc.com/lcsc/2108141930_prosemi-LMP25NF2P0R033_C2838960.pdf" H 8750 5700 50  0001 C CNN
+F 4 "C2838960" V 8750 5700 50  0001 C CNN "LCSC"
+F 5 "LMP25NF2P0R033" V 8750 5700 50  0001 C CNN "manf_num"
 	1    8750 5700
 	0    1    1    0
@@
 AR Path="/61D8AF0A" Ref="Q6"  Part="1"
 AR Path="/5D5FDD98/61D8AF0A" Ref="Q6"  Part="1"
-F 0 "Q6" H 9681 4488 39  0000 L CNN
-F 1 "YJG95G06A" H 9681 4413 39  0000 L CNN
+F 0 "Q6" V 9681 4488 39  0000 R BNN
+F 1 "YJG95G06A" V 9681 4413 39  0000 C TNN
 F 2 "Package_TO_SOT_SMD:TDSON-8-1" H 9550 4375 39  0001 L CIN
 F 3 "" V 9350 4450 50  0001 L CNN
@@
 F 1 "0R033/1%/2W" V 10295 3900 35  0000 C CNN
 F 2 "Resistor_SMD:R_0603_1608Metric" V 10330 3900 50  0001 C CNN
-F 3 "https://www.isabellenhuette.de/fileadmin/Daten/Praezisionswiderstaende/Datenblaetter/BVT.PDF" H 10400 3900 50  0001 C CNN
-F 4 "C2688862" V 10400 3900 50  0001 C CNN "LCSC"
-F 5 "BVS-I-R003-1.0" V 10400 3900 50  0001 C CNN "manf_num"
+F 3 "https://datasheet.lcsc.com/lcsc/2108141930_prosemi-LMP25NF2P0R033_C2838960.pdf" H 10400 3900 50  0001 C CNN
+F 4 "C2838960" V 10400 3900 50  0001 C CNN "LCSC"
+F 5 "LMP25NF2P0R033" V 10400 3900 50  0001 C CNN "manf_num"
 	1    10400 3900
 	0    1    1    0
@@
 F 1 "0R033/1%/2W" V 10295 4200 35  0000 C CNN
 F 2 "Resistor_SMD:R_0603_1608Metric" V 10330 4200 50  0001 C CNN
-F 3 "https://www.isabellenhuette.de/fileadmin/Daten/Praezisionswiderstaende/Datenblaetter/BVT.PDF" H 10400 4200 50  0001 C CNN
-F 4 "C2688862" V 10400 4200 50  0001 C CNN "LCSC"
-F 5 "BVS-I-R003-1.0" V 10400 4200 50  0001 C CNN "manf_num"
+F 3 "https://datasheet.lcsc.com/lcsc/2108141930_prosemi-LMP25NF2P0R033_C2838960.pdf" H 10400 4200 50  0001 C CNN
+F 4 "C2838960" V 10400 4200 50  0001 C CNN "LCSC"
+F 5 "LMP25NF2P0R033" V 10400 4200 50  0001 C CNN "manf_num"
 	1    10400 4200
 	0    1    1    0
@@
 AR Path="/61D9B6B4" Ref="Q2"  Part="1"
 AR Path="/5D5FDD98/61D9B6B4" Ref="Q2"  Part="1"
-F 0 "Q2" H 8031 3188 39  0000 L CNN
-F 1 "YJG95G06A" H 8031 3113 39  0000 L CNN
+F 0 "Q2" V 8031 3188 39  0000 R BNN
+F 1 "YJG95G06A" V 8031 3113 39  0000 C TNN
 F 2 "Package_TO_SOT_SMD:TDSON-8-1" H 7900 3075 39  0001 L CIN
 F 3 "" V 7700 3150 50  0001 L CNN
@@
 F 1 "0R033/1%/2W" V 8645 2600 35  0000 C CNN
 F 2 "Resistor_SMD:R_0603_1608Metric" V 8680 2600 50  0001 C CNN
-F 3 "https://www.isabellenhuette.de/fileadmin/Daten/Praezisionswiderstaende/Datenblaetter/BVT.PDF" H 8750 2600 50  0001 C CNN
-F 4 "C2688862" V 8750 2600 50  0001 C CNN "LCSC"
-F 5 "BVS-I-R003-1.0" V 8750 2600 50  0001 C CNN "manf_num"
+F 3 "https://datasheet.lcsc.com/lcsc/2108141930_prosemi-LMP25NF2P0R033_C2838960.pdf" H 8750 2600 50  0001 C CNN
+F 4 "C2838960" V 8750 2600 50  0001 C CNN "LCSC"
+F 5 "LMP25NF2P0R033" V 8750 2600 50  0001 C CNN "manf_num"
 	1    8750 2600
 	0    1    1    0
@@
 F 1 "0R033/1%/2W" V 8645 2900 35  0000 C CNN
 F 2 "Resistor_SMD:R_0603_1608Metric" V 8680 2900 50  0001 C CNN
-F 3 "https://www.isabellenhuette.de/fileadmin/Daten/Praezisionswiderstaende/Datenblaetter/BVT.PDF" H 8750 2900 50  0001 C CNN
-F 4 "C2688862" V 8750 2900 50  0001 C CNN "LCSC"
-F 5 "BVS-I-R003-1.0" V 8750 2900 50  0001 C CNN "manf_num"
+F 3 "https://datasheet.lcsc.com/lcsc/2108141930_prosemi-LMP25NF2P0R033_C2838960.pdf" H 8750 2900 50  0001 C CNN
+F 4 "C2838960" V 8750 2900 50  0001 C CNN "LCSC"
+F 5 "LMP25NF2P0R033" V 8750 2900 50  0001 C CNN "manf_num"
 	1    8750 2900
 	0    1    1    0
