File: opm-inline/source/Motor Driver.sch (KiCad schematic (older format))
At the start: 38 parts, among them IC1 TMC6200-TA, Q1 YJG95G06A, Q2 YJG95G06A, Q3 YJG95G06A, Q4 YJG95G06A, Q5 YJG95G06A, Q6 YJG95G06A

Commit message: more layout work
Parts:
- R10, R14, R15, R7, R8, R9: value 0R033/1%/2W -> 0R005/1%/1W; footprint Resistor_SMD:R_2512_6332Metric -> Resistor_SMD:R_1206_3216Metric; LCSC C2838960 -> C2692048; manf_num LMP25NF2P0R033 -> SME12ABFR005T
Changed lines of the file:
@@
 P 8750 5400
 F 0 "R9" V 8576 5400 35  0000 C CNN
-F 1 "0R033/1%/2W" V 8645 5400 35  0000 C CNN
-F 2 "Resistor_SMD:R_2512_6332Metric" V 8680 5400 50  0001 C CNN
-F 3 "https://datasheet.lcsc.com/lcsc/2108141930_prosemi-LMP25NF2P0R033_C2838960.pdf" H 8750 5400 50  0001 C CNN
-F 4 "C2838960" V 8750 5400 50  0001 C CNN "LCSC"
-F 5 "LMP25NF2P0R033" V 8750 5400 50  0001 C CNN "manf_num"
+F 1 "0R005/1%/1W" V 8645 5400 35  0000 C CNN
+F 2 "Resistor_SMD:R_1206_3216Metric" V 8680 5400 50  0001 C CNN
+F 3 "https://datasheet.lcsc.com/lcsc/2106062334_SART-Nanjing-Sart-Tech-SME12ABFR005T_C2692048.pdf" H 8750 5400 50  0001 C CNN
+F 4 "C2692048" V 8750 5400 50  0001 C CNN "LCSC"
+F 5 "SME12ABFR005T" V 8750 5400 50  0001 C CNN "manf_num"
 	1    8750 5400
 	0    1    1    0
@@
 P 8750 5700
 F 0 "R10" V 8576 5700 35  0000 C CNN
-F 1 "0R033/1%/2W" V 8645 5700 35  0000 C CNN
-F 2 "Resistor_SMD:R_2512_6332Metric" V 8680 5700 50  0001 C CNN
-F 3 "https://datasheet.lcsc.com/lcsc/2108141930_prosemi-LMP25NF2P0R033_C2838960.pdf" H 8750 5700 50  0001 C CNN
-F 4 "C2838960" V 8750 5700 50  0001 C CNN "LCSC"
-F 5 "LMP25NF2P0R033" V 8750 5700 50  0001 C CNN "manf_num"
+F 1 "0R005/1%/1W" V 8645 5700 35  0000 C CNN
+F 2 "Resistor_SMD:R_1206_3216Metric" V 8680 5700 50  0001 C CNN
+F 3 "https://datasheet.lcsc.com/lcsc/2106062334_SART-Nanjing-Sart-Tech-SME12ABFR005T_C2692048.pdf" H 8750 5700 50  0001 C CNN
+F 4 "C2692048" V 8750 5700 50  0001 C CNN "LCSC"
+F 5 "SME12ABFR005T" V 8750 5700 50  0001 C CNN "manf_num"
 	1    8750 5700
 	0    1    1    0
@@
 P 10400 3900
 F 0 "R14" V 10226 3900 35  0000 C CNN
-F 1 "0R033/1%/2W" V 10295 3900 35  0000 C CNN
-F 2 "Resistor_SMD:R_2512_6332Metric" V 10330 3900 50  0001 C CNN
-F 3 "https://datasheet.lcsc.com/lcsc/2108141930_prosemi-LMP25NF2P0R033_C2838960.pdf" H 10400 3900 50  0001 C CNN
-F 4 "C2838960" V 10400 3900 50  0001 C CNN "LCSC"
-F 5 "LMP25NF2P0R033" V 10400 3900 50  0001 C CNN "manf_num"
+F 1 "0R005/1%/1W" V 10295 3900 35  0000 C CNN
+F 2 "Resistor_SMD:R_1206_3216Metric" V 10330 3900 50  0001 C CNN
+F 3 "https://datasheet.lcsc.com/lcsc/2106062334_SART-Nanjing-Sart-Tech-SME12ABFR005T_C2692048.pdf" H 10400 3900 50  0001 C CNN
+F 4 "C2692048" V 10400 3900 50  0001 C CNN "LCSC"
+F 5 "SME12ABFR005T" V 10400 3900 50  0001 C CNN "manf_num"
 	1    10400 3900
 	0    1    1    0
@@
 P 10400 4200
 F 0 "R15" V 10226 4200 35  0000 C CNN
-F 1 "0R033/1%/2W" V 10295 4200 35  0000 C CNN
-F 2 "Resistor_SMD:R_2512_6332Metric" V 10330 4200 50  0001 C CNN
-F 3 "https://datasheet.lcsc.com/lcsc/2108141930_prosemi-LMP25NF2P0R033_C2838960.pdf" H 10400 4200 50  0001 C CNN
-F 4 "C2838960" V 10400 4200 50  0001 C CNN "LCSC"
-F 5 "LMP25NF2P0R033" V 10400 4200 50  0001 C CNN "manf_num"
+F 1 "0R005/1%/1W" V 10295 4200 35  0000 C CNN
+F 2 "Resistor_SMD:R_1206_3216Metric" V 10330 4200 50  0001 C CNN
+F 3 "https://datasheet.lcsc.com/lcsc/2106062334_SART-Nanjing-Sart-Tech-SME12ABFR005T_C2692048.pdf" H 10400 4200 50  0001 C CNN
+F 4 "C2692048" V 10400 4200 50  0001 C CNN "LCSC"
+F 5 "SME12ABFR005T" V 10400 4200 50  0001 C CNN "manf_num"
 	1    10400 4200
 	0    1    1    0
@@
 P 8750 2600
 F 0 "R7" V 8576 2600 35  0000 C CNN
-F 1 "0R033/1%/2W" V 8645 2600 35  0000 C CNN
-F 2 "Resistor_SMD:R_2512_6332Metric" V 8680 2600 50  0001 C CNN
-F 3 "https://datasheet.lcsc.com/lcsc/2108141930_prosemi-LMP25NF2P0R033_C2838960.pdf" H 8750 2600 50  0001 C CNN
-F 4 "C2838960" V 8750 2600 50  0001 C CNN "LCSC"
-F 5 "LMP25NF2P0R033" V 8750 2600 50  0001 C CNN "manf_num"
+F 1 "0R005/1%/1W" V 8645 2600 35  0000 C CNN
+F 2 "Resistor_SMD:R_1206_3216Metric" V 8680 2600 50  0001 C CNN
+F 3 "https://datasheet.lcsc.com/lcsc/2106062334_SART-Nanjing-Sart-Tech-SME12ABFR005T_C2692048.pdf" H 8750 2600 50  0001 C CNN
+F 4 "C2692048" V 8750 2600 50  0001 C CNN "LCSC"
+F 5 "SME12ABFR005T" V 8750 2600 50  0001 C CNN "manf_num"
 	1    8750 2600
 	0    1    1    0
@@
 P 8750 2900
 F 0 "R8" V 8576 2900 35  0000 C CNN
-F 1 "0R033/1%/2W" V 8645 2900 35  0000 C CNN
-F 2 "Resistor_SMD:R_2512_6332Metric" V 8680 2900 50  0001 C CNN
-F 3 "https://datasheet.lcsc.com/lcsc/2108141930_prosemi-LMP25NF2P0R033_C2838960.pdf" H 8750 2900 50  0001 C CNN
-F 4 "C2838960" V 8750 2900 50  0001 C CNN "LCSC"
-F 5 "LMP25NF2P0R033" V 8750 2900 50  0001 C CNN "manf_num"
+F 1 "0R005/1%/1W" V 8645 2900 35  0000 C CNN
+F 2 "Resistor_SMD:R_1206_3216Metric" V 8680 2900 50  0001 C CNN
+F 3 "https://datasheet.lcsc.com/lcsc/2106062334_SART-Nanjing-Sart-Tech-SME12ABFR005T_C2692048.pdf" H 8750 2900 50  0001 C CNN
+F 4 "C2692048" V 8750 2900 50  0001 C CNN "LCSC"
+F 5 "SME12ABFR005T" V 8750 2900 50  0001 C CNN "manf_num"
 	1    8750 2900
 	0    1    1    0

Commit message: some more layout
Parts:
- C7, C8, C9: footprint Capacitor_SMD:C_0603_1608Metric -> Capacitor_SMD:C_1210_3225Metric; LCSC C92775 -> C385982; manf_num   HMK325B7225KN-T -> HMK325B7225KMHP
Changed lines of the file:
@@
 F 0 "C8" H 8465 4985 35  0000 L CNN
 F 1 "2.2uF/100V" H 8465 4916 35  0000 L CNN
-F 2 "Capacitor_SMD:C_0603_1608Metric" H 8388 4800 50  0001 C CNN
-F 3 "https://www.mouser.fi/datasheet/2/396/mlcc02_e-1307760.pdf" H 8350 4950 50  0001 C CNN
-F 4 "C92775" H 8350 4950 50  0001 C CNN "LCSC"
-F 5 "HMK325B7225KN-T" H 8350 4950 50  0001 C CNN "manf_num  "
+F 2 "Capacitor_SMD:C_1210_3225Metric" H 8388 4800 50  0001 C CNN
+F 3 "https://datasheet.lcsc.com/lcsc/2010231635_Taiyo-Yuden-HMK325B7225KMHP_C385982.pdf" H 8350 4950 50  0001 C CNN
+F 4 "C385982" H 8350 4950 50  0001 C CNN "LCSC"
+F 5 "HMK325B7225KMHP" H 8350 4950 50  0001 C CNN "manf_num  "
 	1    8350 4950
 	1    0    0    -1
@@
 F 0 "C9" H 10115 3485 35  0000 L CNN
 F 1 "2.2uF/100V" H 10115 3416 35  0000 L CNN
-F 2 "Capacitor_SMD:C_0603_1608Metric" H 10038 3300 50  0001 C CNN
-F 3 "https://www.mouser.fi/datasheet/2/396/mlcc02_e-1307760.pdf" H 10000 3450 50  0001 C CNN
-F 4 "C92775" H 10000 3450 50  0001 C CNN "LCSC"
-F 5 "HMK325B7225KN-T" H 10000 3450 50  0001 C CNN "manf_num  "
+F 2 "Capacitor_SMD:C_1210_3225Metric" H 10038 3300 50  0001 C CNN
+F 3 "https://datasheet.lcsc.com/lcsc/2010231635_Taiyo-Yuden-HMK325B7225KMHP_C385982.pdf" H 10000 3450 50  0001 C CNN
+F 4 "C385982" H 10000 3450 50  0001 C CNN "LCSC"
+F 5 "HMK325B7225KMHP" H 10000 3450 50  0001 C CNN "manf_num  "
 	1    10000 3450
 	1    0    0    -1
@@
 F 0 "C7" H 8465 2185 35  0000 L CNN
 F 1 "2.2uF/100V" H 8465 2116 35  0000 L CNN
-F 2 "Capacitor_SMD:C_0603_1608Metric" H 8388 2000 50  0001 C CNN
-F 3 "https://www.mouser.fi/datasheet/2/396/mlcc02_e-1307760.pdf" H 8350 2150 50  0001 C CNN
-F 4 "C92775" H 8350 2150 50  0001 C CNN "LCSC"
-F 5 "HMK325B7225KN-T" H 8350 2150 50  0001 C CNN "manf_num  "
+F 2 "Capacitor_SMD:C_1210_3225Metric" H 8388 2000 50  0001 C CNN
+F 3 "https://datasheet.lcsc.com/lcsc/2010231635_Taiyo-Yuden-HMK325B7225KMHP_C385982.pdf" H 8350 2150 50  0001 C CNN
+F 4 "C385982" H 8350 2150 50  0001 C CNN "LCSC"
+F 5 "HMK325B7225KMHP" H 8350 2150 50  0001 C CNN "manf_num  "
 	1    8350 2150
 	1    0    0    -1

Commit message: more layout
Parts:
- removed Q1, Q2, Q3, Q4, Q5, Q6: YJG95G06A, Libraries:PDFN-8, symbol opm-inline-rescue:opm-inline-rescue_YJG95G06A-Transistor_FET-opm-v1.1-rescue-op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
- added Q1, Q2, Q3, Q4, Q5, Q6: HYG025N06LS1C2, Libraries:PDFN-8, symbol opm-inline-rescue:HYG025N06LS1C2
- C13, C19: value 2,2μF/50V -> 2,2uF/50V
- IC1: JLCPCB BOM (none) -> No
- R1, R11, R13, R3, R4, R6: value 22Ω/1% -> 22R/1%
- R26: value 0Ω -> 0R
Connections:
- wire segments 154 -> 149
Other:
- moved on the sheet: C1, C10, C13, C18, C19, C2, C20, C3, C4, C5, C6, C7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

Commit message: update from latest
Parts:
- Q5: footprint Libraries:PDFN-8 -> Package_DFN_QFN:DFN-8-1EP_6x5mm_P1.27mm_EP4x4mm
Changed lines of the file:
@@
 F 0 "Q5" H 9000 3138 39  0000 L CNN
 F 1 "HYG025N06LS1C2" H 9000 3063 39  0000 L CNN
-F 2 "Libraries:PDFN-8" H 8900 3100 39  0001 L CIN
+F 2 "Package_DFN_QFN:DFN-8-1EP_6x5mm_P1.27mm_EP4x4mm" H 8900 3100 39  0001 L CIN
 F 3 "https://datasheet.lcsc.com/lcsc/2105242011_HUAYI-HYG025N06LS1C2_C2827231.pdf" V 8700 3100 50  0001 L CNN
 F 4 "C2827231" H 8800 3100 50  0001 C CNN "LCSC"
