File: opm-inline/source/Motor Driver.sch (KiCad schematic (older format))
At the start: 38 parts, among them IC1 TMC6200-TA, Q1 HYG025N06LS1C2, Q2 HYG025N06LS1C2, Q3 HYG025N06LS1C2, Q4 HYG025N06LS1C2, Q5 HYG025N06LS1C2, Q6 HYG025N06LS1C2

Commit message: fix some parts
Parts:
- C4: value 470nF -> 470nF/16V
- Q5: footprint Package_DFN_QFN:DFN-8-1EP_6x5mm_P1.27mm_EP4x4mm -> Libraries:PDFN-8
Changed lines of the file:
@@
 P 5000 2850
 F 0 "C4" V 4781 2850 35  0000 C CNN
-F 1 "470nF" V 4850 2850 35  0000 C CNN
+F 1 "470nF/16V" V 4850 2850 35  0000 C CNN
 F 2 "Capacitor_SMD:C_0603_1608Metric" H 5038 2700 50  0001 C CNN
 F 3 "https://www.mouser.fi/datasheet/2/447/yago_s_a0011723860_1-2286802.pdf" H 5000 2850 50  0001 C CNN
@@
 F 0 "Q5" H 9000 3138 39  0000 L CNN
 F 1 "HYG025N06LS1C2" H 9000 3063 39  0000 L CNN
-F 2 "Package_DFN_QFN:DFN-8-1EP_6x5mm_P1.27mm_EP4x4mm" H 8900 3100 39  0001 L CIN
+F 2 "Libraries:PDFN-8" H 8900 3100 39  0001 L CIN
 F 3 "https://datasheet.lcsc.com/lcsc/2105242011_HUAYI-HYG025N06LS1C2_C2827231.pdf" V 8700 3100 50  0001 L CNN
 F 4 "C2827231" H 8800 3100 50  0001 C CNN "LCSC"
