File: opm-inline/source/MotorDriver.sch (KiCad schematic (older format))
At the start: 38 parts, among them IC1 TMC6200-TA, Q1 HYG025N06LS1C2, Q2 HYG025N06LS1C2, Q3 HYG025N06LS1C2, Q4 HYG025N06LS1C2, Q5 HYG025N06LS1C2, Q6 HYG025N06LS1C2

Commit message: heatsink
Parts:
- C13, C19: value 2,2uF/50V -> 2.2uF/50V
Changed lines of the file:
@@
 $Descr A4 11693 8268
 encoding utf-8
-Sheet 2 3
+Sheet 3 3
 Title "TMC6100-EVAL"
 Date "2019-10-28"
@@
 P 1400 3500
 F 0 "C13" V 1250 3500 39  0000 C CNN
-F 1 "2,2uF/50V" V 1550 3500 39  0000 C CNN
+F 1 "2.2uF/50V" V 1550 3500 39  0000 C CNN
 F 2 "Capacitor_SMD:C_0805_2012Metric" H 1438 3350 39  0001 C CNN
 F 3 "https://datasheet.lcsc.com/lcsc/1811101411_FH-Guangdong-Fenghua-Advanced-Tech-0805F225M500NT_C49217.pdf" H 1400 3500 39  0001 C CNN
@@
 P 2300 3500
 F 0 "C19" V 2150 3500 39  0000 C CNN
-F 1 "2,2uF/50V" V 2450 3500 39  0000 C CNN
+F 1 "2.2uF/50V" V 2450 3500 39  0000 C CNN
 F 2 "Capacitor_SMD:C_0805_2012Metric" H 2338 3350 39  0001 C CNN
 F 3 "https://datasheet.lcsc.com/lcsc/1811101411_FH-Guangdong-Fenghua-Advanced-Tech-0805F225M500NT_C49217.pdf" H 2300 3500 39  0001 C CNN

Commit message: update parts
Parts:
- C4, C5, C6: LCSC C519409 -> C106851; manf_num CC0603KRX7R7BB471 -> CC0603KRX7R7BB474
- C7, C8, C9: LCSC C385982 -> C412614; manf_num   HMK325B7225KMHP -> HMJ325AB7225KMHP
Changed lines of the file:
@@
 F 1 "2.2uF/100V" H 7815 4366 35  0000 L CNN
 F 2 "Capacitor_SMD:C_1210_3225Metric" H 7738 4250 50  0001 C CNN
-F 3 "https://datasheet.lcsc.com/lcsc/2010231635_Taiyo-Yuden-HMK325B7225KMHP_C385982.pdf" H 7700 4400 50  0001 C CNN
-F 4 "C385982" H 7700 4400 50  0001 C CNN "LCSC"
-F 5 "HMK325B7225KMHP" H 7700 4400 50  0001 C CNN "manf_num  "
+F 3 "https://datasheet.lcsc.com/lcsc/1912111437_Taiyo-Yuden-HMJ325AB7225KMHP_C412614.pdf" H 7700 4400 50  0001 C CNN
+F 4 "C412614" H 7700 4400 50  0001 C CNN "LCSC"
+F 5 "HMJ325AB7225KMHP" H 7700 4400 50  0001 C CNN "manf_num  "
 	1    7700 4400
 	1    0    0    -1
@@
 F 1 "470nF/16V" H 6065 4016 35  0000 L CNN
 F 2 "Capacitor_SMD:C_0603_1608Metric" H 5988 3900 50  0001 C CNN
-F 3 "https://www.mouser.fi/datasheet/2/447/yago_s_a0011723860_1-2286802.pdf" H 5950 4050 50  0001 C CNN
-F 4 "C519409" H 5950 4050 50  0001 C CNN "LCSC"
-F 5 "CC0603KRX7R7BB471" H 5950 4050 50  0001 C CNN "manf_num"
+F 3 "https://datasheet.lcsc.com/lcsc/1811082118_YAGEO-CC0603KRX7R7BB474_C106851.pdf" H 5950 4050 50  0001 C CNN
+F 4 "C106851" H 5950 4050 50  0001 C CNN "LCSC"
+F 5 "CC0603KRX7R7BB474" H 5950 4050 50  0001 C CNN "manf_num"
 F 6 "CC0603JRX7R7BB471" H 5950 4050 50  0001 C CNN "alt"
 	1    5950 4050
@@
 F 1 "2.2uF/100V" H 9465 2866 35  0000 L CNN
 F 2 "Capacitor_SMD:C_1210_3225Metric" H 9388 2750 50  0001 C CNN
-F 3 "https://datasheet.lcsc.com/lcsc/2010231635_Taiyo-Yuden-HMK325B7225KMHP_C385982.pdf" H 9350 2900 50  0001 C CNN
-F 4 "C385982" H 9350 2900 50  0001 C CNN "LCSC"
-F 5 "HMK325B7225KMHP" H 9350 2900 50  0001 C CNN "manf_num  "
+F 3 "https://datasheet.lcsc.com/lcsc/1912111437_Taiyo-Yuden-HMJ325AB7225KMHP_C412614.pdf" H 9350 2900 50  0001 C CNN
+F 4 "C412614" H 9350 2900 50  0001 C CNN "LCSC"
+F 5 "HMJ325AB7225KMHP" H 9350 2900 50  0001 C CNN "manf_num  "
 	1    9350 2900
 	1    0    0    -1
@@
 F 1 "2.2uF/100V" H 7815 1566 35  0000 L CNN
 F 2 "Capacitor_SMD:C_1210_3225Metric" H 7738 1450 50  0001 C CNN
-F 3 "https://datasheet.lcsc.com/lcsc/2010231635_Taiyo-Yuden-HMK325B7225KMHP_C385982.pdf" H 7700 1600 50  0001 C CNN
-F 4 "C385982" H 7700 1600 50  0001 C CNN "LCSC"
-F 5 "HMK325B7225KMHP" H 7700 1600 50  0001 C CNN "manf_num  "
+F 3 "https://datasheet.lcsc.com/lcsc/1912111437_Taiyo-Yuden-HMJ325AB7225KMHP_C412614.pdf" H 7700 1600 50  0001 C CNN
+F 4 "C412614" H 7700 1600 50  0001 C CNN "LCSC"
+F 5 "HMJ325AB7225KMHP" H 7700 1600 50  0001 C CNN "manf_num  "
 	1    7700 1600
 	1    0    0    -1
@@
 F 1 "470nF/16V" V 4850 2850 35  0000 C CNN
 F 2 "Capacitor_SMD:C_0603_1608Metric" H 5038 2700 50  0001 C CNN
-F 3 "https://www.mouser.fi/datasheet/2/447/yago_s_a0011723860_1-2286802.pdf" H 5000 2850 50  0001 C CNN
-F 4 "C519409" V 5000 2850 50  0001 C CNN "LCSC"
-F 5 "CC0603KRX7R7BB471" V 5000 2850 50  0001 C CNN "manf_num"
+F 3 "https://datasheet.lcsc.com/lcsc/1811082118_YAGEO-CC0603KRX7R7BB474_C106851.pdf" H 5000 2850 50  0001 C CNN
+F 4 "C106851" V 5000 2850 50  0001 C CNN "LCSC"
+F 5 "CC0603KRX7R7BB474" V 5000 2850 50  0001 C CNN "manf_num"
 F 6 "CC0603JRX7R7BB471" V 5000 2850 50  0001 C CNN "alt"
 	1    5000 2850
@@
 F 1 "470nF/16V" V 5950 3200 35  0000 C CNN
 F 2 "Capacitor_SMD:C_0603_1608Metric" H 6138 3050 50  0001 C CNN
-F 3 "https://www.mouser.fi/datasheet/2/447/yago_s_a0011723860_1-2286802.pdf" H 6100 3200 50  0001 C CNN
-F 4 "C519409" V 6100 3200 50  0001 C CNN "LCSC"
-F 5 "CC0603KRX7R7BB471" V 6100 3200 50  0001 C CNN "manf_num"
+F 3 "https://datasheet.lcsc.com/lcsc/1811082118_YAGEO-CC0603KRX7R7BB474_C106851.pdf" H 6100 3200 50  0001 C CNN
+F 4 "C106851" V 6100 3200 50  0001 C CNN "LCSC"
+F 5 "CC0603KRX7R7BB474" V 6100 3200 50  0001 C CNN "manf_num"
 F 6 "CC0603JRX7R7BB471" V 6100 3200 50  0001 C CNN "alt"
 	1    6100 3200

Commit message: increase caps
Parts:
- C7, C8, C9: value 2.2uF/100V -> 4.7uF/100V; LCSC C412614 -> C697607; manf_num   HMJ325AB7225KMHP -> HMK325C7475KN-TE
Changed lines of the file:
@@
 P 7700 4400
 F 0 "C8" H 7815 4435 35  0000 L CNN
-F 1 "2.2uF/100V" H 7815 4366 35  0000 L CNN
+F 1 "4.7uF/100V" H 7815 4366 35  0000 L CNN
 F 2 "Capacitor_SMD:C_1210_3225Metric" H 7738 4250 50  0001 C CNN
 F 3 "https://datasheet.lcsc.com/lcsc/1912111437_Taiyo-Yuden-HMJ325AB7225KMHP_C412614.pdf" H 7700 4400 50  0001 C CNN
-F 4 "C412614" H 7700 4400 50  0001 C CNN "LCSC"
-F 5 "HMJ325AB7225KMHP" H 7700 4400 50  0001 C CNN "manf_num  "
+F 4 "C697607" H 7700 4400 50  0001 C CNN "LCSC"
+F 5 "HMK325C7475KN-TE" H 7700 4400 50  0001 C CNN "manf_num  "
 	1    7700 4400
 	1    0    0    -1
@@
 P 9350 2900
 F 0 "C9" H 9465 2935 35  0000 L CNN
-F 1 "2.2uF/100V" H 9465 2866 35  0000 L CNN
+F 1 "4.7uF/100V" H 9465 2866 35  0000 L CNN
 F 2 "Capacitor_SMD:C_1210_3225Metric" H 9388 2750 50  0001 C CNN
 F 3 "https://datasheet.lcsc.com/lcsc/1912111437_Taiyo-Yuden-HMJ325AB7225KMHP_C412614.pdf" H 9350 2900 50  0001 C CNN
-F 4 "C412614" H 9350 2900 50  0001 C CNN "LCSC"
-F 5 "HMJ325AB7225KMHP" H 9350 2900 50  0001 C CNN "manf_num  "
+F 4 "C697607" H 9350 2900 50  0001 C CNN "LCSC"
+F 5 "HMK325C7475KN-TE" H 9350 2900 50  0001 C CNN "manf_num  "
 	1    9350 2900
 	1    0    0    -1
@@
 F 3 "" H 7700 1800 50  0001 C CNN
 	1    7700 1800
-	1    0    0    -1
-$EndComp
-$Comp
-L Device:C C7
-U 1 1 61D9B6F4
-P 7700 1600
-F 0 "C7" H 7815 1635 35  0000 L CNN
-F 1 "2.2uF/100V" H 7815 1566 35  0000 L CNN
-F 2 "Capacitor_SMD:C_1210_3225Metric" H 7738 1450 50  0001 C CNN
-F 3 "https://datasheet.lcsc.com/lcsc/1912111437_Taiyo-Yuden-HMJ325AB7225KMHP_C412614.pdf" H 7700 1600 50  0001 C CNN
-F 4 "C412614" H 7700 1600 50  0001 C CNN "LCSC"
-F 5 "HMJ325AB7225KMHP" H 7700 1600 50  0001 C CNN "manf_num  "
-	1    7700 1600
 	1    0    0    -1
 $EndComp
@@
 Wire Wire Line
 	7150 1350 7700 1350
+$Comp
+L Device:C C7
+U 1 1 61D9B6F4
+P 7700 1600
+F 0 "C7" H 7815 1635 35  0000 L CNN
+F 1 "4.7uF/100V" H 7815 1566 35  0000 L CNN
+F 2 "Capacitor_SMD:C_1210_3225Metric" H 7738 1450 50  0001 C CNN
+F 3 "https://datasheet.lcsc.com/lcsc/1912111437_Taiyo-Yuden-HMJ325AB7225KMHP_C412614.pdf" H 7700 1600 50  0001 C CNN
+F 4 "C697607" H 7700 1600 50  0001 C CNN "LCSC"
+F 5 "HMK325C7475KN-TE" H 7700 1600 50  0001 C CNN "manf_num  "
+	1    7700 1600
+	1    0    0    -1
+$EndComp
 $EndSCHEMATC

Commit message: try routing
Parts:
- Q1, Q2, Q3, Q4, Q5, Q6: symbol opm-inline-rescue:HYG025N06LS1C2 -> opm-inline-rescue:HYG025N06LS1C2-opm-inline-rescue
Other:
- moved on the sheet: Q1, Q2, Q3, Q4, Q5, Q6
Changed lines of the file:
@@
 	5600 2000 7150 2000
 $Comp
-L opm-inline-rescue:HYG025N06LS1C2 Q2
+L opm-inline-rescue:HYG025N06LS1C2-opm-inline-rescue Q2
 U 1 1 61CBF26F
 P 7150 2600
+AR Path="/61CBF26F" Ref="Q2"  Part="1"
+AR Path="/5D5FDD98/61CBF26F" Ref="Q2"  Part="1"
 F 0 "Q2" H 7350 2638 39  0000 L CNN
 F 1 "HYG025N06LS1C2" H 7350 2563 39  0000 L CNN
@@
 	7000 1350 7150 1350
 $Comp
-L opm-inline-rescue:HYG025N06LS1C2 Q1
+L opm-inline-rescue:HYG025N06LS1C2-opm-inline-rescue Q1
 U 1 1 61CDF1C7
 P 7150 1800
+AR Path="/61CDF1C7" Ref="Q1"  Part="1"
+AR Path="/5D5FDD98/61CDF1C7" Ref="Q1"  Part="1"
 F 0 "Q1" H 7350 1838 39  0000 L CNN
 F 1 "HYG025N06LS1C2" H 7350 1763 39  0000 L CNN
@@
 	7000 4150 7150 4150
 $Comp
-L opm-inline-rescue:HYG025N06LS1C2 Q3
+L opm-inline-rescue:HYG025N06LS1C2-opm-inline-rescue Q3
 U 1 1 61CE05AE
 P 7150 4600
+AR Path="/61CE05AE" Ref="Q3"  Part="1"
+AR Path="/5D5FDD98/61CE05AE" Ref="Q3"  Part="1"
 F 0 "Q3" H 7350 4638 39  0000 L CNN
 F 1 "HYG025N06LS1C2" H 7350 4563 39  0000 L CNN
@@
 $EndComp
 $Comp
-L opm-inline-rescue:HYG025N06LS1C2 Q6
+L opm-inline-rescue:HYG025N06LS1C2-opm-inline-rescue Q6
 U 1 1 61CE16E2
 P 8800 3900
+AR Path="/61CE16E2" Ref="Q6"  Part="1"
+AR Path="/5D5FDD98/61CE16E2" Ref="Q6"  Part="1"
 F 0 "Q6" H 9000 3938 39  0000 L CNN
 F 1 "HYG025N06LS1C2" H 9000 3863 39  0000 L CNN
@@
 $EndComp
 $Comp
-L opm-inline-rescue:HYG025N06LS1C2 Q5
+L opm-inline-rescue:HYG025N06LS1C2-opm-inline-rescue Q5
 U 1 1 61CE29B9
 P 8800 3100
+AR Path="/61CE29B9" Ref="Q5"  Part="1"
+AR Path="/5D5FDD98/61CE29B9" Ref="Q5"  Part="1"
 F 0 "Q5" H 9000 3138 39  0000 L CNN
 F 1 "HYG025N06LS1C2" H 9000 3063 39  0000 L CNN
@@
 Connection ~ 8800 3300
 $Comp
-L opm-inline-rescue:HYG025N06LS1C2 Q4
+L opm-inline-rescue:HYG025N06LS1C2-opm-inline-rescue Q4
 U 1 1 61CE42A8
 P 7150 5400
+AR Path="/61CE42A8" Ref="Q4"  Part="1"
+AR Path="/5D5FDD98/61CE42A8" Ref="Q4"  Part="1"
 F 0 "Q4" H 7350 5438 39  0000 L CNN
 F 1 "HYG025N06LS1C2" H 7350 5363 39  0000 L CNN

Commit message: more routing
Parts:
- Q1, Q2, Q3, Q4, Q5, Q6: symbol opm-inline-rescue:HYG025N06LS1C2-opm-inline-rescue -> opm-inline-rescue:HYG025N06LS1C2
Connections:
- net +VM: now also Q1.5 (D), Q1.6 (D), Q1.7 (D), Q1.8 (D), Q3.5 (D), Q3.6 (D), Q3.7 (D), Q3.8 (D), Q5.5 (D), Q5.6 (D), Q5.7 (D), Q5.8 (D); no longer Q1.1 (S), Q1.2 (S), Q1.3 (S), Q3.1 (S), Q3.2 (S), Q3.3 (S), Q5.1 (S), Q5.2 (S), Q5.3 (S)
- net GND: now also Q2.1 (S), Q2.2 (S), Q2.3 (S), Q4.1 (S), Q4.2 (S), Q4.3 (S), Q6.1 (S), Q6.2 (S), Q6.3 (S); no longer Q2.5 (D), Q2.6 (D), Q2.7 (D), Q2.8 (D), Q4.5 (D), Q4.6 (D), Q4.7 (D), Q4.8 (D), Q6.5 (D), Q6.6 (D), Q6.7 (D), Q6.8 (D)
- net W: now reaches R10.1, R5.1, R9.1
- net V: now reaches R12.1, R14.1, R15.1
- net U: now reaches R2.1, R7.1, R8.1
- net +Vcc_IO renamed +VCC_IO
- new net: C5.2, IC1.38 (W), Q3.1 (S), Q3.2 (S), Q3.3 (S), Q4.5 (D), Q4.6 (D), Q4.7 (D), Q4.8 (D), R10.2, R9.2
- new net: C6.1, IC1.42 (V), Q5.1 (S), Q5.2 (S), Q5.3 (S), Q6.5 (D), Q6.6 (D), Q6.7 (D), Q6.8 (D), R14.2, R15.2
- new net: C4.1, IC1.47 (U), Q1.1 (S), Q1.2 (S), Q1.3 (S), Q2.5 (D), Q2.6 (D), Q2.7 (D), Q2.8 (D), R7.2, R8.2
Other:
- moved on the sheet: C7, C9, Q1, Q2, Q3, Q4, Q5, Q6, R1, R11

Commit message: add pic
Parts:
- C4: value 470nF/16V -> 4.7uF/16V; LCSC C106851 -> C19666; alt CC0603JRX7R7BB471 -> (none); manf_num CC0603KRX7R7BB474 -> CL10A475KO8NNNC
- C5, C6: value 470nF/16V -> 4.7UF/16V; LCSC C106851 -> C19666; alt CC0603JRX7R7BB471 -> (none); manf_num CC0603KRX7R7BB474 -> CL10A475KO8NNNC
- R1, R11, R13, R3, R4, R6: value 22R/1% -> 2R2/1%; LCSC C23345 -> C22939; manf_num 0603WAF220JT5E -> 0603WAF220KT5E
Changed lines of the file:
@@
 P 6400 4600
 F 0 "R4" V 6226 4600 35  0000 C CNN
-F 1 "22R/1%" V 6295 4600 35  0000 C CNN
+F 1 "2R2/1%" V 6295 4600 35  0000 C CNN
 F 2 "Resistor_SMD:R_0603_1608Metric" V 6330 4600 50  0001 C CNN
-F 3 "https://datasheet.lcsc.com/szlcsc/Uniroyal-Elec-0603WAF220JT5E_C23345.pdf" H 6400 4600 50  0001 C CNN
-F 4 "C23345" V 6400 4600 50  0001 C CNN "LCSC"
-F 5 "0603WAF220JT5E" V 6400 4600 50  0001 C CNN "manf_num"
+F 3 "https://datasheet.lcsc.com/lcsc/2110252030_UNI-ROYAL-Uniroyal-Elec-0603WAF220KT5E_C22939.pdf" H 6400 4600 50  0001 C CNN
+F 4 "C22939" V 6400 4600 50  0001 C CNN "LCSC"
+F 5 "0603WAF220KT5E" V 6400 4600 50  0001 C CNN "manf_num"
 F 6 "" V 6400 4600 50  0001 C CNN "alt"
 	1    6400 4600
@@
 P 6400 5400
 F 0 "R6" V 6226 5400 35  0000 C CNN
-F 1 "22R/1%" V 6295 5400 35  0000 C CNN
+F 1 "2R2/1%" V 6295 5400 35  0000 C CNN
 F 2 "Resistor_SMD:R_0603_1608Metric" V 6330 5400 50  0001 C CNN
-F 3 "https://datasheet.lcsc.com/szlcsc/Uniroyal-Elec-0603WAF220JT5E_C23345.pdf" H 6400 5400 50  0001 C CNN
-F 4 "C23345" V 6400 5400 50  0001 C CNN "LCSC"
-F 5 "0603WAF220JT5E" V 6400 5400 50  0001 C CNN "manf_num"
+F 3 "https://datasheet.lcsc.com/lcsc/2110252030_UNI-ROYAL-Uniroyal-Elec-0603WAF220KT5E_C22939.pdf" H 6400 5400 50  0001 C CNN
+F 4 "C22939" V 6400 5400 50  0001 C CNN "LCSC"
+F 5 "0603WAF220KT5E" V 6400 5400 50  0001 C CNN "manf_num"
 F 6 "" V 6400 5400 50  0001 C CNN "alt"
 	1    6400 5400
@@
 P 5950 4050
 F 0 "C5" H 6065 4085 35  0000 L CNN
-F 1 "470nF/16V" H 6065 4016 35  0000 L CNN
+F 1 "4.7UF/16V" H 6065 4016 35  0000 L CNN
 F 2 "Capacitor_SMD:C_0603_1608Metric" H 5988 3900 50  0001 C CNN
-F 3 "https://datasheet.lcsc.com/lcsc/1811082118_YAGEO-CC0603KRX7R7BB474_C106851.pdf" H 5950 4050 50  0001 C CNN
-F 4 "C106851" H 5950 4050 50  0001 C CNN "LCSC"
-F 5 "CC0603KRX7R7BB474" H 5950 4050 50  0001 C CNN "manf_num"
-F 6 "CC0603JRX7R7BB471" H 5950 4050 50  0001 C CNN "alt"
+F 3 "https://datasheet.lcsc.com/lcsc/1810261514_Samsung-Electro-Mechanics-CL10A475KO8NNNC_C19666.pdf" H 5950 4050 50  0001 C CNN
+F 4 "C19666" H 5950 4050 50  0001 C CNN "LCSC"
+F 5 "CL10A475KO8NNNC" H 5950 4050 50  0001 C CNN "manf_num"
+F 6 "" H 5950 4050 50  0001 C CNN "alt"
 	1    5950 4050
 	1    0    0    -1
@@
 P 8050 3000
 F 0 "R11" V 7876 3000 35  0000 C CNN
-F 1 "22R/1%" V 7945 3000 35  0000 C CNN
+F 1 "2R2/1%" V 7945 3000 35  0000 C CNN
 F 2 "Resistor_SMD:R_0603_1608Metric" V 7980 3000 50  0001 C CNN
-F 3 "https://datasheet.lcsc.com/szlcsc/Uniroyal-Elec-0603WAF220JT5E_C23345.pdf" H 8050 3000 50  0001 C CNN
-F 4 "C23345" V 8050 3000 50  0001 C CNN "LCSC"
-F 5 "0603WAF220JT5E" V 8050 3000 50  0001 C CNN "manf_num"
+F 3 "https://datasheet.lcsc.com/lcsc/2110252030_UNI-ROYAL-Uniroyal-Elec-0603WAF220KT5E_C22939.pdf" H 8050 3000 50  0001 C CNN
+F 4 "C22939" V 8050 3000 50  0001 C CNN "LCSC"
+F 5 "0603WAF220KT5E" V 8050 3000 50  0001 C CNN "manf_num"
 F 6 "" V 8050 3000 50  0001 C CNN "alt"
 	1    8050 3000
@@
 P 8050 3900
 F 0 "R13" V 7876 3900 35  0000 C CNN
-F 1 "22R/1%" V 7945 3900 35  0000 C CNN
+F 1 "2R2/1%" V 7945 3900 35  0000 C CNN
 F 2 "Resistor_SMD:R_0603_1608Metric" V 7980 3900 50  0001 C CNN
-F 3 "https://datasheet.lcsc.com/szlcsc/Uniroyal-Elec-0603WAF220JT5E_C23345.pdf" H 8050 3900 50  0001 C CNN
-F 4 "C23345" V 8050 3900 50  0001 C CNN "LCSC"
-F 5 "0603WAF220JT5E" V 8050 3900 50  0001 C CNN "manf_num"
+F 3 "https://datasheet.lcsc.com/lcsc/2110252030_UNI-ROYAL-Uniroyal-Elec-0603WAF220KT5E_C22939.pdf" H 8050 3900 50  0001 C CNN
+F 4 "C22939" V 8050 3900 50  0001 C CNN "LCSC"
+F 5 "0603WAF220KT5E" V 8050 3900 50  0001 C CNN "manf_num"
 F 6 "" V 8050 3900 50  0001 C CNN "alt"
 	1    8050 3900
@@
 P 6400 2600
 F 0 "R3" V 6226 2600 35  0000 C CNN
-F 1 "22R/1%" V 6295 2600 35  0000 C CNN
+F 1 "2R2/1%" V 6295 2600 35  0000 C CNN
 F 2 "Resistor_SMD:R_0603_1608Metric" V 6330 2600 50  0001 C CNN
-F 3 "https://datasheet.lcsc.com/szlcsc/Uniroyal-Elec-0603WAF220JT5E_C23345.pdf" H 6400 2600 50  0001 C CNN
-F 4 "C23345" V 6400 2600 50  0001 C CNN "LCSC"
-F 5 "0603WAF220JT5E" V 6400 2600 50  0001 C CNN "manf_num"
+F 3 "https://datasheet.lcsc.com/lcsc/2110252030_UNI-ROYAL-Uniroyal-Elec-0603WAF220KT5E_C22939.pdf" H 6400 2600 50  0001 C CNN
+F 4 "C22939" V 6400 2600 50  0001 C CNN "LCSC"
+F 5 "0603WAF220KT5E" V 6400 2600 50  0001 C CNN "manf_num"
 F 6 "" V 6400 2600 50  0001 C CNN "alt"
 	1    6400 2600
@@
 P 5000 2850
 F 0 "C4" V 4781 2850 35  0000 C CNN
-F 1 "470nF/16V" V 4850 2850 35  0000 C CNN
+F 1 "4.7uF/16V" V 4850 2850 35  0000 C CNN
 F 2 "Capacitor_SMD:C_0603_1608Metric" H 5038 2700 50  0001 C CNN
-F 3 "https://datasheet.lcsc.com/lcsc/1811082118_YAGEO-CC0603KRX7R7BB474_C106851.pdf" H 5000 2850 50  0001 C CNN
-F 4 "C106851" V 5000 2850 50  0001 C CNN "LCSC"
-F 5 "CC0603KRX7R7BB474" V 5000 2850 50  0001 C CNN "manf_num"
-F 6 "CC0603JRX7R7BB471" V 5000 2850 50  0001 C CNN "alt"
+F 3 "https://datasheet.lcsc.com/lcsc/1810261514_Samsung-Electro-Mechanics-CL10A475KO8NNNC_C19666.pdf" H 5000 2850 50  0001 C CNN
+F 4 "C19666" V 5000 2850 50  0001 C CNN "LCSC"
+F 5 "CL10A475KO8NNNC" V 5000 2850 50  0001 C CNN "manf_num"
+F 6 "" V 5000 2850 50  0001 C CNN "alt"
 	1    5000 2850
 	0    1    1    0
@@
 P 6100 3200
 F 0 "C6" V 5881 3200 35  0000 C CNN
-F 1 "470nF/16V" V 5950 3200 35  0000 C CNN
+F 1 "4.7UF/16V" V 5950 3200 35  0000 C CNN
 F 2 "Capacitor_SMD:C_0603_1608Metric" H 6138 3050 50  0001 C CNN
-F 3 "https://datasheet.lcsc.com/lcsc/1811082118_YAGEO-CC0603KRX7R7BB474_C106851.pdf" H 6100 3200 50  0001 C CNN
-F 4 "C106851" V 6100 3200 50  0001 C CNN "LCSC"
-F 5 "CC0603KRX7R7BB474" V 6100 3200 50  0001 C CNN "manf_num"
-F 6 "CC0603JRX7R7BB471" V 6100 3200 50  0001 C CNN "alt"
+F 3 "https://datasheet.lcsc.com/lcsc/1810261514_Samsung-Electro-Mechanics-CL10A475KO8NNNC_C19666.pdf" H 6100 3200 50  0001 C CNN
+F 4 "C19666" V 6100 3200 50  0001 C CNN "LCSC"
+F 5 "CL10A475KO8NNNC" V 6100 3200 50  0001 C CNN "manf_num"
+F 6 "" V 6100 3200 50  0001 C CNN "alt"
 	1    6100 3200
 	0    1    1    0
@@
 P 6400 1650
 F 0 "R1" V 6226 1650 35  0000 C CNN
-F 1 "22R/1%" V 6295 1650 35  0000 C CNN
+F 1 "2R2/1%" V 6295 1650 35  0000 C CNN
 F 2 "Resistor_SMD:R_0603_1608Metric" V 6330 1650 50  0001 C CNN
-F 3 "https://datasheet.lcsc.com/szlcsc/Uniroyal-Elec-0603WAF220JT5E_C23345.pdf" H 6400 1650 50  0001 C CNN
-F 4 "C23345" V 6400 1650 50  0001 C CNN "LCSC"
-F 5 "0603WAF220JT5E" V 6400 1650 50  0001 C CNN "manf_num"
+F 3 "https://datasheet.lcsc.com/lcsc/2110252030_UNI-ROYAL-Uniroyal-Elec-0603WAF220KT5E_C22939.pdf" H 6400 1650 50  0001 C CNN
+F 4 "C22939" V 6400 1650 50  0001 C CNN "LCSC"
+F 5 "0603WAF220KT5E" V 6400 1650 50  0001 C CNN "manf_num"
 F 6 "" V 6400 1650 50  0001 C CNN "alt"
 	1    6400 1650

Commit message: update connections
Connections:
- net SPI1_MISO is gone; now on net +VCC_IO: IC1.16 (SDO_SINGLE)
Changed lines of the file:
@@
 Text HLabel 3650 3600 0    28   Input ~ 0
 SPI1_MOSI
-Text HLabel 3650 3650 0    28   Input ~ 0
-SPI1_MISO
 Text HLabel 3650 3200 0    28   Input ~ 0
 DRV_EN
@@
 Wire Wire Line
 	8500 5000 8800 5000
+Wire Wire Line
+	3650 3650 3150 3650
+Wire Wire Line
+	3150 3650 3150 3950
+Text HLabel 3150 3950 3    31   Input ~ 0
++VCC_IO
 $EndSCHEMATC

Commit message: use pins
Connections:
- net SPI1_MOSI is gone; now on net +VCC_IO: IC1.15 (SDI/AMPLx10)
- net SPI1_SCK is gone; now on net GND: IC1.14 (SCK/IDRV1)
- net ~CS_DRIVER is gone; now on net GND: IC1.13 (CS/IDRV0)
Changed lines of the file:
@@
 Text HLabel 3650 4000 0    28   Input ~ 0
 WL
-Text HLabel 3650 3500 0    28   Input ~ 0
-~CS_DRIVER
-Text HLabel 3650 3550 0    28   Input ~ 0
-SPI1_SCK
-Text HLabel 3650 3600 0    28   Input ~ 0
-SPI1_MOSI
 Text HLabel 3650 3200 0    28   Input ~ 0
 DRV_EN
@@
 Wire Wire Line
 	8500 5000 8800 5000
-Wire Wire Line
-	3650 3650 3150 3650
-Wire Wire Line
-	3150 3650 3150 3950
-Text HLabel 3150 3950 3    31   Input ~ 0
+Text HLabel 3450 3650 0    31   Input ~ 0
 +VCC_IO
+Text HLabel 3450 3600 0    31   Input ~ 0
++VCC_IO
+Wire Wire Line
+	3450 3600 3650 3600
+Wire Wire Line
+	3650 3650 3450 3650
+$Comp
+L power:GND #PWR?
+U 1 1 61F1E038
+P 3150 3550
+F 0 "#PWR?" H 3150 3300 39  0001 C CNN
+F 1 "GND" H 3150 3400 39  0000 C CNN
+F 2 "" H 3150 3550 39  0001 C CNN
+F 3 "" H 3150 3550 39  0001 C CNN
+	1    3150 3550
+	-1   0    0    1
+$EndComp
+$Comp
+L power:GND #PWR?
+U 1 1 61F1F1E2
+P 3400 3500
+F 0 "#PWR?" H 3400 3250 39  0001 C CNN
+F 1 "GND" H 3400 3350 39  0000 C CNN
+F 2 "" H 3400 3500 39  0001 C CNN
+F 3 "" H 3400 3500 39  0001 C CNN
+	1    3400 3500
+	-1   0    0    1
+$EndComp
+Wire Wire Line
+	3650 3550 3150 3550
+Wire Wire Line
+	3650 3500 3400 3500
 $EndSCHEMATC
