File: opm-inline/source/Connectors.sch (KiCad schematic (older format))
At the start: 27 parts, among them J1 SPI/Info, J2 VCC_IO, J3 PWMx6, J5 Temperature, J6 Current Sensing, U2 TerminalBlock_2_P5.08mm, U3 TerminalBlock_3_P5.08mm

Commit message: update position
Parts:
- H201, H202: footprint MountingHole:MountingHole_3.2mm_M3_Pad -> MountingHole:MountingHole_3.2mm_M3_DIN965_Pad
Changed lines of the file:
@@
 F 0 "H202" V 6750 1450 39  0000 L CNN
 F 1 "MountingHole" V 6800 1450 39  0000 L CNN
-F 2 "MountingHole:MountingHole_3.2mm_M3_Pad" H 6800 1300 39  0001 C CNN
+F 2 "MountingHole:MountingHole_3.2mm_M3_DIN965_Pad" H 6800 1300 39  0001 C CNN
 F 3 "~" H 6800 1300 39  0001 C CNN
 F 4 "No" V 6800 1300 50  0001 C CNN "JLCPCB BOM"
@@
 F 0 "H201" V 6750 1250 39  0000 L CNN
 F 1 "MountingHole" V 6800 1250 39  0000 L CNN
-F 2 "MountingHole:MountingHole_3.2mm_M3_Pad" H 6800 1100 39  0001 C CNN
+F 2 "MountingHole:MountingHole_3.2mm_M3_DIN965_Pad" H 6800 1100 39  0001 C CNN
 F 3 "~" H 6800 1100 39  0001 C CNN
 F 4 "No" V 6800 1100 50  0001 C CNN "JLCPCB BOM"

Commit message: try routing
Parts:
- H201, H202: footprint MountingHole:MountingHole_3.2mm_M3_DIN965_Pad -> MountingHole:MountingHole_3.2mm_M3_Pad_Via
Changed lines of the file:
@@
 F 0 "H202" V 6750 1450 39  0000 L CNN
 F 1 "MountingHole" V 6800 1450 39  0000 L CNN
-F 2 "MountingHole:MountingHole_3.2mm_M3_DIN965_Pad" H 6800 1300 39  0001 C CNN
+F 2 "MountingHole:MountingHole_3.2mm_M3_Pad_Via" H 6800 1300 39  0001 C CNN
 F 3 "~" H 6800 1300 39  0001 C CNN
 F 4 "No" V 6800 1300 50  0001 C CNN "JLCPCB BOM"
@@
 F 0 "H201" V 6750 1250 39  0000 L CNN
 F 1 "MountingHole" V 6800 1250 39  0000 L CNN
-F 2 "MountingHole:MountingHole_3.2mm_M3_DIN965_Pad" H 6800 1100 39  0001 C CNN
+F 2 "MountingHole:MountingHole_3.2mm_M3_Pad_Via" H 6800 1100 39  0001 C CNN
 F 3 "~" H 6800 1100 39  0001 C CNN
 F 4 "No" V 6800 1100 50  0001 C CNN "JLCPCB BOM"

Commit message: try routing
Parts:
- H202: footprint MountingHole:MountingHole_3.2mm_M3_Pad_Via -> MountingHole:MountingHole_3mm_Pad
Changed lines of the file:
@@
 F 0 "H202" V 6750 1450 39  0000 L CNN
 F 1 "MountingHole" V 6800 1450 39  0000 L CNN
-F 2 "MountingHole:MountingHole_3.2mm_M3_Pad_Via" H 6800 1300 39  0001 C CNN
+F 2 "MountingHole:MountingHole_3mm_Pad" H 6800 1300 39  0001 C CNN
 F 3 "~" H 6800 1300 39  0001 C CNN
 F 4 "No" V 6800 1300 50  0001 C CNN "JLCPCB BOM"

Commit message: more routing
Parts:
- H202: footprint MountingHole:MountingHole_3mm_Pad -> MountingHole:MountingHole_3.2mm_M3_Pad_Via
Connections:
- net VCC_IO is gone; now on net +VCC_IO: J2.1 (Pin_1)
Changed lines of the file:
@@
 F 0 "H202" V 6750 1450 39  0000 L CNN
 F 1 "MountingHole" V 6800 1450 39  0000 L CNN
-F 2 "MountingHole:MountingHole_3mm_Pad" H 6800 1300 39  0001 C CNN
+F 2 "MountingHole:MountingHole_3.2mm_M3_Pad_Via" H 6800 1300 39  0001 C CNN
 F 3 "~" H 6800 1300 39  0001 C CNN
 F 4 "No" V 6800 1300 50  0001 C CNN "JLCPCB BOM"
@@
 $EndComp
 Text HLabel 1050 4450 2    39   Output ~ 0
-VCC_IO
++VCC_IO
 $Comp
 L power:GND #PWR0110

Commit message: add pic
Connections:
- net +VCC_IO: now also R16.1
Changed lines of the file:
@@
 	1    0    0    -1
 $EndComp
+Text HLabel 3800 4100 2    31   Input ~ 0
++VCC_IO
 $EndSCHEMATC

Commit message: update connections
Parts:
- removed J5: Temperature, Connector_JST:JST_PH_B2B-PH-K_1x02_P2.00mm_Vertical, symbol Connector:Conn_01x02_Female
- added J4: Fan, Connector_JST:JST_PH_B2B-PH-K_1x02_P2.00mm_Vertical, symbol Connector:Conn_01x02_Female
Connections:
- net Fault is gone; now on net FAULT: R20.2
- net SPI1_MISO is gone; now on net DRV_EN: J1.4 (Pin_4)
- net DRV_EN: no longer J1.5 (Pin_5)
- net GND: now also J4.2 (Pin_2)
- net TEMP_PCB: now reaches C17.1, R17.2, R18.1
- net TEMP_PCB: now also J1.5 (Pin_5)
Other:
- note added: "Fan"
- note removed: "Temperature"
Changed lines of the file:
@@
 $EndComp
 Text HLabel 4100 3000 0    50   Input ~ 0
-Fault
+FAULT
 Wire Wire Line
 	4700 3000 5150 3000
@@
 	1    0    0    -1
 $EndComp
-$Comp
-L Connector:Conn_01x02_Female J5
-U 1 1 61C07AC4
-P 5650 5150
-F 0 "J5" H 5400 5200 50  0000 L CNN
-F 1 "Temperature" H 5700 5150 50  0000 L CNN
-F 2 "Connector_JST:JST_PH_B2B-PH-K_1x02_P2.00mm_Vertical" H 5650 5150 50  0001 C CNN
-F 3 "https://datasheet.lcsc.com/lcsc/1811151524_JST-Sales-America-B2B-PH-K-S-LF-SN_C131337.pdf" H 5650 5150 50  0001 C CNN
-F 4 "C131337" H 5650 5150 50  0001 C CNN "LCSC"
-F 5 "B2B-PH-K-S(LF)(SN)" H 5650 5150 50  0001 C CNN "manf_num"
-	1    5650 5150
-	1    0    0    -1
-$EndComp
 Wire Wire Line
 	3800 4650 3800 4400
-Wire Wire Line
-	5450 5150 4700 5150
 Wire Wire Line
 	3800 4950 3800 5150
@@
 Wire Wire Line
 	4700 5250 4700 5150
-Connection ~ 4700 5150
 Wire Wire Line
 	4700 5150 3800 5150
@@
 	1    0    0    -1
 $EndComp
-$Comp
-L power:GND #PWR0109
-U 1 1 61C0E704
-P 5350 5650
-F 0 "#PWR0109" H 5350 5400 39  0001 C CNN
-F 1 "GND" H 5350 5500 39  0000 C CNN
-F 2 "" H 5350 5650 50  0001 C CNN
-F 3 "" H 5350 5650 50  0001 C CNN
-	1    5350 5650
-	1    0    0    -1
-$EndComp
-Wire Wire Line
-	5450 5250 5350 5250
-Wire Wire Line
-	5350 5250 5350 5650
 Wire Wire Line
 	4700 5550 4700 5650
 Wire Wire Line
 	3800 5550 3800 5650
-Text Notes 3850 5100 0    39   ~ 0
-Temperature
 $Comp
 L Connector:Conn_01x06_Female J3
@@
 $EndComp
 Text HLabel 1400 5600 0    50   Input ~ 0
-SPI1_MISO
+DRV_EN
 Text HLabel 1400 5700 0    50   Input ~ 0
-DRV_EN
+TEMP_PCB
 Text HLabel 1400 5800 0    50   Input ~ 0
 FAULT
@@
 Text HLabel 3800 4100 2    31   Input ~ 0
 +VCC_IO
+Wire Notes Line
+	3500 7700 6300 7700
+Wire Notes Line
+	6300 7700 6300 6200
+Wire Notes Line
+	6300 6200 3500 6200
+Wire Notes Line
+	3500 6200 3500 7700
+$Comp
+L Connector:Conn_01x02_Female J4
+U 1 1 61EB9C93
+P 5650 6700
+F 0 "J4" H 5400 6750 50  0000 L CNN
+F 1 "Fan" H 5700 6700 50  0000 L CNN
+F 2 "Connector_JST:JST_PH_B2B-PH-K_1x02_P2.00mm_Vertical" H 5650 6700 50  0001 C CNN
+F 3 "https://datasheet.lcsc.com/lcsc/1811151524_JST-Sales-America-B2B-PH-K-S-LF-SN_C131337.pdf" H 5650 6700 50  0001 C CNN
+F 4 "C131337" H 5650 6700 50  0001 C CNN "LCSC"
+F 5 "B2B-PH-K-S(LF)(SN)" H 5650 6700 50  0001 C CNN "manf_num"
+	1    5650 6700
+	1    0    0    -1
+$EndComp
+Wire Wire Line
+	5450 6700 4700 6700
+$Comp
+L power:GND #PWR011
+U 1 1 61EB9F7E
+P 5350 7200
+F 0 "#PWR011" H 5350 6950 39  0001 C CNN
+F 1 "GND" H 5350 7050 39  0000 C CNN
+F 2 "" H 5350 7200 50  0001 C CNN
+F 3 "" H 5350 7200 50  0001 C CNN
+	1    5350 7200
+	1    0    0    -1
+$EndComp
+Wire Wire Line
+	5450 6800 5350 6800
+Wire Wire Line
+	5350 6800 5350 7200
+Text HLabel 5450 5150 2    31   Input ~ 0
+TEMP_PCB
+Wire Wire Line
+	4700 5150 5450 5150
+Connection ~ 4700 5150
+Text Notes 3650 6450 0    79   ~ 0
+Fan
 $EndSCHEMATC

Commit message: use pins
Parts:
- J1: value SPI/Info -> Info; footprint Connector_JST:JST_PH_B6B-PH-K_1x06_P2.00mm_Vertical -> Connector_JST:JST_PH_B3B-PH-K_1x03_P2.00mm_Vertical; symbol Connector:Conn_01x06_Female -> Connector:Conn_01x03_Female; LCSC C265365 -> (none); manf_num B6B-PH-KL(LF)(SN) -> (none)
Connections:
- net SPI1_MOSI is gone; now on net FAULT: J1.3 (Pin_3)
- net SPI1_SCK is gone; now on net TEMP_PCB: J1.2 (Pin_2)
- net ~CS_DRIVER is gone; now on net DRV_EN: J1.1 (Pin_1)
- net DRV_EN: no longer J1.4 (Pin_4)
- net FAULT: no longer J1.6 (Pin_6)
- net TEMP_PCB: no longer J1.5 (Pin_5)
Changed lines of the file:
@@
 Wire Wire Line
 	1700 1750 2350 1750
-$Comp
-L Connector:Conn_01x06_Female J1
-U 1 1 61C4DAFD
-P 1600 5500
-F 0 "J1" H 1700 5400 50  0000 C CNN
-F 1 "SPI/Info" H 1800 5500 50  0000 C CNN
-F 2 "Connector_JST:JST_PH_B6B-PH-K_1x06_P2.00mm_Vertical" H 1600 5500 50  0001 C CNN
-F 3 "https://datasheet.lcsc.com/lcsc/1912111437_JST-Sales-America-B6B-PH-KL-LF-SN_C265365.pdf" H 1600 5500 50  0001 C CNN
-F 4 "C265365" H 1600 5500 50  0001 C CNN "LCSC"
-F 5 "B6B-PH-KL(LF)(SN)" H 1600 5500 50  0001 C CNN "manf_num"
-F 6 "copper when possible over brass" H 1600 5500 50  0001 C CNN "comment"
-	1    1600 5500
-	1    0    0    -1
-$EndComp
+Text HLabel 1400 5400 0    50   Input ~ 0
+DRV_EN
+Text HLabel 1400 5500 0    50   Input ~ 0
+TEMP_PCB
 Text HLabel 1400 5600 0    50   Input ~ 0
-DRV_EN
-Text HLabel 1400 5700 0    50   Input ~ 0
-TEMP_PCB
-Text HLabel 1400 5800 0    50   Input ~ 0
 FAULT
-Text HLabel 1400 5400 0    50   Input ~ 0
-SPI1_SCK
-Text HLabel 1400 5300 0    50   Input ~ 0
-~CS_DRIVER
-Text HLabel 1400 5500 0    50   Input ~ 0
-SPI1_MOSI
 Wire Notes Line
 	8500 750  7500 750
@@
 Text Notes 3650 6450 0    79   ~ 0
 Fan
+$Comp
+L Connector:Conn_01x03_Female J1
+U 1 1 61C4DAFD
+P 1600 5500
+F 0 "J1" H 1700 5400 50  0000 C CNN
+F 1 "Info" H 1800 5500 50  0000 C CNN
+F 2 "Connector_JST:JST_PH_B3B-PH-K_1x03_P2.00mm_Vertical" H 1600 5500 50  0001 C CNN
+F 3 "" H 1600 5500 50  0001 C CNN
+F 4 "" H 1600 5500 50  0001 C CNN "LCSC"
+F 5 "" H 1600 5500 50  0001 C CNN "manf_num"
+F 6 "copper when possible over brass" H 1600 5500 50  0001 C CNN "comment"
+	1    1600 5500
+	1    0    0    -1
+$EndComp
 $EndSCHEMATC

Commit message: update connections
Parts:
- D2: value 19-217/GHC-YR1S2/3T -> Red LED; Info Green -> Red; LCSC C72043 -> C2286; manf_num 19-217/GHC-YR1S2/3T -> KT-0603R
- J1: LCSC (none) -> C131339; manf_num (none) -> B3B-PH-K-S(LF)(SN)
Connections:
- net FAULT: no longer R20.2
- new net FAULT_LED: R20.2
Changed lines of the file:
@@
 $Descr A4 11693 8268
 encoding utf-8
-Sheet 2 3
+Sheet 3 3
 Title "TMC6100-EVAL"
 Date "2019-10-28"
@@
 P 5300 3000
 F 0 "D2" H 5293 2745 50  0000 C CNN
-F 1 "19-217/GHC-YR1S2/3T" H 5293 2836 50  0000 C CNN
+F 1 "Red LED" H 5293 2836 50  0000 C CNN
 F 2 "LED_SMD:LED_0603_1608Metric" H 5300 3000 50  0001 C CNN
-F 3 "https://datasheet.lcsc.com/lcsc/1811101510_Everlight-Elec-19-217-GHC-YR1S2-3T_C72043.pdf" H 5300 3000 50  0001 C CNN
-F 4 "Green" H 5300 3000 50  0001 C CNN "Info"
-F 5 "C72043" H 5300 3000 50  0001 C CNN "LCSC"
-F 6 "19-217/GHC-YR1S2/3T" H 5300 3000 50  0001 C CNN "manf_num"
+F 3 "https://datasheet.lcsc.com/lcsc/1810231112_Hubei-KENTO-Elec-KT-0603R_C2286.pdf" H 5300 3000 50  0001 C CNN
+F 4 "Red" H 5300 3000 50  0001 C CNN "Info"
+F 5 "C2286" H 5300 3000 50  0001 C CNN "LCSC"
+F 6 "KT-0603R" H 5300 3000 50  0001 C CNN "manf_num"
 	1    5300 3000
 	-1   0    0    1
 $EndComp
 Text HLabel 4100 3000 0    50   Input ~ 0
-FAULT
+FAULT_LED
 Wire Wire Line
 	4700 3000 5150 3000
@@
 Text HLabel 1350 6350 0    50   Input ~ 0
 ADC_I_u
-Text HLabel 1350 6450 0    50   Input ~ 0
-ADC_I_v
 Text HLabel 1350 6550 0    50   Input ~ 0
 ADC_I_w
@@
 Wire Wire Line
 	5350 6800 5350 7200
-Text HLabel 5450 5150 2    31   Input ~ 0
+Text HLabel 5450 5150 2    31   Output ~ 0
 TEMP_PCB
 Wire Wire Line
@@
 F 1 "Info" H 1800 5500 50  0000 C CNN
 F 2 "Connector_JST:JST_PH_B3B-PH-K_1x03_P2.00mm_Vertical" H 1600 5500 50  0001 C CNN
-F 3 "" H 1600 5500 50  0001 C CNN
-F 4 "" H 1600 5500 50  0001 C CNN "LCSC"
-F 5 "" H 1600 5500 50  0001 C CNN "manf_num"
+F 3 "https://datasheet.lcsc.com/lcsc/1811151524_JST-Sales-America-B3B-PH-K-S-LF-SN_C131339.pdf" H 1600 5500 50  0001 C CNN
+F 4 "C131339" H 1600 5500 50  0001 C CNN "LCSC"
+F 5 "B3B-PH-K-S(LF)(SN)" H 1600 5500 50  0001 C CNN "manf_num"
 F 6 "copper when possible over brass" H 1600 5500 50  0001 C CNN "comment"
 	1    1600 5500
 	1    0    0    -1
 $EndComp
+Text HLabel 1350 6450 0    50   Input ~ 0
+ADC_I_v
 $EndSCHEMATC
