File: opm-inline/source/Connectors.sch (KiCad schematic (older format))
At the start: 27 parts, among them J1 Info, J2 VCC_IO, J3 PWMx6, J4 Fan, J6 Current Sensing, U2 TerminalBlock_2_P5.08mm, U3 TerminalBlock_3_P5.08mm

Commit message: rearrange
Parts:
- D1: value 19-217/GHC-YR1S2/3T -> Green LED
Changed lines of the file:
@@
 P 5300 1500
 F 0 "D1" H 5293 1245 50  0000 C CNN
-F 1 "19-217/GHC-YR1S2/3T" H 5293 1336 50  0000 C CNN
+F 1 "Green LED" H 5293 1336 50  0000 C CNN
 F 2 "LED_SMD:LED_0603_1608Metric" H 5300 1500 50  0001 C CNN
 F 3 "https://datasheet.lcsc.com/lcsc/1811101510_Everlight-Elec-19-217-GHC-YR1S2-3T_C72043.pdf" H 5300 1500 50  0001 C CNN

Commit message: use pins
Connections:
- net FAULT is gone; now on net GND: J1.3 (Pin_3)
- net FAULT_LED is gone; now on net GND: R20.2
Other:
- moved on the sheet: D2, R20
Changed lines of the file:
@@
 L Device:R R20
 U 1 1 61C21201
-P 4550 3000
-F 0 "R20" V 4343 3000 50  0000 C CNN
-F 1 "150R/1%" V 4434 3000 50  0000 C CNN
-F 2 "Resistor_SMD:R_0603_1608Metric" V 4480 3000 50  0001 C CNN
-F 3 "https://datasheet.lcsc.com/lcsc/2110252030_UNI-ROYAL-Uniroyal-Elec-0603WAF1500T5E_C22808.pdf" H 4550 3000 50  0001 C CNN
-F 4 "C22808" V 4550 3000 50  0001 C CNN "LCSC"
-F 5 "0603WAF1500T5E" V 4550 3000 50  0001 C CNN "manf_num"
-	1    4550 3000
+P 4450 2950
+F 0 "R20" V 4243 2950 50  0000 C CNN
+F 1 "150R/1%" V 4334 2950 50  0000 C CNN
+F 2 "Resistor_SMD:R_0603_1608Metric" V 4380 2950 50  0001 C CNN
+F 3 "https://datasheet.lcsc.com/lcsc/2110252030_UNI-ROYAL-Uniroyal-Elec-0603WAF1500T5E_C22808.pdf" H 4450 2950 50  0001 C CNN
+F 4 "C22808" V 4450 2950 50  0001 C CNN "LCSC"
+F 5 "0603WAF1500T5E" V 4450 2950 50  0001 C CNN "manf_num"
+	1    4450 2950
 	0    1    1    0
-$EndComp
-$Comp
-L power:GND #PWR0106
-U 1 1 61C2120B
-P 5650 3200
-F 0 "#PWR0106" H 5650 2950 39  0001 C CNN
-F 1 "GND" H 5650 3050 39  0000 C CNN
-F 2 "" H 5650 3200 50  0001 C CNN
-F 3 "" H 5650 3200 50  0001 C CNN
-	1    5650 3200
-	1    0    0    -1
 $EndComp
 $Comp
 L Device:LED D2
 U 1 1 61C21218
-P 5300 3000
-F 0 "D2" H 5293 2745 50  0000 C CNN
-F 1 "Red LED" H 5293 2836 50  0000 C CNN
-F 2 "LED_SMD:LED_0603_1608Metric" H 5300 3000 50  0001 C CNN
-F 3 "https://datasheet.lcsc.com/lcsc/1810231112_Hubei-KENTO-Elec-KT-0603R_C2286.pdf" H 5300 3000 50  0001 C CNN
-F 4 "Red" H 5300 3000 50  0001 C CNN "Info"
-F 5 "C2286" H 5300 3000 50  0001 C CNN "LCSC"
-F 6 "KT-0603R" H 5300 3000 50  0001 C CNN "manf_num"
-	1    5300 3000
+P 5200 2950
+F 0 "D2" H 5193 2695 50  0000 C CNN
+F 1 "Red LED" H 5193 2786 50  0000 C CNN
+F 2 "LED_SMD:LED_0603_1608Metric" H 5200 2950 50  0001 C CNN
+F 3 "https://datasheet.lcsc.com/lcsc/1810231112_Hubei-KENTO-Elec-KT-0603R_C2286.pdf" H 5200 2950 50  0001 C CNN
+F 4 "Red" H 5200 2950 50  0001 C CNN "Info"
+F 5 "C2286" H 5200 2950 50  0001 C CNN "LCSC"
+F 6 "KT-0603R" H 5200 2950 50  0001 C CNN "manf_num"
+	1    5200 2950
 	-1   0    0    1
 $EndComp
-Text HLabel 4100 3000 0    50   Input ~ 0
-FAULT_LED
-Wire Wire Line
-	4700 3000 5150 3000
-Wire Wire Line
-	5450 3000 5650 3000
-Wire Wire Line
-	5650 3000 5650 3200
-Wire Wire Line
-	4100 3000 4400 3000
+Text HLabel 4000 2950 0    50   Input ~ 0
+FAULT
+Wire Wire Line
+	4600 2950 5050 2950
+Wire Wire Line
+	5350 2950 5450 2950
+Wire Wire Line
+	4000 2950 4300 2950
 Wire Wire Line
 	6550 1300 6550 1850
@@
 Text HLabel 1350 6450 0    50   Input ~ 0
 ADC_I_v
+Text HLabel 5550 2950 2    50   Output ~ 0
+FAULT
+$Comp
+L power:GND #PWR?
+U 1 1 61E2CD97
+P 5450 3200
+F 0 "#PWR?" H 5450 2950 39  0001 C CNN
+F 1 "GND" H 5450 3050 39  0000 C CNN
+F 2 "" H 5450 3200 50  0001 C CNN
+F 3 "" H 5450 3200 50  0001 C CNN
+	1    5450 3200
+	1    0    0    -1
+$EndComp
+Wire Wire Line
+	5450 3200 5450 2950
+Connection ~ 5450 2950
+Wire Wire Line
+	5450 2950 5550 2950
 $EndSCHEMATC

Commit message: rearrange
Parts:
- H201, H202: footprint MountingHole:MountingHole_3.2mm_M3_Pad_Via -> MountingHole:MountingHole_2.2mm_M2_Pad_Via
Changed lines of the file:
@@
 F 0 "H202" V 6750 1450 39  0000 L CNN
 F 1 "MountingHole" V 6800 1450 39  0000 L CNN
-F 2 "MountingHole:MountingHole_3.2mm_M3_Pad_Via" H 6800 1300 39  0001 C CNN
+F 2 "MountingHole:MountingHole_2.2mm_M2_Pad_Via" H 6800 1300 39  0001 C CNN
 F 3 "~" H 6800 1300 39  0001 C CNN
 F 4 "No" V 6800 1300 50  0001 C CNN "JLCPCB BOM"
@@
 F 0 "H201" V 6750 1250 39  0000 L CNN
 F 1 "MountingHole" V 6800 1250 39  0000 L CNN
-F 2 "MountingHole:MountingHole_3.2mm_M3_Pad_Via" H 6800 1100 39  0001 C CNN
+F 2 "MountingHole:MountingHole_2.2mm_M2_Pad_Via" H 6800 1100 39  0001 C CNN
 F 3 "~" H 6800 1100 39  0001 C CNN
 F 4 "No" V 6800 1100 50  0001 C CNN "JLCPCB BOM"

Commit message: rearrange
Parts:
- added D4: 10V, Diode_SMD:D_SOD-123, symbol Simulation_SPICE:DIODE
- added Q7: WSD90P06DN56, Libraries:PDFN-8, symbol opm-inline-rescue:HYG025N06LS1C2
- added R27: 100KR, Resistor_SMD:R_0603_1608Metric, symbol Device:R
Connections:
- net +VCC_IO: now also J4.1 (Pin_1)
- net +VM: now also D4.2 (K), Q7.1 (S), Q7.2 (S), Q7.3 (S); no longer U2.2
- net GND: now also R27.2
- new net: Q7.5 (D), Q7.6 (D), Q7.7 (D), Q7.8 (D), U2.2
- new net: D4.1 (A), Q7.4 (G), R27.1
Other:
- moved on the sheet: C15, C16, U2
Changed lines of the file:
@@
 Wire Notes Line
 	600  750  3400 750
-Text Notes 700  950  0    79   ~ 0
+Text Notes 700  900  0    79   ~ 0
 Power Connector
 Wire Notes Line
@@
 L opm-cache:Conector_library_Metz_31330102 U2
 U 1 1 61BFF192
-P 1500 1300
-F 0 "U2" H 1500 1100 39  0000 C CNN
-F 1 "TerminalBlock_2_P5.08mm" H 1500 1150 39  0000 C CNN
-F 2 "Libraries:TerminalBlock_bornier-2_P5.08mm" H 1500 1150 39  0001 C CNN
-F 3 "https://datasheet.lcsc.com/lcsc/1912251636_Ningbo-Kangnex-Elec-WJ500V-5-08-2P_C8465.pdf" H 1550 1300 39  0001 C CNN
-F 4 "C8465" H 1500 1300 50  0001 C CNN "LCSC"
-F 5 "WJ500V-5.08-2P" H 1500 1300 50  0001 C CNN "manf_num"
-	1    1500 1300
+P 750 1200
+F 0 "U2" H 750 1000 39  0000 C CNN
+F 1 "TerminalBlock_2_P5.08mm" H 750 1050 39  0000 C CNN
+F 2 "Libraries:TerminalBlock_bornier-2_P5.08mm" H 750 1050 39  0001 C CNN
+F 3 "https://datasheet.lcsc.com/lcsc/1912251636_Ningbo-Kangnex-Elec-WJ500V-5-08-2P_C8465.pdf" H 800 1200 39  0001 C CNN
+F 4 "C8465" H 750 1200 50  0001 C CNN "LCSC"
+F 5 "WJ500V-5.08-2P" H 750 1200 50  0001 C CNN "manf_num"
+	1    750  1200
 	-1   0    0    1
 $EndComp
 Wire Wire Line
-	1700 1350 1600 1350
+	950  1250 850  1250
 $Comp
 L Device:CP1 C15
 U 1 1 61BFF3DC
-P 2350 1500
-F 0 "C15" V 2200 1500 39  0000 C CNN
-F 1 "330uF/63V" V 2500 1500 39  0000 C CNN
-F 2 "Capacitor_THT:C_Radial_D10.0mm_H20.0mm_P5.00mm" V 2550 1500 39  0001 C CNN
-F 3 "~" H 2350 1500 39  0001 C CNN
-F 4 "C338235" V 2350 1500 50  0001 C CNN "LCSC"
-F 5 "63ZLH330MEFC10X23" V 2350 1500 50  0001 C CNN "manf_num"
-	1    2350 1500
+P 2450 1400
+F 0 "C15" V 2300 1400 39  0000 C CNN
+F 1 "330uF/63V" V 2600 1400 39  0000 C CNN
+F 2 "Capacitor_THT:C_Radial_D10.0mm_H20.0mm_P5.00mm" V 2650 1400 39  0001 C CNN
+F 3 "~" H 2450 1400 39  0001 C CNN
+F 4 "C338235" V 2450 1400 50  0001 C CNN "LCSC"
+F 5 "63ZLH330MEFC10X23" V 2450 1400 50  0001 C CNN "manf_num"
+	1    2450 1400
 	1    0    0    -1
 $EndComp
@@
 L Device:CP1 C16
 U 1 1 61BFF3E8
-P 2850 1500
-F 0 "C16" V 2700 1500 39  0000 C CNN
-F 1 "330uF/63V" V 3000 1500 39  0000 C CNN
-F 2 "Capacitor_THT:C_Radial_D10.0mm_H20.0mm_P5.00mm" H 2850 1500 39  0001 C CNN
-F 3 "~" H 2850 1500 39  0001 C CNN
-F 4 "C338235" V 2850 1500 50  0001 C CNN "LCSC"
-F 5 "63ZLH330MEFC10X23" V 2850 1500 50  0001 C CNN "manf_num"
-	1    2850 1500
-	1    0    0    -1
-$EndComp
-Wire Wire Line
-	2850 1350 2850 1250
-Wire Wire Line
-	2850 1250 2350 1250
-Wire Wire Line
-	2350 1250 2350 1350
-Wire Wire Line
-	2350 1650 2350 1750
-Wire Wire Line
-	2350 1750 2850 1750
-Wire Wire Line
-	2850 1750 2850 1650
-Connection ~ 2350 1250
+P 2950 1400
+F 0 "C16" V 2800 1400 39  0000 C CNN
+F 1 "330uF/63V" V 3100 1400 39  0000 C CNN
+F 2 "Capacitor_THT:C_Radial_D10.0mm_H20.0mm_P5.00mm" H 2950 1400 39  0001 C CNN
+F 3 "~" H 2950 1400 39  0001 C CNN
+F 4 "C338235" V 2950 1400 50  0001 C CNN "LCSC"
+F 5 "63ZLH330MEFC10X23" V 2950 1400 50  0001 C CNN "manf_num"
+	1    2950 1400
+	1    0    0    -1
+$EndComp
+Wire Wire Line
+	2950 1250 2950 1150
+Wire Wire Line
+	2950 1150 2450 1150
+Wire Wire Line
+	2450 1150 2450 1250
+Wire Wire Line
+	2450 1550 2450 1650
+Wire Wire Line
+	2450 1650 2950 1650
+Wire Wire Line
+	2950 1650 2950 1550
 $Comp
 L power:GND #PWR0104
 U 1 1 61BFF3F9
-P 2850 1850
-F 0 "#PWR0104" H 2850 1600 39  0001 C CNN
-F 1 "GND" H 2850 1700 39  0000 C CNN
-F 2 "" H 2850 1850 50  0001 C CNN
-F 3 "" H 2850 1850 50  0001 C CNN
-	1    2850 1850
-	1    0    0    -1
-$EndComp
-Text HLabel 3100 1250 2    39   Output ~ 0
+P 2950 1750
+F 0 "#PWR0104" H 2950 1500 39  0001 C CNN
+F 1 "GND" H 2950 1600 39  0000 C CNN
+F 2 "" H 2950 1750 50  0001 C CNN
+F 3 "" H 2950 1750 50  0001 C CNN
+	1    2950 1750
+	1    0    0    -1
+$EndComp
+Text HLabel 3200 1150 2    39   Output ~ 0
 +VM
 Wire Wire Line
-	2850 1750 2850 1850
-Connection ~ 2850 1750
-Wire Wire Line
-	1700 1350 1700 1750
-Connection ~ 2350 1750
-Wire Wire Line
-	2850 1250 3100 1250
-Connection ~ 2850 1250
+	2950 1650 2950 1750
+Connection ~ 2950 1650
+Wire Wire Line
+	2950 1150 3200 1150
+Connection ~ 2950 1150
 Wire Notes Line
 	600  3750 600  6900
@@
 Text HLabel 1350 6550 0    50   Input ~ 0
 ADC_I_w
-Wire Wire Line
-	1600 1250 2350 1250
-Wire Wire Line
-	1700 1750 2350 1750
 Text HLabel 1400 5400 0    50   Input ~ 0
 DRV_EN
@@
 Wire Wire Line
 	5450 2950 5550 2950
+$Comp
+L Device:R R27
+U 1 1 61FF437F
+P 1700 1700
+F 0 "R27" H 1770 1746 50  0000 L CNN
+F 1 "100KR" H 1770 1655 50  0000 L CNN
+F 2 "Resistor_SMD:R_0603_1608Metric" V 1630 1700 50  0001 C CNN
+F 3 "https://datasheet.lcsc.com/lcsc/2110260030_UNI-ROYAL-Uniroyal-Elec-0603WAF1003T5E_C25803.pdf" H 1700 1700 50  0001 C CNN
+F 4 "C25803" H 1700 1700 50  0001 C CNN "LCSC"
+F 5 "0603WAF1003T5E" H 1700 1700 50  0001 C CNN "manf_num"
+	1    1700 1700
+	1    0    0    -1
+$EndComp
+$Comp
+L Simulation_SPICE:DIODE D4
+U 1 1 61FF80EA
+P 2150 1300
+F 0 "D4" V 2196 1220 50  0000 R CNN
+F 1 "10V" V 2105 1220 50  0000 R CNN
+F 2 "Diode_SMD:D_SOD-123" H 2150 1300 50  0001 C CNN
+F 3 "https://datasheet.lcsc.com/lcsc/1809291220_onsemi-MMSZ5240BT1G_C82084.pdf" H 2150 1300 50  0001 C CNN
+F 4 "MMSZ5240BT1G" V 2150 1300 50  0001 C CNN "manf_num"
+F 5 "C82084" V 2150 1300 50  0001 C CNN "LCSC"
+	1    2150 1300
+	0    -1   -1   0
+$EndComp
+Wire Wire Line
+	1700 1850 1700 1900
+Wire Wire Line
+	1700 1450 1700 1550
+Wire Wire Line
+	2150 1450 2150 1550
+Wire Wire Line
+	2150 1550 1700 1550
+Connection ~ 1700 1550
+Wire Wire Line
+	1900 1150 2150 1150
+Wire Wire Line
+	2150 1150 2450 1150
+Connection ~ 2150 1150
+Connection ~ 2450 1150
+$Comp
+L power:GND #PWR0115
+U 1 1 6202D3B9
+P 1700 2000
+F 0 "#PWR0115" H 1700 1750 39  0001 C CNN
+F 1 "GND" H 1700 1850 39  0000 C CNN
+F 2 "" H 1700 2000 50  0001 C CNN
+F 3 "" H 1700 2000 50  0001 C CNN
+	1    1700 2000
+	1    0    0    -1
+$EndComp
+Wire Wire Line
+	1700 1900 1700 2000
+Connection ~ 1700 1900
+Wire Wire Line
+	950  1250 950  1900
+Wire Wire Line
+	850  1150 1500 1150
+Wire Wire Line
+	950  1900 1700 1900
+$Comp
+L opm-inline-rescue:HYG025N06LS1C2 Q7
+U 1 1 6204314F
+P 1700 1250
+F 0 "Q7" V 2144 1250 39  0000 C CNN
+F 1 "WSD90P06DN56" V 2069 1250 39  0000 C CNN
+F 2 "Libraries:PDFN-8" H 1900 1175 39  0001 L CIN
+F 3 "" V 1700 1250 50  0001 L CNN
+F 4 "C719104" V 1700 1250 50  0001 C CNN "LCSC"
+F 5 "WSD90P06DN56" V 1700 1250 50  0001 C CNN "manf_num"
+	1    1700 1250
+	0    -1   -1   0
+$EndComp
+Text HLabel 4700 6700 0    50   Input ~ 0
++VCC_IO
 $EndSCHEMATC

Commit message: more routing
Parts:
- added D3, D5: SP0505BAJT, Package_TO_SOT_SMD:SOT-363_SC-70-6, symbol Power_Protection:SP0505BAJT
- added D6: TVS DIODE, Diode_SMD:D_SMA, symbol Simulation_SPICE:DIODE
- J1, J6: symbol Connector:Conn_01x03_Female -> Connector_Generic:Conn_01x03
- J2: symbol Connector:Conn_01x02_Female -> Connector_Generic:Conn_01x02
- J3: symbol Connector:Conn_01x06_Female -> Connector_Generic:Conn_01x06
Connections:
- net +VCC_IO: now also D5.1 (K)
- net DRV_EN: now also D5.5 (K)
- net GND: now also D5.3 (K), D6.1 (A)
- net TEMP_PCB: now also D5.4 (K)
- net UH: now also D5.6 (K)
- net UL: now also D3.1 (K)
- net VH: now also D3.3 (K)
- net VL: now also D3.4 (K)
- net WH: now also D3.5 (K)
- net WL: now also D3.6 (K)
- net at Q7.5 (D), Q7.6 (D), Q7.7 (D)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: now also D6.2 (K)
Other:
- moved on the sheet: J2

Commit message: more routing
Connections:
- net GND: now also D3.2 (A), D5.2 (A)
Other:
- moved on the sheet: D3, D5, J1, J2, J3, J6

Commit message: esd
Parts:
- added D7: NUP4114UCW1T2G, Libraries:NUP4114UCW1T2G, symbol Power_Protection:SP0505BAJT
- D3, D5: value SP0505BAJT -> NUP4114UCW1T2G; footprint Package_TO_SOT_SMD:SOT-363_SC-70-6 -> Libraries:NUP4114UCW1T2G; LCSC (none) -> C463643; manf_num (none) -> NUP4114UCW1T2G
Connections:
- net ADC_I_u: now also J6.3 (Pin_3), D7.6 (K); no longer J6.1 (Pin_1)
- net ADC_I_v: now also D7.4 (K)
- net ADC_I_w: now also J6.1 (Pin_1), D7.1 (K); no longer J6.3 (Pin_3)
- net GND: now also D7.2 (A)
Other:
- moved on the sheet: D3, D5, J1, J2, J3, J6
