File: opm-inline/source/Connectors.sch (KiCad schematic (older format))
At the start: 34 parts, among them J1 Info, J2 VCC_IO, J3 PWMx6, J4 Fan, J6 Current Sensing, Q7 WSD90P06DN56, U2 TerminalBlock_2_P5.08mm, U3 TerminalBlock_3_P5.08mm

Commit message: esd
Parts:
- D6: LCSC C499728 -> C523249; manf_num SMAJ58CA -> SMA(DO-214AC)
Connections:
- net UH: now also D3.6 (K); no longer D5.6 (K)
- net UL: now also D3.5 (K); no longer D3.1 (K)
- net WH: now also D3.1 (K); no longer D3.5 (K)
- net WL: now also D5.6 (K); no longer D3.6 (K)
Changed lines of the file:
@@
 $EndComp
 Wire Wire Line
-	1000 5300 2150 5300
-Wire Wire Line
 	1000 5800 2350 5800
-Wire Wire Line
-	2150 4650 2150 5300
-Connection ~ 2150 5300
-Wire Wire Line
-	2150 5300 2900 5300
 Wire Wire Line
 	2250 4650 2250 5700
@@
 Wire Wire Line
 	1000 6200 2950 6200
-Wire Wire Line
-	2550 4650 2550 6100
-Wire Wire Line
-	1000 6100 2550 6100
-Connection ~ 2550 6100
-Wire Wire Line
-	2550 6100 2900 6100
 $Comp
 L Simulation_SPICE:DIODE D6
@@
 F 1 "TVS DIODE" V 1255 1420 50  0000 R CNN
 F 2 "Diode_SMD:D_SMA" H 1300 1500 50  0001 C CNN
-F 3 "https://datasheet.lcsc.com/lcsc/2009171004_SMC-Sangdest-Microelectronicstronic--Nanjing-SMAJ58CA_C499728.pdf" H 1300 1500 50  0001 C CNN
-F 4 "C499728" V 1300 1500 50  0001 C CNN "LCSC"
-F 5 "SMAJ58CA" V 1300 1500 50  0001 C CNN "manf_num"
+F 3 "https://datasheet.lcsc.com/lcsc/2007161833_Brightking-Elec--TAIWAN-SMAJ58CA-AT_C523249.pdf" H 1300 1500 50  0001 C CNN
+F 4 "C523249" V 1300 1500 50  0001 C CNN "LCSC"
+F 5 "SMA(DO-214AC)" V 1300 1500 50  0001 C CNN "manf_num"
 	1    1300 1500
 	0    -1   -1   0
@@
 Connection ~ 1450 5000
 Wire Wire Line
-	1250 4800 2900 4800
-Connection ~ 1250 4800
-Wire Wire Line
-	1350 4900 2900 4900
-Connection ~ 1350 4900
-Wire Wire Line
-	1650 5200 2900 5200
-Connection ~ 1650 5200
-Wire Wire Line
 	1550 5100 2900 5100
 Connection ~ 1550 5100
-Wire Wire Line
-	1000 5200 1650 5200
 Wire Wire Line
 	1000 5100 1550 5100
 Wire Wire Line
 	1000 5000 1450 5000
-Wire Wire Line
-	1000 4900 1350 4900
-Wire Wire Line
-	1000 4800 1250 4800
 $Comp
 L power:GND #PWR0116
@@
 $EndComp
 Wire Wire Line
-	1650 4650 1650 5200
-Wire Wire Line
 	1550 4650 1550 5100
 Wire Wire Line
 	1450 4650 1450 5000
-Wire Wire Line
-	1350 4650 1350 4900
-Wire Wire Line
-	1250 4650 1250 4800
 $Comp
 L Power_Protection:SP0505BAJT D3
@@
 	1    0    0    -1
 $EndComp
+Wire Wire Line
+	2150 4650 2150 4800
+Connection ~ 2150 4800
+Wire Wire Line
+	2150 4800 2900 4800
+Wire Wire Line
+	1000 4800 2150 4800
+Wire Wire Line
+	1250 4650 1250 5300
+Wire Wire Line
+	1000 5300 1250 5300
+Connection ~ 1250 5300
+Wire Wire Line
+	1250 5300 2900 5300
+Wire Wire Line
+	1000 6100 2550 6100
+Wire Wire Line
+	2550 6100 2900 6100
+Connection ~ 2550 6100
+Wire Wire Line
+	2550 4650 2550 6100
+Wire Wire Line
+	1000 4900 1650 4900
+Wire Wire Line
+	1350 4650 1350 5200
+Wire Wire Line
+	1000 5200 1350 5200
+Connection ~ 1350 5200
+Wire Wire Line
+	1350 5200 2900 5200
+Wire Wire Line
+	1650 4650 1650 4900
+Connection ~ 1650 4900
+Wire Wire Line
+	1650 4900 2900 4900
 $EndSCHEMATC

Commit message: esd
Connections:
- net +VCC_IO: now also D5.3 (K); no longer D5.1 (K)
- net DRV_EN: now also D5.4 (K); no longer D5.5 (K)
- net GND: no longer D5.3 (K), J1.3 (Pin_3), R20.2
- net TEMP_PCB: now also D5.6 (K); no longer D5.4 (K)
- net VH: now also D3.4 (K); no longer D3.3 (K)
- net VL: now also D3.3 (K); no longer D3.4 (K)
- net WL: now also D5.5 (K); no longer D5.6 (K)
- new net FAULT: D5.1 (K), J1.3 (Pin_3), R20.2
Changed lines of the file:
@@
 Text HLabel 2900 6650 2    50   Output ~ 0
 ADC_I_v
-Text HLabel 5550 2950 2    50   Output ~ 0
-FAULT
 $Comp
 L power:GND #PWR0114
@@
 Wire Wire Line
 	5450 3200 5450 2950
-Connection ~ 5450 2950
-Wire Wire Line
-	5450 2950 5550 2950
 $Comp
 L Device:R R27
@@
 $EndComp
 Wire Wire Line
-	1000 5800 2350 5800
-Wire Wire Line
-	2250 4650 2250 5700
-Wire Wire Line
-	1000 5700 2250 5700
-Connection ~ 2250 5700
-Wire Wire Line
-	2250 5700 2900 5700
-Wire Wire Line
-	2350 4650 2350 5800
-Connection ~ 2350 5800
-Wire Wire Line
-	2350 5800 2900 5800
-Wire Wire Line
-	2450 4650 2450 5900
-Wire Wire Line
-	1000 5900 2450 5900
-Connection ~ 2450 5900
-Wire Wire Line
-	2450 5900 2900 5900
-Wire Wire Line
 	1000 6200 2950 6200
 $Comp
@@
 	-1   0    0    1
 $EndComp
-Wire Wire Line
-	1450 5000 2900 5000
-Connection ~ 1450 5000
-Wire Wire Line
-	1550 5100 2900 5100
-Connection ~ 1550 5100
-Wire Wire Line
-	1000 5100 1550 5100
-Wire Wire Line
-	1000 5000 1450 5000
 $Comp
 L power:GND #PWR0116
@@
 	-1   0    0    1
 $EndComp
-Wire Wire Line
-	1550 4650 1550 5100
-Wire Wire Line
-	1450 4650 1450 5000
 $Comp
 L Power_Protection:SP0505BAJT D3
@@
 $EndComp
 Wire Wire Line
-	2150 4650 2150 4800
-Connection ~ 2150 4800
-Wire Wire Line
-	2150 4800 2900 4800
-Wire Wire Line
-	1000 4800 2150 4800
-Wire Wire Line
 	1250 4650 1250 5300
 Wire Wire Line
@@
 	1250 5300 2900 5300
 Wire Wire Line
-	1000 6100 2550 6100
-Wire Wire Line
-	2550 6100 2900 6100
-Connection ~ 2550 6100
-Wire Wire Line
-	2550 4650 2550 6100
-Wire Wire Line
 	1000 4900 1650 4900
 Wire Wire Line
@@
 Wire Wire Line
 	1650 4900 2900 4900
+Wire Wire Line
+	1000 5000 1550 5000
+Wire Wire Line
+	1000 5100 1450 5100
+Wire Wire Line
+	1550 4650 1550 5000
+Connection ~ 1550 5000
+Wire Wire Line
+	1550 5000 2900 5000
+Wire Wire Line
+	1450 4650 1450 5100
+Connection ~ 1450 5100
+Wire Wire Line
+	1450 5100 2900 5100
+Wire Wire Line
+	2350 4650 2350 5700
+Wire Wire Line
+	1000 5700 2350 5700
+Connection ~ 2350 5700
+Wire Wire Line
+	2350 5700 2900 5700
+Wire Wire Line
+	1000 6100 2450 6100
+Wire Wire Line
+	2450 4650 2450 6100
+Connection ~ 2450 6100
+Wire Wire Line
+	2450 6100 2900 6100
+Wire Wire Line
+	2550 4650 2550 5900
+Wire Wire Line
+	1000 5900 2550 5900
+Connection ~ 2550 5900
+Wire Wire Line
+	2550 5900 2900 5900
+Wire Wire Line
+	1000 5800 2150 5800
+Wire Wire Line
+	1000 4800 2250 4800
+Wire Wire Line
+	2150 4650 2150 5800
+Connection ~ 2150 5800
+Wire Wire Line
+	2150 5800 2900 5800
+Wire Wire Line
+	2250 4650 2250 4800
+Connection ~ 2250 4800
+Wire Wire Line
+	2250 4800 2900 4800
 $EndSCHEMATC

Commit message: update
Other:
- note added: "Logos and Silk Screen"
Changed lines of the file:
@@
 	7500 4250 8500 4250
-Wire Notes Line
-	8500 4250 8500 2250
 Wire Notes Line
 	8500 2250 7500 2250
@@
 P 2350 4450
 F 0 "D5" H 2045 4404 50  0000 R CNN
-F 1 "NUP4114UCW1T2G" H 2045 4495 50  0000 R CNN
+F 1 "NUP4114UCW1T2G" H 2045 4495 50  0001 R CNN
 F 2 "Libraries:NUP4114UCW1T2G" H 2650 4400 50  0001 L CNN
 F 3 "https://datasheet.lcsc.com/lcsc/2001031717_onsemi-NUP4114UCW1T2G_C463643.pdf" H 2475 4575 50  0001 C CNN
@@
 P 1450 4450
 F 0 "D3" H 1145 4404 50  0000 R CNN
-F 1 "NUP4114UCW1T2G" H 1145 4495 50  0000 R CNN
+F 1 "NUP4114UCW1T2G" H 1145 4495 50  0001 R CNN
 F 2 "Libraries:NUP4114UCW1T2G" H 1750 4400 50  0001 L CNN
 F 3 "https://datasheet.lcsc.com/lcsc/2001031717_onsemi-NUP4114UCW1T2G_C463643.pdf" H 1575 4575 50  0001 C CNN
@@
 P 1450 7250
 F 0 "D7" H 1755 7296 50  0000 L CNN
-F 1 "NUP4114UCW1T2G" H 1755 7205 50  0000 L CNN
+F 1 "NUP4114UCW1T2G" H 1755 7205 50  0001 L CNN
 F 2 "Libraries:NUP4114UCW1T2G" H 1750 7200 50  0001 L CNN
 F 3 "https://datasheet.lcsc.com/lcsc/2001031717_onsemi-NUP4114UCW1T2G_C463643.pdf" H 1575 7375 50  0001 C CNN
@@
 Wire Wire Line
 	2250 4800 2900 4800
+Wire Notes Line
+	11100 4400 11100 6050
+Wire Notes Line
+	11100 6050 6400 6050
+Wire Notes Line
+	6400 6050 6400 4400
+Wire Notes Line
+	6400 4400 11100 4400
+Wire Notes Line
+	8500 2250 8500 4250
+$Comp
+L Graphic:Logo_Open_Hardware_Small #LOGO1
+U 1 1 61E56420
+P 7000 5200
+F 0 "#LOGO1" H 7000 5475 50  0000 C CNN
+F 1 "Logo_Open_Hardware_Small" H 7000 4975 50  0001 C CNN
+F 2 "Symbol:OSHW-Logo2_9.8x8mm_SilkScreen" H 7000 5200 50  0001 C CNN
+F 3 "~" H 7000 5200 50  0001 C CNN
+	1    7000 5200
+	1    0    0    -1
+$EndComp
+Text Notes 6550 4700 0    79   ~ 0
+Logos and Silk Screen
 $EndSCHEMATC

Commit message: update
Parts:
- HS1: footprint Libraries:Heatsink_30x30mm_2xFixation3mm -> Symbol:OSHW-Logo2_7.3x6mm_Copper; back (none) -> Libraries:Heatsink_30x30mm_2xFixation3mm
Changed lines of the file:
@@
-	1    0    0    -1
-$EndComp
-$Comp
-L power:GND #PWR0111
-U 1 1 61C3E273
-P 6850 3750
-F 0 "#PWR0111" H 6850 3500 39  0001 C CNN
-F 1 "GND" H 6850 3600 39  0000 C CNN
-F 2 "" H 6850 3750 50  0001 C CNN
-F 3 "" H 6850 3750 50  0001 C CNN
-	1    6850 3750
 	1    0    0    -1
 $EndComp
@@
 Wire Notes Line
 	7200 3400 7200 3750
-Wire Notes Line
-	7200 3750 6600 3750
 Wire Notes Line
 	6600 3750 6600 3400
@@
 Text Notes 7550 2450 0    79   ~ 0
 VCC_IO VOFS
-Text Notes 6900 3750 0    28   ~ 0
-Not Mounted
 $Comp
 L Connector_Generic:Conn_01x03 J6
@@
 L Mechanical:Heatsink HS1
 U 1 1 61CA5775
-P 7950 1550
-F 0 "HS1" H 8092 1671 50  0000 L CNN
-F 1 "Heatsink" H 8092 1580 50  0000 L CNN
-F 2 "Libraries:Heatsink_30x30mm_2xFixation3mm" H 7962 1550 50  0001 C CNN
-F 3 "~" H 7962 1550 50  0001 C CNN
-	1    7950 1550
+P 7850 1600
+F 0 "HS1" H 7992 1721 50  0001 L CNN
+F 1 "Heatsink" H 7992 1630 50  0001 L CNN
+F 2 "Symbol:OSHW-Logo2_7.3x6mm_Copper" H 7862 1600 50  0001 C CNN
+F 3 "~" H 7862 1600 50  0001 C CNN
+F 4 "Libraries:Heatsink_30x30mm_2xFixation3mm" H 7850 1600 50  0001 C CNN "back"
+	1    7850 1600
 	1    0    0    -1
 $EndComp
@@
 U 1 1 61E56420
 P 7000 5200
-F 0 "#LOGO1" H 7000 5475 50  0000 C CNN
-F 1 "Logo_Open_Hardware_Small" H 7000 4975 50  0001 C CNN
+F 0 "#LOGO1" H 7000 5475 50  0001 C CNN
+F 1 "Logo_Open_Hardware_Small" H 7000 4975 50  0000 C CNN
 F 2 "Symbol:OSHW-Logo2_9.8x8mm_SilkScreen" H 7000 5200 50  0001 C CNN
 F 3 "~" H 7000 5200 50  0001 C CNN
@@
 Text Notes 6550 4700 0    79   ~ 0
 Logos and Silk Screen
+Wire Notes Line
+	7650 1700 8350 1700
+Wire Notes Line
+	8350 1700 8350 1300
+Wire Notes Line
+	8350 1300 7650 1300
+Wire Notes Line
+	7650 1300 7650 1700
+Text Notes 6900 3750 0    28   ~ 0
+Not Mounted
+Wire Notes Line
+	7200 3750 6600 3750
+$Comp
+L power:GND #PWR0111
+U 1 1 61C3E273
+P 6850 3750
+F 0 "#PWR0111" H 6850 3500 39  0001 C CNN
+F 1 "GND" H 6850 3600 39  0000 C CNN
+F 2 "" H 6850 3750 50  0001 C CNN
+F 3 "" H 6850 3750 50  0001 C CNN
+	1    6850 3750
+	1    0    0    -1
+$EndComp
 $EndSCHEMATC
