File: opm-inline/source/opm-inline.kicad_pcb (KiCad board)
At the start: 4 copper layers, 58 x 40 mm, 65 parts, among them IC1 TMC6200-TA, J1 SPI/Info, J2 VCC_IO, J3 PWMx6, J5 Temperature, J6 Current Sensing, Q1 HYG025N06LS1C2, Q2 HYG025N06LS1C2, Q3 HYG025N06LS1C2, Q4 HYG025N06LS1C2, Q5 HYG025N06LS1C2, Q6 HYG025N06LS1C2, U2 TerminalBlock_2_P5.08mm, U3 TerminalBlock_3_P5.08mm

Commit message: try routing
Routing:
- net Net-(R12-Pad1): vias 5 -> 0
- net Net-(R10-Pad1): vias 10 -> 9
- net /+VM: vias 18 -> 24
- added copper zone on B.Cu, net /+VM
- added copper zone on In2.Cu, net GND
Changed lines of the file:
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@@
     (1 In1.Cu signal hide)
     (2 In2.Cu signal hide)
-    (31 B.Cu mixed)
+    (31 B.Cu mixed hide)
     (32 B.Adhes user)
     (33 F.Adhes user)
@@
   (segment (start 162.56 73.66) (end 167.64 73.66) (width 4) (layer In2.Cu) (net 3) (status 40000))
   (segment (start 167.64 73.66) (end 171.45 69.85) (width 4) (layer In2.Cu) (net 3) (status 40000))
-  (segment (start 151.13 73.66) (end 162.56 73.66) (width 4) (layer In2.Cu) (net 3) (status 40000))
   (segment (start 162.56 73.66) (end 167.64 73.66) (width 4) (layer B.Cu) (net 3) (status 40000))
   (segment (start 167.64 73.66) (end 171.45 69.85) (width 4) (layer B.Cu) (net 3) (status 40000))
@@
   (via (at 176.93 104.14) (size 0.6) (drill 0.3) (layers F.Cu B.Cu) (net 57))
   (via (at 176.93 105.41) (size 0.6) (drill 0.3) (layers F.Cu B.Cu) (net 57))
-  (via (at 175.66 105.41) (size 0.6) (drill 0.3) (layers F.Cu B.Cu) (net 57))
+  (via (at 175.66 105.41) (size 0.6) (drill 0.3) (layers F.Cu B.Cu) (net 3))
   (via (at 175.66 104.14) (size 0.6) (drill 0.3) (layers F.Cu B.Cu) (net 57))
   (via (at 175.66 102.87) (size 0.6) (drill 0.3) (layers F.Cu B.Cu) (net 57))
   (via (at 175.66 101.6) (size 0.6) (drill 0.3) (layers F.Cu B.Cu) (net 57))
   (via (at 175.66 100.33) (size 0.6) (drill 0.3) (layers F.Cu B.Cu) (net 57))
-  (via (at 167.64 88.9) (size 0.6) (drill 0.3) (layers F.Cu B.Cu) (net 58))
-  (via (at 167.64 90.17) (size 0.6) (drill 0.3) (layers F.Cu B.Cu) (net 58))
-  (via (at 167.64 91.44) (size 0.6) (drill 0.3) (layers F.Cu B.Cu) (net 58))
-  (via (at 167.64 92.71) (size 0.6) (drill 0.3) (layers F.Cu B.Cu) (net 58))
-  (via (at 167.64 93.98) (size 0.6) (drill 0.3) (layers F.Cu B.Cu) (net 58))
+  (via (at 167.64 88.9) (size 0.6) (drill 0.3) (layers F.Cu B.Cu) (net 3))
+  (via (at 167.64 90.17) (size 0.6) (drill 0.3) (layers F.Cu B.Cu) (net 3))
+  (via (at 167.64 91.44) (size 0.6) (drill 0.3) (layers F.Cu B.Cu) (net 3))
+  (via (at 167.64 92.71) (size 0.6) (drill 0.3) (layers F.Cu B.Cu) (net 3))
+  (via (at 167.64 93.98) (size 0.6) (drill 0.3) (layers F.Cu B.Cu) (net 3))
+  (segment (start 151.13 73.66) (end 162.56 73.66) (width 4) (layer In2.Cu) (net 3) (status 40000))
   (zone (net 13) (net_name /W) (layer B.Cu) (hatch edge 0.508)
     (priority 1)
@@
       )
     )
+  )
+  (zone (net 3) (net_name /+VM) (layer B.Cu) (hatch edge 0.508)
+    (connect_pads (clearance 0.508))
+    (min_thickness 0.254)
+    (fill yes (arc_segments 32) (thermal_gap 0) (thermal_bridge_width 0.508) (smoothing fillet) (radius 0.4))
+    (polygon
+      (pts
+        (xy 187.39 106.18) (xy 130.24 106.18) (xy 130.24 66.81) (xy 187.39 66.81)
+      )
+    )
+  )
+  (zone (net 5) (net_name GND) (layer In2.Cu) (hatch edge 0.508)
+    (connect_pads (clearance 0.508))
+    (min_thickness 0.254)
+    (fill yes (arc_segments 32) (thermal_gap 0) (thermal_bridge_width 0.508) (smoothing fillet) (radius 0.4))
+    (polygon
+      (pts
+        (xy 187.39 106.18) (xy 130.24 106.18) (xy 130.24 66.81) (xy 187.39 66.81)
+      )
+    )

Commit message: more routing
Parts:
- H202: footprint MountingHole:MountingHole_3mm_Pad -> MountingHole:MountingHole_3.2mm_M3_Pad_Via
- moved R21 47.3 mm to (180.4, 75.4)
- moved R23 45.7 mm to (177.5, 75.4)
- moved R22 41.4 mm to (174.5, 75.4)
- moved R24 5.88 mm to (143.5, 96.5)
- moved R1 2.10 mm to (171.5, 75.4)
- moved D2 1.27 mm to (180.3, 69.1)
- moved C18 0.92 mm to (143.8, 98.4)
- moved D1 0.79 mm to (180.3, 72.4)
- moved Q5 0.40 mm to (163.4, 87.6)
- moved Q6 0.40 mm to (163.4, 94.0)
- moved C20 0.20 mm to (137.5, 97.5)
- moved C12 0.20 mm to (174.2, 90.2)
- moved R15 0.20 mm to (170.4, 92.5), turned to 180 degrees
- moved R4 0.20 mm to (174.2, 93.2)
- turned R10 to 180 degrees
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Connections:
- net /+Vcc_IO renamed /Motor Driver/+VCC_IO
- J2 pad 1: /Connectors/VCC_IO -> /Connectors/+VCC_IO
- Q1 pad 1: Net-(R2-Pad1) -> Net-(C4-Pad1)
- Q1 pad 2: Net-(R2-Pad1) -> Net-(C4-Pad1)
- Q1 pad 3: Net-(R2-Pad1) -> Net-(C4-Pad1)
- Q2 pad 5: Net-(R2-Pad1) -> Net-(C4-Pad1)
- Q2 pad 6: Net-(R2-Pad1) -> Net-(C4-Pad1)
- Q2 pad 7: Net-(R2-Pad1) -> Net-(C4-Pad1)
- Q2 pad 8: Net-(R2-Pad1) -> Net-(C4-Pad1)
- Q3 pad 1: Net-(R10-Pad1) -> Net-(C5-Pad2)
- Q3 pad 2: Net-(R10-Pad1) -> Net-(C5-Pad2)
- Q3 pad 3: Net-(R10-Pad1) -> Net-(C5-Pad2)
- Q4 pad 5: Net-(R10-Pad1) -> Net-(C5-Pad2)
- Q4 pad 6: Net-(R10-Pad1) -> Net-(C5-Pad2)
- Q4 pad 7: Net-(R10-Pad1) -> Net-(C5-Pad2)
- Q4 pad 8: Net-(R10-Pad1) -> Net-(C5-Pad2)
- Q5 pad 1: Net-(R12-Pad1) -> Net-(C6-Pad1)
- Q5 pad 2: Net-(R12-Pad1) -> Net-(C6-Pad1)
- Q5 pad 3: Net-(R12-Pad1) -> Net-(C6-Pad1)
- Q6 pad 5: Net-(R12-Pad1) -> Net-(C6-Pad1)
- Q6 pad 6: Net-(R12-Pad1) -> Net-(C6-Pad1)
- Q6 pad 7: Net-(R12-Pad1) -> Net-(C6-Pad1)
- Q6 pad 8: Net-(R12-Pad1) -> Net-(C6-Pad1)
- R10 pad 1: Net-(R10-Pad1) -> /W
- R10 pad 2: /W -> Net-(C5-Pad2)
- R12 pad 1: Net-(R12-Pad1) -> /V
- R14 pad 1: Net-(R12-Pad1) -> /V
- R15 pad 1: Net-(R12-Pad1) -> /V
- R2 pad 1: Net-(R2-Pad1) -> /U
- R4 pad 1: /V -> Net-(Q3-Pad4)
- R5 pad 1: Net-(R10-Pad1) -> /W
- R7 pad 1: Net-(R2-Pad1) -> /U
- R7 pad 2: /U -> Net-(C4-Pad1)
- R8 pad 1: Net-(R2-Pad1) -> /U
- R8 pad 2: /U -> Net-(C4-Pad1)
- R9 pad 1: Net-(R10-Pad1) -> /W
- R9 pad 2: /W -> Net-(C5-Pad2)
Routing:
- net Net-(R2-Pad1): vias 10 -> 0
- net Net-(R10-Pad1): vias 9 -> 0
- net Net-(C6-Pad1): vias 0 -> 9
- net Net-(C5-Pad2): vias 0 -> 10
- net Net-(C4-Pad1): vias 0 -> 10
- net /+VM: vias 24 -> 27
- added copper zone on F.Cu, net Net-(C4-Pad1)
- added copper zone on F.Cu, net Net-(C5-Pad2)
- removed copper zone on B.Cu, net /U
- removed copper zone on B.Cu, net /V
- removed copper zone on B.Cu, net /W
- removed copper zone on F.Cu, net Net-(R10-Pad1)
- removed copper zone on F.Cu, net Net-(R12-Pad1)
- removed copper zone on F.Cu, net Net-(R2-Pad1)

Commit message: more routing
Routing:
- net Net-(C6-Pad1): vias 9 -> 8
- added copper zone on B.Cu, net /U
- added copper zone on B.Cu, net /V
- added copper zone on B.Cu, net /W
- added copper zone on B.Cu, net Net-(C4-Pad1)
- added copper zone on B.Cu, net Net-(C5-Pad2)
- added copper zone on B.Cu, net Net-(C6-Pad1)
- added copper zone on F.Cu, net Net-(C6-Pad1)
- removed copper zone on In2.Cu, net GND
- removed copper zone on B.Cu, net Net-(R10-Pad1)

Commit message: add pic
Parts:
- C4: value 470nF/16V -> 4.7uF/16V
- C5, C6: value 470nF/16V -> 4.7UF/16V
- R1, R11, R13, R3, R4, R6: value 22R/1% -> 2R2/1%
Connections:
- R16 pad 1: Net-(R16-Pad1) -> /Connectors/+VCC_IO
Routing:
- net Net-(C4-Pad1): vias 10 -> 9
- net GND: vias 0 -> 2
- net /+VM: vias 27 -> 26
- added copper zone on F.Cu, net GND

Commit message: update connections
Parts:
- removed J5: Temperature, Connector_JST:JST_PH_B2B-PH-K_1x02_P2.00mm_Vertical
- added J4: Fan, Connector_JST:JST_PH_B2B-PH-K_1x02_P2.00mm_Vertical, F.Cu at (185.4, 104.1)
- moved R18 6.25 mm to (152.2, 81.3)
- moved C17 4.21 mm to (153.7, 78.3), turned to 90 degrees
- moved R16 2.09 mm to (155.1, 80.5)
- moved R17 1.27 mm to (153.7, 81.3), turned to 90 degrees
- turned R20 to 180 degrees
Connections:
- C17 pad 1: Net-(C17-Pad1) -> /Connectors/TEMP_PCB
- IC1 pad 16: /SPI1_MISO -> /Motor Driver/+VCC_IO
- J1 pad 4: /SPI1_MISO -> /DRV_EN
- J1 pad 5: /DRV_EN -> /Connectors/TEMP_PCB
- R17 pad 2: Net-(C17-Pad1) -> /Connectors/TEMP_PCB
- R18 pad 1: Net-(C17-Pad1) -> /Connectors/TEMP_PCB
- R20 pad 2: /Connectors/Fault -> /Connectors/FAULT

Commit message: use pins
Parts:
- J1: value SPI/Info -> Info; footprint Connector_JST:JST_PH_B6B-PH-K_1x06_P2.00mm_Vertical -> Connector_JST:JST_PH_B3B-PH-K_1x03_P2.00mm_Vertical
- moved J1 6.05 mm to (139.4, 73.7)
- moved J4 2.54 mm to (185.4, 101.6), turned to 270 degrees
- moved Q3 0.40 mm to (171.4, 97.4)
- moved Q4 0.40 mm to (171.4, 103.3)
Connections:
- IC1 pad 13: /~CS_DRIVER -> GND
- IC1 pad 14: /SPI1_SCK -> GND
- IC1 pad 15: /SPI1_MOSI -> /Motor Driver/+VCC_IO
- J1 pad 1: /~CS_DRIVER -> /DRV_EN
- J1 pad 2: /SPI1_SCK -> /Connectors/TEMP_PCB
- J1 pad 3: /SPI1_MOSI -> /Connectors/FAULT
Routing:
- net GND: vias 2 -> 10
- net /+VM: vias 26 -> 27

Commit message: update connections
Parts:
- D2: value 19-217/GHC-YR1S2/3T -> Red LED
- moved HS1 17.8 mm to (241.3, 94.0)
- moved J1 0.45 mm to (139.4, 74.1)
- moved J6 0.40 mm to (185.4, 77.1)
- moved R11 0.20 mm to (164.7, 82.8)
- moved R2 0.20 mm to (164.7, 79.8)
- moved J4 0.10 mm to (185.4, 101.7)
- moved R18 0.10 mm to (152.1, 81.3)
- moved R16 0.05 mm to (155.2, 80.5)
- turned R12 to 180 degrees
Connections:
- net Net-(IC1-Pad26) renamed /Fault
Routing:
- net Net-(C4-Pad1): vias 9 -> 10
- net GND: vias 10 -> 16
Other:
- rule via_min_size: 0.4 -> 0.3

Commit message: rearrange
Parts:
- D1: value 19-217/GHC-YR1S2/3T -> Green LED
- moved J4 53.9 mm to (133.1, 88.9)
- moved J6 40.7 mm to (144.8, 75.2), turned to 180 degrees
- moved HS1 17.3 mm to (227.3, 104.1)
- moved R25 17.0 mm to (148.6, 82.5), turned to 180 degrees
- moved C13 16.5 mm to (151.1, 82.9)
- moved J1 7.52 mm to (131.9, 74.1)
- moved R1 5.08 mm to (176.6, 75.4)
- moved R21 5.08 mm to (185.5, 75.4)
- moved R23 5.08 mm to (182.6, 75.4)
- moved R22 5.08 mm to (179.6, 75.4)
- moved D1 4.14 mm to (181.9, 68.6)
- moved R19 3.47 mm to (161.6, 77.5)
- moved R20 3.37 mm to (164.7, 77.5)
- moved D2 2.99 mm to (181.9, 71.6)
- moved C10 2.86 mm to (145.6, 83.2)
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Connections:
- net /Connectors/TEMP_PCB renamed /TEMP_PCB
- C20 pad 1: /Motor Driver/+VCC_IO -> /+VCC_IO
- IC1 pad 10: /Motor Driver/ADC_I_v -> /ADC_I_v
- IC1 pad 15: /Motor Driver/+VCC_IO -> /+VCC_IO
- IC1 pad 16: /Motor Driver/+VCC_IO -> /+VCC_IO
- IC1 pad 19: /Motor Driver/+VCC_IO -> /+VCC_IO
- IC1 pad 26: /Fault -> /FAULT
- J1 pad 3: /Connectors/FAULT -> /FAULT
- J2 pad 1: /Connectors/+VCC_IO -> /+VCC_IO
- R16 pad 1: /Connectors/+VCC_IO -> /+VCC_IO
- R20 pad 2: /Connectors/FAULT -> /Connectors/FAULT_LED
- R21 pad 1: /Connectors/+VCC_IO -> /+VCC_IO
- R23 pad 1: /Connectors/+VCC_IO -> /+VCC_IO
