File: opm-inline/source/opm-inline.kicad_pcb (KiCad board)
At the start: 4 copper layers, 58 x 40 mm, 71 parts, among them IC1 TMC6200-TA, J1 Info, J2 VCC_IO, J3 PWMx6, J4 Fan, J6 Current Sensing, Q1 HYG025N06LS1C2, Q2 HYG025N06LS1C2, Q3 HYG025N06LS1C2, Q4 HYG025N06LS1C2, Q5 HYG025N06LS1C2, Q6 HYG025N06LS1C2, U2 TerminalBlock_2_P5.08mm, U3 TerminalBlock_3_P5.08mm

Commit message: rearrange
Parts:
- added D4: 10V, Diode_SMD:D_SOD-123, F.Cu at (169.4, 72.0)
- added Q7: WSD90P06DN56, Libraries:PDFN-8, F.Cu at (174.1, 69.8)
- added R27: 100KR, Resistor_SMD:R_0603_1608Metric, F.Cu at (172.2, 73.5)
- moved J2 55.1 mm to (132.7, 79.9)
- moved R21 44.9 mm to (141.7, 85.3), turned to 180 degrees
- moved R22 38.8 mm to (141.7, 83.8)
- moved D1 37.1 mm to (145.0, 68.3)
- moved D2 35.8 mm to (146.6, 68.3)
- moved U2 8.22 mm to (185.5, 69.8)
- moved R1 7.11 mm to (169.5, 75.2)
- moved J4 6.36 mm to (133.3, 95.2)
- moved H202 6.13 mm to (133.2, 88.5)
- moved HS1 4.83 mm to (241.0, 104.5)
- moved R20 4.13 mm to (158.3, 76.8), turned to 0 degrees
- moved H201 1.88 mm to (133.2, 103.3)
- moved R19 1.14 mm to (158.3, 78.5)
- moved C15 0.84 mm to (162.9, 73.7)
Connections:
- IC1 pad 3: GND -> Net-(IC1-Pad3)
- J4 pad 1: Net-(J4-Pad1) -> /+VCC_IO
- R6 pad 2: GND -> Net-(IC1-Pad3)
- U2 pad 2: /+VM -> Net-(Q7-Pad5)
Routing:
- net Net-(IC1-Pad37): track 0.00 -> 28.9 mm, vias 0 -> 2
- net /+VCC_IO: track 102.7 -> 79.5 mm
- net Net-(IC1-Pad3): track 0.00 -> 20.3 mm, vias 0 -> 2
- net /+VM: track 81.3 -> 61.7 mm, vias 42 -> 41
- net Net-(D1-Pad2): track 29.1 -> 19.4 mm
- net /Connectors/VOFS: track 10.5 -> 1.84 mm, vias 2 -> 0
- net Net-(IC1-Pad48): track 27.2 -> 19.0 mm
- net Net-(Q1-Pad4): track 3.16 -> 10.6 mm
- net Net-(D2-Pad2): track 22.0 -> 17.4 mm
- net Net-(D4-Pad1): track 0.00 -> 4.50 mm
- net Net-(IC1-Pad4): track 13.4 -> 16.8 mm
- net /U: track 26.6 -> 25.8 mm
- net GND: track 29.1 -> 29.9 mm, vias 36 -> 35
- net Net-(C4-Pad2): track 4.87 -> 5.37 mm
- added copper zone on B.Cu, net /+VM
- added copper zone on In1.Cu, net /+VM
- added copper zone on B.Cu, net /U
- added copper zone on B.Cu, net /V
- added copper zone on B.Cu, net /W
- added copper zone on B.Cu, net GND
- added copper zone on B.Cu, net Net-(C4-Pad1)
- added copper zone on B.Cu, net Net-(C5-Pad2)
- added copper zone on F.Cu, net Net-(Q7-Pad5)

Commit message: more routing
Routing:
- net GND: vias 35 -> 43
- net /+VM: vias 41 -> 40
Changed lines of the file:
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@@
     (thickness 1.6)
     (drawings 4)
-    (tracks 543)
+    (tracks 549)
     (zones 0)
     (modules 74)
@@
   (page A4)
   (layers
-    (0 F.Cu signal)
+    (0 F.Cu signal hide)
     (1 In1.Cu signal hide)
-    (2 In2.Cu signal hide)
+    (2 In2.Cu signal)
     (31 B.Cu mixed hide)
     (32 B.Adhes user)
@@
   (via (at 170.18 77.978) (size 0.6) (drill 0.3) (layers F.Cu B.Cu) (net 3))
   (via (at 171.45 78.74) (size 0.6) (drill 0.3) (layers F.Cu B.Cu) (net 3))
-  (via (at 161.29 85.09) (size 0.6) (drill 0.3) (layers F.Cu B.Cu) (net 3))
-  (via (at 166.37 84.32) (size 0.6) (drill 0.3) (layers F.Cu B.Cu) (net 3))
+  (via (at 161.925 84.963) (size 0.6) (drill 0.3) (layers F.Cu B.Cu) (net 3))
+  (via (at 166.37 84.582) (size 0.6) (drill 0.3) (layers F.Cu B.Cu) (net 3))
   (via (at 161.29 87.63) (size 0.6) (drill 0.3) (layers F.Cu B.Cu) (net 3))
-  (via (at 160.147 86.487) (size 0.6) (drill 0.3) (layers F.Cu B.Cu) (net 3))
-  (via (at 158.877 85.344) (size 0.6) (drill 0.3) (layers F.Cu B.Cu) (net 3))
-  (via (at 168.5 84.32) (size 0.6) (drill 0.3) (layers F.Cu B.Cu) (net 3))
-  (via (at 163.83 84.32) (size 0.6) (drill 0.3) (layers F.Cu B.Cu) (net 3))
+  (via (at 160.655 86.106) (size 0.6) (drill 0.3) (layers F.Cu B.Cu) (net 3))
+  (via (at 159.512 85.09) (size 0.6) (drill 0.3) (layers F.Cu B.Cu) (net 3))
+  (via (at 163.957 84.582) (size 0.6) (drill 0.3) (layers F.Cu B.Cu) (net 3))
   (via (at 162.56 86.36) (size 0.6) (drill 0.3) (layers F.Cu B.Cu) (net 3))
   (segment (start 152.4 73.66) (end 163.83 73.66) (width 4) (layer In2.Cu) (net 3) (status 40000))
@@
   (via (at 155.47 101.1) (size 0.6) (drill 0.3) (layers F.Cu B.Cu) (net 3))
   (via (at 154.2 101.1) (size 0.6) (drill 0.3) (layers F.Cu B.Cu) (net 3))
-  (via (at 158.75 87.63) (size 0.6) (drill 0.3) (layers F.Cu B.Cu) (net 3))
+  (via (at 159.385 87.63) (size 0.6) (drill 0.3) (layers F.Cu B.Cu) (net 3))
   (segment (start 152.654 78.296) (end 152.654 77.343) (width 0.6) (layer F.Cu) (net 3))
   (via (at 152.654 77.343) (size 0.6) (drill 0.3) (layers F.Cu B.Cu) (net 3))
@@
   (segment (start 177.419 90.166) (end 177.415 90.17) (width 0.2) (layer F.Cu) (net 5))
   (segment (start 177.419 89.027) (end 177.419 90.166) (width 0.2) (layer F.Cu) (net 5))
-  (via (at 161.036 92.964) (size 0.6) (drill 0.3) (layers F.Cu B.Cu) (net 5))
-  (via (at 163.068 92.964) (size 0.6) (drill 0.3) (layers F.Cu B.Cu) (net 5))
-  (via (at 162.052 93.726) (size 0.6) (drill 0.3) (layers F.Cu B.Cu) (net 5))
-  (via (at 163.068 94.615) (size 0.6) (drill 0.3) (layers F.Cu B.Cu) (net 5))
-  (via (at 167.259 82.35) (size 0.6) (drill 0.3) (layers F.Cu B.Cu) (net 5))
-  (via (at 168.402 82.35) (size 0.6) (drill 0.3) (layers F.Cu B.Cu) (net 5))
+  (via (at 160.782 92.837) (size 0.6) (drill 0.3) (layers F.Cu B.Cu) (net 5))
+  (via (at 163.068 93.091) (size 0.6) (drill 0.3) (layers F.Cu B.Cu) (net 5))
+  (via (at 162.306 93.853) (size 0.6) (drill 0.3) (layers F.Cu B.Cu) (net 5))
+  (via (at 162.941 94.869) (size 0.6) (drill 0.3) (layers F.Cu B.Cu) (net 5))
+  (via (at 167.132 82.55) (size 0.6) (drill 0.3) (layers F.Cu B.Cu) (net 5))
+  (via (at 168.529 82.55) (size 0.6) (drill 0.3) (layers F.Cu B.Cu) (net 5))
   (via (at 169.672 82.35) (size 0.6) (drill 0.3) (layers F.Cu B.Cu) (net 5))
-  (via (at 170.334 82.958) (size 0.6) (drill 0.3) (layers F.Cu B.Cu) (net 5))
-  (via (at 171.069 83.747) (size 0.6) (drill 0.3) (layers F.Cu B.Cu) (net 5))
+  (via (at 170.942 82.804) (size 0.6) (drill 0.3) (layers F.Cu B.Cu) (net 5))
+  (via (at 171.069 83.82) (size 0.6) (drill 0.3) (layers F.Cu B.Cu) (net 5))
   (via (at 153.416 81.026) (size 0.6) (drill 0.3) (layers F.Cu B.Cu) (net 5))
   (segment (start 153.416 82.108) (end 153.416 81.026) (width 0.6) (layer F.Cu) (net 5))
@@
   (via (at 136.017 77.978) (size 0.6) (drill 0.3) (layers F.Cu B.Cu) (net 5))
   (via (at 140.843 81.28) (size 0.6) (drill 0.3) (layers F.Cu B.Cu) (net 5))
+  (via (at 165.862 104.013) (size 0.6) (drill 0.3) (layers F.Cu B.Cu) (net 5))
+  (via (at 167.132 104.013) (size 0.6) (drill 0.3) (layers F.Cu B.Cu) (net 5))
+  (via (at 168.275 104.013) (size 0.6) (drill 0.3) (layers F.Cu B.Cu) (net 5))
+  (via (at 169.545 104.013) (size 0.6) (drill 0.3) (layers F.Cu B.Cu) (net 5))
+  (via (at 170.815 104.013) (size 0.6) (drill 0.3) (layers F.Cu B.Cu) (net 5))
+  (via (at 165.608 82.55) (size 0.6) (drill 0.3) (layers F.Cu B.Cu) (net 5))
+  (via (at 161.925 92.837) (size 0.6) (drill 0.3) (layers F.Cu B.Cu) (net 5))
+  (via (at 164.592 101.854) (size 0.6) (drill 0.3) (layers F.Cu B.Cu) (net 5))
   (via (at 159.004 101.092) (size 0.6) (drill 0.3) (layers F.Cu B.Cu) (net 21))
   (via (at 156.464 76.835) (size 0.6) (drill 0.3) (layers F.Cu B.Cu) (net 20))
@@
   (segment (start 163.092 98.83) (end 164.084 99.822) (width 0.6) (layer F.Cu) (net 13))
   (segment (start 162.94 98.83) (end 163.092 98.83) (width 0.2) (layer F.Cu) (net 13))
-  (segment (start 165.192001 100.930001) (end 164.084 99.822) (width 0.2) (layer In2.Cu) (net 13))
-  (segment (start 180.711997 100.930001) (end 165.192001 100.930001) (width 0.2) (layer In2.Cu) (net 13))
-  (segment (start 180.803998 100.838) (end 180.711997 100.930001) (width 0.2) (layer In2.Cu) (net 13))
-  (segment (start 184.023 100.838) (end 180.803998 100.838) (width 0.2) (layer In2.Cu) (net 13))
+  (segment (start 165.192001 100.930001) (end 164.084 99.822) (width 0.2) (layer B.Cu) (net 13))
+  (segment (start 183.930999 100.930001) (end 165.192001 100.930001) (width 0.2) (layer B.Cu) (net 13))
+  (segment (start 184.023 100.838) (end 183.930999 100.930001) (width 0.2) (layer B.Cu) (net 13))
   (segment (start 161.925 96.393) (end 162.052 96.52) (width 0.2) (layer F.Cu) (net 14))
   (via (at 174.625 92.456) (size 0.6) (drill 0.3) (layers F.Cu B.Cu) (net 14))

Commit message: more routing
Parts:
- added D3: SP0505BAJT, Package_TO_SOT_SMD:SOT-363_SC-70-6, F.Cu at (141.1, 92.6)
- added D5: SP0505BAJT, Package_TO_SOT_SMD:SOT-363_SC-70-6, F.Cu at (141.0, 89.7)
- added D6: TVS DIODE, Diode_SMD:D_SMA, F.Cu at (174.2, 74.5)
- moved HS1 11.1 mm to (233.7, 96.3)
- moved R1 7.47 mm to (162.4, 77.5)
- moved R27 3.58 mm to (169.0, 75.2), turned to 180 degrees
Routing:
- net Net-(Q1-Pad4): track 10.6 -> 17.8 mm, vias 0 -> 2
- net Net-(IC1-Pad48): track 19.0 -> 13.7 mm
- net /U: track 25.8 -> 27.2 mm
- net GND: track 29.9 -> 30.8 mm, vias 43 -> 44

Commit message: more routing
Connections:
- D3 pad 2: Net-(D3-Pad2) -> GND
- D5 pad 2: Net-(D5-Pad2) -> GND
Changed lines of the file:
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@@
     (zones 0)
     (modules 77)
-    (nets 58)
+    (nets 56)
   )
   (page A4)
@@
     (1 In1.Cu signal hide)
     (2 In2.Cu signal hide)
-    (31 B.Cu mixed hide)
+    (31 B.Cu mixed)
     (32 B.Adhes user)
     (33 F.Adhes user)
@@
   (net 52 /+VCC_IO)
   (net 53 /TEMP_PCB)
-  (net 54 "Net-(D3-Pad2)")
-  (net 55 "Net-(D4-Pad1)")
-  (net 56 "Net-(D5-Pad2)")
-  (net 57 "Net-(D6-Pad2)")
+  (net 54 "Net-(D4-Pad1)")
+  (net 55 "Net-(D6-Pad2)")
   (net_class Default "This is the default net class."
     (clearance 0.2)
@@
     (add_net "Net-(D1-Pad2)")
     (add_net "Net-(D2-Pad2)")
-    (add_net "Net-(D3-Pad2)")
     (add_net "Net-(D4-Pad1)")
-    (add_net "Net-(D5-Pad2)")
     (add_net "Net-(D6-Pad2)")
     (add_net "Net-(IC1-Pad24)")
@@
       (net 5 GND))
     (pad 2 thru_hole circle (at 5.08 0 180) (size 3 3) (drill 1.52) (layers *.Cu *.Mask)
-      (net 57 "Net-(D6-Pad2)"))
+      (net 55 "Net-(D6-Pad2)"))
     (model ${KISYS3DMOD}/TerminalBlock_Phoenix.3dshapes/TerminalBlock_Phoenix_MKDS-1,5-2-5.08_1x02_P5.08mm_Horizontal.wrl
       (at (xyz 0 0 0))
@@
       (net 3 /+VM))
     (pad 4 smd rect (at -2.9 1.905) (size 0.85 0.5) (layers F.Cu F.Mask)
-      (net 55 "Net-(D4-Pad1)"))
+      (net 54 "Net-(D4-Pad1)"))
     (pad 2 smd rect (at -2.9 -0.635) (size 0.85 0.5) (layers F.Cu F.Mask)
       (net 3 /+VM))
@@
       (net 3 /+VM))
     (pad 5 smd rect (at 2.925 1.905) (size 0.8 0.6) (layers F.Cu F.Mask)
-      (net 57 "Net-(D6-Pad2)"))
+      (net 55 "Net-(D6-Pad2)"))
     (pad 6 smd rect (at 2.925 0.635) (size 0.8 0.6) (layers F.Cu F.Mask)
-      (net 57 "Net-(D6-Pad2)"))
+      (net 55 "Net-(D6-Pad2)"))
     (pad 7 smd rect (at 2.925 -0.635) (size 0.8 0.6) (layers F.Cu F.Mask)
-      (net 57 "Net-(D6-Pad2)"))
+      (net 55 "Net-(D6-Pad2)"))
     (pad 8 smd rect (at 2.925 -1.905) (size 0.8 0.6) (layers F.Cu F.Mask)
-      (net 57 "Net-(D6-Pad2)"))
+      (net 55 "Net-(D6-Pad2)"))
     (pad 5 smd rect (at 0.65 0) (size 3.75 4.41) (layers F.Cu F.Mask)
-      (net 57 "Net-(D6-Pad2)"))
+      (net 55 "Net-(D6-Pad2)"))
     (model ${KISYS3DMOD}/Package_DFN_QFN.3dshapes/DFN-8-1EP_6x5mm_Pitch1.27mm.wrl
       (at (xyz 0 0 0))
@@
     )
     (pad 1 smd rect (at -1.65 0 90) (size 0.9 1.2) (layers F.Cu F.Paste F.Mask)
-      (net 55 "Net-(D4-Pad1)"))
+      (net 54 "Net-(D4-Pad1)"))
     (pad 2 smd rect (at 1.65 0 90) (size 0.9 1.2) (layers F.Cu F.Paste F.Mask)
       (net 3 /+VM))
@@
     )
     (pad 1 smd roundrect (at -0.825 0 180) (size 0.8 0.95) (layers F.Cu F.Paste F.Mask) (roundrect_rratio 0.25)
-      (net 55 "Net-(D4-Pad1)"))
+      (net 54 "Net-(D4-Pad1)"))
     (pad 2 smd roundrect (at 0.825 0 180) (size 0.8 0.95) (layers F.Cu F.Paste F.Mask) (roundrect_rratio 0.25)
       (net 5 GND))
@@
       (net 29 /VL))
     (pad 2 smd rect (at -0.95 0) (size 0.65 0.4) (layers F.Cu F.Paste F.Mask)
-      (net 54 "Net-(D3-Pad2)"))
+      (net 5 GND))
     (pad 5 smd rect (at 0.95 0) (size 0.65 0.4) (layers F.Cu F.Paste F.Mask)
       (net 30 /WH))
@@
       (net 34 /DRV_EN))
     (pad 2 smd rect (at -0.95 0) (size 0.65 0.4) (layers F.Cu F.Paste F.Mask)
-      (net 56 "Net-(D5-Pad2)"))
+      (net 5 GND))
     (pad 4 smd rect (at 0.95 0.65) (size 0.65 0.4) (layers F.Cu F.Paste F.Mask)
       (net 53 /TEMP_PCB))
@@
       (net 5 GND))
     (pad 2 smd rect (at 2 0 180) (size 2.5 1.8) (layers F.Cu F.Paste F.Mask)
-      (net 57 "Net-(D6-Pad2)"))
+      (net 55 "Net-(D6-Pad2)"))
     (model ${KISYS3DMOD}/Diode_SMD.3dshapes/D_SMA.wrl
       (at (xyz 0 0 0))
@@
   (via (at 177.419 89.027) (size 0.6) (drill 0.3) (layers F.Cu B.Cu) (net 5))
   (segment (start 177.419 90.166) (end 177.415 90.17) (width 0.2) (layer F.Cu) (net 5))
-  (segment (start 177.419 89.027) (end 177.419 90.166) (width 0.2) (layer F.Cu) (net 5))
+  (segment (start 177.419 89.027) (end 177.419 90.166) (width 0.6) (layer F.Cu) (net 5))
   (via (at 160.782 92.837) (size 0.6) (drill 0.3) (layers F.Cu B.Cu) (net 5))
   (via (at 163.068 93.091) (size 0.6) (drill 0.3) (layers F.Cu B.Cu) (net 5))
@@
   (segment (start 147.574 77.089) (end 146.939 77.724) (width 0.2) (layer F.Cu) (net 53))
   (segment (start 148.082 77.089) (end 147.574 77.089) (width 0.2) (layer F.Cu) (net 53))
-  (segment (start 171.217 71.86) (end 169.418 73.659) (width 0.2) (layer F.Cu) (net 55))
-  (segment (start 171.217 71.755) (end 171.217 71.86) (width 0.2) (layer F.Cu) (net 55))
-  (segment (start 169.368 74.69) (end 169.862 75.184) (width 0.2) (layer F.Cu) (net 55))
-  (segment (start 169.368 73.659) (end 169.368 74.69) (width 0.2) (layer F.Cu) (net 55))
+  (segment (start 171.217 71.86) (end 169.418 73.659) (width 0.2) (layer F.Cu) (net 54))
+  (segment (start 171.217 71.755) (end 171.217 71.86) (width 0.2) (layer F.Cu) (net 54))
+  (segment (start 169.368 74.69) (end 169.862 75.184) (width 0.2) (layer F.Cu) (net 54))
+  (segment (start 169.368 73.659) (end 169.368 74.69) (width 0.2) (layer F.Cu) (net 54))
   (zone (net 15) (net_name /U) (layer F.Cu) (hatch edge 0.508)
     (priority 2)
@@
     )
   )
-  (zone (net 57) (net_name "Net-(D6-Pad2)") (layer F.Cu) (hatch edge 0.508)
+  (zone (net 55) (net_name "Net-(D6-Pad2)") (layer F.Cu) (hatch edge 0.508)
     (priority 1)
     (connect_pads yes (clearance 0.508))

Commit message: esd
Parts:
- added D7: NUP4114UCW1T2G, Libraries:NUP4114UCW1T2G, F.Cu at (143.9, 79.0)
- D3, D5: value SP0505BAJT -> NUP4114UCW1T2G; footprint Package_TO_SOT_SMD:SOT-363_SC-70-6 -> Libraries:NUP4114UCW1T2G
Connections:
- J6 pad 1: /ADC_I_u -> /ADC_I_w
- J6 pad 3: /ADC_I_w -> /ADC_I_u

Commit message: esd
Parts:
- moved D3 13.8 mm to (139.8, 78.9)
- moved D5 11.8 mm to (136.5, 78.7)
- moved J6 4.42 mm to (140.5, 74.2), turned to 0 degrees
- moved D7 0.81 mm to (144.5, 79.5), turned to 0 degrees
Connections:
- D3 pad 1: /UL -> /WH
- D3 pad 5: /WH -> /UL
- D3 pad 6: /WL -> /UH
- D5 pad 6: /UH -> /WL
Routing:
- net /ADC_I_v: track 14.7 -> 18.2 mm
- net /UL: track 27.2 -> 23.7 mm, vias 1 -> 2
- net /ADC_I_w: track 15.3 -> 17.0 mm
- net /ADC_I_u: track 14.0 -> 15.5 mm
- net GND: track 30.8 -> 31.7 mm
- net /UH: track 26.9 -> 27.6 mm, vias 1 -> 3

Commit message: esd
Routing:
- net /UL: track 23.7 -> 28.3 mm, vias 2 -> 3
Changed lines of the file:
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@@
     (thickness 1.6)
     (drawings 4)
-    (tracks 592)
+    (tracks 600)
     (zones 0)
     (modules 78)
@@
   (via (at 160.147 76.835) (size 0.6) (drill 0.3) (layers F.Cu B.Cu) (net 5))
   (segment (start 159.13 76.835) (end 160.147 76.835) (width 0.6) (layer F.Cu) (net 5))
-  (via (at 136.017 77.978) (size 0.6) (drill 0.3) (layers F.Cu B.Cu) (net 5))
-  (via (at 140.843 81.28) (size 0.6) (drill 0.3) (layers F.Cu B.Cu) (net 5))
+  (via (at 135.636 85.09) (size 0.6) (drill 0.3) (layers F.Cu B.Cu) (net 5))
+  (via (at 142.367 79.502) (size 0.6) (drill 0.3) (layers F.Cu B.Cu) (net 5))
   (via (at 165.862 104.013) (size 0.6) (drill 0.3) (layers F.Cu B.Cu) (net 5))
   (via (at 167.132 104.013) (size 0.6) (drill 0.3) (layers F.Cu B.Cu) (net 5))
@@
   (segment (start 146.76 88.19) (end 146.685 88.265) (width 0.2) (layer F.Cu) (net 5))
   (segment (start 147.9117 88.19) (end 146.76 88.19) (width 0.2) (layer F.Cu) (net 5))
+  (via (at 140.97 80.264) (size 0.6) (drill 0.3) (layers F.Cu B.Cu) (net 27))
   (via (at 140.843 77.47) (size 0.6) (drill 0.3) (layers F.Cu B.Cu) (net 26))
   (via (at 141.605 78.232) (size 0.6) (drill 0.3) (layers F.Cu B.Cu) (net 26))
@@
   (segment (start 147.891701 90.17) (end 147.9117 90.189999) (width 0.2) (layer F.Cu) (net 26))
   (segment (start 141.88 68.58) (end 141.88 68.94) (width 0.2) (layer F.Cu) (net 26))
-  (segment (start 141.605 83.947) (end 141.605 78.232) (width 0.2) (layer B.Cu) (net 26))
   (segment (start 141.589999 78.216999) (end 141.605 78.232) (width 0.2) (layer F.Cu) (net 26))
   (segment (start 140.776998 78.216999) (end 141.589999 78.216999) (width 0.2) (layer F.Cu) (net 26))
@@
   (segment (start 145.415 87.884) (end 146.050001 88.519001) (width 0.2) (layer F.Cu) (net 26))
   (segment (start 141.605 84.074) (end 141.605 83.947) (width 0.2) (layer B.Cu) (net 26))
-  (segment (start 145.415 87.884) (end 141.605 84.074) (width 0.2) (layer B.Cu) (net 26))
+  (segment (start 141.605 84.074) (end 142.0495 84.5185) (width 0.2) (layer B.Cu) (net 26))
+  (segment (start 141.605 78.232) (end 141.605 84.074) (width 0.2) (layer B.Cu) (net 26))
+  (segment (start 145.415 87.884) (end 142.0495 84.5185) (width 0.2) (layer B.Cu) (net 26))
   (segment (start 146.37 90.69) (end 147.9117 90.69) (width 0.2) (layer F.Cu) (net 27))
   (segment (start 145.45 89.77) (end 146.37 90.69) (width 0.2) (layer F.Cu) (net 27))
-  (segment (start 139.7 84.02) (end 145.45 89.77) (width 0.2) (layer B.Cu) (net 27))
-  (segment (start 138.83001 83.15001) (end 139.7 84.02) (width 0.2) (layer B.Cu) (net 27))
   (segment (start 139.19398 69.26602) (end 139.88 68.58) (width 0.2) (layer B.Cu) (net 27))
   (segment (start 139.19398 76.58298) (end 139.19398 69.26602) (width 0.2) (layer B.Cu) (net 27))
@@
   (segment (start 140.326999 78.866999) (end 140.081 78.621) (width 0.2) (layer F.Cu) (net 27))
   (segment (start 140.776998 78.866999) (end 140.326999 78.866999) (width 0.2) (layer F.Cu) (net 27))
+  (segment (start 141.116999 78.866999) (end 141.326999 79.076999) (width 0.2) (layer F.Cu) (net 27))
+  (segment (start 140.776998 78.866999) (end 141.116999 78.866999) (width 0.2) (layer F.Cu) (net 27))
+  (segment (start 140.97 80.264) (end 141.326999 79.907001) (width 0.2) (layer F.Cu) (net 27))
+  (segment (start 141.326999 79.076999) (end 141.326999 79.907001) (width 0.2) (layer F.Cu) (net 27))
+  (segment (start 140.242999 84.562999) (end 141.1875 85.5075) (width 0.2) (layer B.Cu) (net 27))
+  (segment (start 140.242999 80.991001) (end 140.242999 84.562999) (width 0.2) (layer B.Cu) (net 27))
+  (segment (start 140.97 80.264) (end 140.242999 80.991001) (width 0.2) (layer B.Cu) (net 27))
+  (segment (start 145.45 89.77) (end 141.1875 85.5075) (width 0.2) (layer B.Cu) (net 27))
   (segment (start 147.9117 91.690001) (end 147.570001 91.690001) (width 0.2) (layer F.Cu) (net 28))
   (via (at 146.4843 91.69) (size 0.6) (drill 0.3) (layers F.Cu B.Cu) (net 28))

Commit message: esd
Parts:
- moved D5 0.28 mm to (136.3, 78.9)
Connections:
- D3 pad 3: /VH -> /VL
- D3 pad 4: /VL -> /VH
- D5 pad 1: /+VCC_IO -> /FAULT
- D5 pad 3: GND -> /+VCC_IO
- D5 pad 4: /TEMP_PCB -> /DRV_EN
- D5 pad 5: /DRV_EN -> /WL
- D5 pad 6: /WL -> /TEMP_PCB
- IC1 pad 26: GND -> /FAULT
- J1 pad 3: GND -> /FAULT
- R20 pad 2: GND -> /FAULT
Routing:
- net /FAULT: track 0.00 -> 62.8 mm, vias 0 -> 4
- net /+VCC_IO: track 79.5 -> 63.8 mm, vias 0 -> 2
- net /TEMP_PCB: track 36.4 -> 42.5 mm
- net /DRV_EN: track 35.2 -> 37.1 mm, vias 1 -> 2
- net /WH: track 31.0 -> 32.6 mm, vias 1 -> 2
- net /WL: track 33.5 -> 34.8 mm, vias 1 -> 2
- net /VH: track 29.7 -> 30.9 mm, vias 1 -> 2
- net /UL: track 28.3 -> 27.4 mm, vias 3 -> 2
- net /VL: track 30.6 -> 30.0 mm, vias 1 -> 2
- net GND: track 31.7 -> 31.2 mm, vias 44 -> 48
- net /UH: track 27.7 -> 27.5 mm, vias 3 -> 2
