File: opm-inline/source/opm-inline.sch (KiCad schematic (older format))
At the start: 0 parts

Commit message: update connections
Connections:
- no-connect marks 1 -> 0
Changed lines of the file:
@@
 	7150 3550 7250 3550
 Wire Wire Line
-	7150 3650 7250 3650
-Wire Wire Line
 	6150 2950 6050 2950
 Wire Wire Line
-	6050 3150 6150 3150
-Wire Wire Line
 	6050 3250 6150 3250
 Wire Wire Line
 	6050 3350 6150 3350
 Wire Wire Line
-	6150 3450 6050 3450
-Wire Wire Line
-	6050 3550 6150 3550
-Wire Wire Line
-	6050 3650 6150 3650
-Wire Wire Line
 	6050 3750 6150 3750
 Wire Wire Line
@@
 	5250 2950 5150 2950
 Wire Wire Line
-	5150 3050 5250 3050
-Wire Wire Line
-	5150 3150 5250 3150
-Wire Wire Line
 	5150 3250 5250 3250
 Wire Wire Line
@@
 	5150 3750 5250 3750
 Wire Wire Line
-	5150 3850 5250 3850
-Wire Wire Line
 	5250 3950 5150 3950
 Wire Wire Line
-	5150 4050 5250 4050
-Wire Wire Line
-	5150 4150 5250 4150
-Wire Wire Line
 	5150 4250 5250 4250
 Wire Wire Line
@@
 Wire Wire Line
 	4050 3150 4150 3150
-Wire Wire Line
-	4050 3250 4150 3250
 Wire Wire Line
 	4050 3350 4150 3350
 Text Label 6050 3050 2    39   ~ 0
-+Vcc_IO
++VCC_IO
 Text Label 4050 3350 2    39   ~ 0
-+Vcc_IO
-Text Label 6050 3150 2    39   ~ 0
-+5V_VM
-Text Label 5250 3150 0    39   ~ 0
-+5V_VM
-NoConn ~ 5250 3050
++VCC_IO
 Text Label 5250 2950 0    39   ~ 0
 +VM
@@
 ADC_I_w
 Text Label 7250 3550 0    39   ~ 0
-Fault
+FAULT
 Text Label 5250 3550 0    39   ~ 0
 UH
@@
 Text Label 4050 3150 2    39   ~ 0
 ADC_I_w
-Text Label 5250 3850 0    39   ~ 0
-~CS_DRIVER
-Text Label 6050 3450 2    39   ~ 0
-~CS_DRIVER
 Text Label 6050 3250 2    39   ~ 0
 DRV_EN
 Text Label 5250 3950 0    39   ~ 0
 DRV_EN
-Text Label 5250 4050 0    39   ~ 0
-SPI1_MOSI
-Text Label 6050 3650 2    39   ~ 0
-SPI1_MOSI
-Text Label 6050 3550 2    39   ~ 0
-SPI1_SCK
-Text Label 5250 4150 0    39   ~ 0
-SPI1_SCK
-Text Label 4050 3250 2    39   ~ 0
-SPI1_MISO
-Text Label 7250 3650 0    39   ~ 0
-SPI1_MISO
 Text Label 5250 4550 0    39   ~ 0
 SPE
 Text Label 6050 3350 2    39   ~ 0
 SPE
-Text Label 4050 3900 2    39   ~ 0
-+3,3V
-Wire Wire Line
-	4050 3900 4150 3900
 Wire Wire Line
 	4050 3800 4150 3800
@@
 	4150 3500 4050 3500
 Wire Wire Line
-	4150 3700 4050 3700
-Wire Wire Line
 	7150 3850 7250 3850
 Wire Wire Line
@@
 Wire Wire Line
 	7150 4050 7250 4050
-Wire Wire Line
-	7150 4150 7250 4150
 Text Label 7250 3850 0    39   ~ 0
 VSA
@@
 Text Label 7250 4050 0    39   ~ 0
 5Vout
-Text Label 7250 4150 0    39   ~ 0
-VCP
 Text Label 4050 3500 2    39   ~ 0
 VSA
@@
 Text Label 4050 3800 2    39   ~ 0
 5Vout
-Text Label 4050 3700 2    39   ~ 0
-VCP
 Wire Wire Line
 	4150 3050 4050 3050
 Text Label 4050 3050 2    39   ~ 0
 ADC_I_v
-$Sheet
-S 4150 2850 1000 2000
-U 5BA8C4E4
-F0 "Connectors" 39
-F1 "Connectors.sch" 39
-F2 "+VM" O R 5150 2950 39
-F3 "+5V_USB" O R 5150 3050 39
-F4 "+5V_VM" O R 5150 3150 39
-F5 "W" B R 5150 3450 39
-F6 "V" B R 5150 3350 39
-F7 "U" B R 5150 3250 39
-F8 "ADC_I_w" I L 4150 3150 39
-F9 "UH" O R 5150 3550 39
-F10 "VH" O R 5150 3650 39
-F11 "WH" O R 5150 3750 39
-F12 "~CS_DRIVER" O R 5150 3850 39
-F13 "SPI1_MISO" I L 4150 3250 39
-F14 "DRV_EN" O R 5150 3950 39
-F15 "SPI1_MOSI" O R 5150 4050 39
-F16 "SPI1_SCK" O R 5150 4150 39
-F17 "WL" O R 5150 4450 39
-F18 "VL" O R 5150 4350 39
-F19 "UL" O R 5150 4250 39
-F20 "ADC_I_u" I L 4150 2950 39
-F21 "SPE" O R 5150 4550 39
-F22 "+Vcc_IO" I L 4150 3350 39
-F23 "VSA" I L 4150 3500 39
-F24 "12Vout" I L 4150 3600 39
-F25 "VCP" I L 4150 3700 39
-F26 "5Vout" I L 4150 3800 39
-F27 "+3,3V" I L 4150 3900 39
-F28 "ADC_I_v" I L 4150 3050 39
-F29 "VCC" I L 4150 4400 28
-$EndSheet
 $Sheet
 S 6150 2850 1000 2000
@@
 F6 "DRV_EN" I L 6150 3250 39
 F7 "SPE" I L 6150 3350 39
-F8 "SPI1_SCK" I L 6150 3550 39
-F9 "SPI1_MOSI" I L 6150 3650 39
-F10 "SPI1_MISO" O R 7150 3650 39
-F11 "UH" I L 6150 3750 39
-F12 "UL" I L 6150 3850 39
-F13 "VH" I L 6150 3950 39
-F14 "VL" I L 6150 4050 39
-F15 "WH" I L 6150 4150 39
-F16 "WL" I L 6150 4250 39
-F17 "+Vcc_IO" I L 6150 3050 39
-F18 "~CS_DRIVER" I L 6150 3450 39
-F19 "+5V_VM" I L 6150 3150 39
-F20 "U" B R 7150 2950 39
-F21 "V" B R 7150 3050 39
-F22 "W" B R 7150 3150 39
-F23 "VSA" O R 7150 3850 39
-F24 "12Vout" O R 7150 3950 39
-F25 "5Vout" O R 7150 4050 39
-F26 "VCP" O R 7150 4150 39
+F8 "UH" I L 6150 3750 39
+F9 "UL" I L 6150 3850 39
+F10 "VH" I L 6150 3950 39
+F11 "VL" I L 6150 4050 39
+F12 "WH" I L 6150 4150 39
+F13 "WL" I L 6150 4250 39
+F14 "+VCC_IO" I L 6150 3050 39
+F15 "U" B R 7150 2950 39
+F16 "V" B R 7150 3050 39
+F17 "W" B R 7150 3150 39
+F18 "VSA" O R 7150 3850 39
+F19 "12Vout" O R 7150 3950 39
+F20 "5Vout" O R 7150 4050 39
 $EndSheet
+Wire Wire Line
+	7150 3350 7250 3350
+Text Label 7250 3350 0    39   ~ 0
+ADC_I_v
+Text HLabel 7150 3350 0    39   Input ~ 0
+ADC_I_v
+Text Label 5250 4050 0    39   ~ 0
+FAULT
+$Sheet
+S 4150 2850 1000 2000
+U 5BA8C4E4
+F0 "Connectors" 39
+F1 "Connectors.sch" 39
+F2 "+VM" O R 5150 2950 39
+F3 "W" B R 5150 3450 39
+F4 "V" B R 5150 3350 39
+F5 "U" B R 5150 3250 39
+F6 "ADC_I_w" I L 4150 3150 39
+F7 "UH" O R 5150 3550 39
+F8 "VH" O R 5150 3650 39
+F9 "WH" O R 5150 3750 39
+F10 "DRV_EN" O R 5150 3950 39
+F11 "WL" O R 5150 4450 39
+F12 "VL" O R 5150 4350 39
+F13 "UL" O R 5150 4250 39
+F14 "ADC_I_u" I L 4150 2950 39
+F15 "SPE" O R 5150 4550 39
+F16 "+VCC_IO" I L 4150 3350 39
+F17 "VSA" I L 4150 3500 39
+F18 "12Vout" I L 4150 3600 39
+F19 "5Vout" I L 4150 3800 39
+F20 "ADC_I_v" I L 4150 3050 39
+$EndSheet
+Text HLabel 5150 4050 0    39   Input ~ 0
+FAULT
+Wire Wire Line
+	5150 4050 5250 4050
+Text HLabel 5150 4150 0    39   Input ~ 0
+TEMP_PCB
+Text Label 5250 4150 0    39   ~ 0
+TEMP_PCB
+Wire Wire Line
+	5150 4150 5250 4150
 $EndSCHEMATC

Commit message: rearrange
Changed lines of the file:
@@
 F19 "12Vout" O R 7150 3950 39
 F20 "5Vout" O R 7150 4050 39
+F21 "ADC_I_v" O R 7150 3350 39
 $EndSheet
 Wire Wire Line
 	7150 3350 7250 3350
 Text Label 7250 3350 0    39   ~ 0
-ADC_I_v
-Text HLabel 7150 3350 0    39   Input ~ 0
 ADC_I_v
 Text Label 5250 4050 0    39   ~ 0
@@
 F19 "5Vout" I L 4150 3800 39
 F20 "ADC_I_v" I L 4150 3050 39
+F21 "TEMP_PCB" O R 5150 4150 39
+F22 "FAULT" O R 5150 4050 39
 $EndSheet
-Text HLabel 5150 4050 0    39   Input ~ 0
-FAULT
 Wire Wire Line
 	5150 4050 5250 4050
-Text HLabel 5150 4150 0    39   Input ~ 0
-TEMP_PCB
 Text Label 5250 4150 0    39   ~ 0
 TEMP_PCB
