File: opm-inline/source/MotorDriver.kicad_sch (KiCad schematic)
At the start: 44 parts, among them IC1 TMC6200-TA, Q1 HYG025N06LS1C2, Q2 HYG025N06LS1C2, Q3 HYG025N06LS1C2, Q4 HYG025N06LS1C2, Q5 HYG025N06LS1C2, Q6 HYG025N06LS1C2

Commit message: remove files
Parts:
- C21, C22, C23, C24, C25, C26, C7, C8, C9: LCSC C385977 -> C338074; manf_num   HMK212BC7105KGHTE -> CGA4J3X7S2A105KT0Y0N
Changed lines of the file:
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@@
       (effects (font (size 1.27 1.27)) hide)
     )
-    (property "Datasheet" "https://datasheet.lcsc.com/lcsc/2105241210_Taiyo-Yuden-HMK212BC7105KGHTE_C385977.pdf" (id 3) (at 195.58 111.76 0)
-      (effects (font (size 1.27 1.27)) hide)
-    )
-    (property "LCSC" "C385977" (id 4) (at 195.58 111.76 0)
-      (effects (font (size 1.27 1.27)) hide)
-    )
-    (property "manf_num  " "HMK212BC7105KGHTE" (id 5) (at 195.58 111.76 0)
+    (property "Datasheet" "https://datasheet.lcsc.com/lcsc/1912111437_TDK-CGA4J3X7S2A105KT0Y0N_C338074.pdf" (id 3) (at 195.58 111.76 0)
+      (effects (font (size 1.27 1.27)) hide)
+    )
+    (property "LCSC" "C338074" (id 4) (at 195.58 111.76 0)
+      (effects (font (size 1.27 1.27)) hide)
+    )
+    (property "manf_num  " "CGA4J3X7S2A105KT0Y0N" (id 5) (at 195.58 111.76 0)
       (effects (font (size 1.27 1.27)) hide)
     )
@@
       (effects (font (size 1.27 1.27)) hide)
     )
-    (property "Datasheet" "https://datasheet.lcsc.com/lcsc/2105241210_Taiyo-Yuden-HMK212BC7105KGHTE_C385977.pdf" (id 3) (at 209.55 36.83 0)
-      (effects (font (size 1.27 1.27)) hide)
-    )
-    (property "LCSC" "C385977" (id 4) (at 209.55 36.83 0)
-      (effects (font (size 1.27 1.27)) hide)
-    )
-    (property "manf_num  " "HMK212BC7105KGHTE" (id 5) (at 209.55 36.83 0)
+    (property "Datasheet" "https://datasheet.lcsc.com/lcsc/1912111437_TDK-CGA4J3X7S2A105KT0Y0N_C338074.pdf" (id 3) (at 209.55 36.83 0)
+      (effects (font (size 1.27 1.27)) hide)
+    )
+    (property "LCSC" "C338074" (id 4) (at 209.55 36.83 0)
+      (effects (font (size 1.27 1.27)) hide)
+    )
+    (property "manf_num  " "CGA4J3X7S2A105KT0Y0N" (id 5) (at 209.55 36.83 0)
       (effects (font (size 1.27 1.27)) hide)
     )
@@
       (effects (font (size 1.27 1.27)) hide)
     )
-    (property "Datasheet" "https://datasheet.lcsc.com/lcsc/2105241210_Taiyo-Yuden-HMK212BC7105KGHTE_C385977.pdf" (id 3) (at 223.52 36.83 0)
-      (effects (font (size 1.27 1.27)) hide)
-    )
-    (property "LCSC" "C385977" (id 4) (at 223.52 36.83 0)
-      (effects (font (size 1.27 1.27)) hide)
-    )
-    (property "manf_num  " "HMK212BC7105KGHTE" (id 5) (at 223.52 36.83 0)
+    (property "Datasheet" "https://datasheet.lcsc.com/lcsc/1912111437_TDK-CGA4J3X7S2A105KT0Y0N_C338074.pdf" (id 3) (at 223.52 36.83 0)
+      (effects (font (size 1.27 1.27)) hide)
+    )
+    (property "LCSC" "C338074" (id 4) (at 223.52 36.83 0)
+      (effects (font (size 1.27 1.27)) hide)
+    )
+    (property "manf_num  " "CGA4J3X7S2A105KT0Y0N" (id 5) (at 223.52 36.83 0)
       (effects (font (size 1.27 1.27)) hide)
     )
@@
       (effects (font (size 1.27 1.27)) hide)
     )
-    (property "Datasheet" "https://datasheet.lcsc.com/lcsc/2105241210_Taiyo-Yuden-HMK212BC7105KGHTE_C385977.pdf" (id 3) (at 237.49 71.12 0)
-      (effects (font (size 1.27 1.27)) hide)
-    )
-    (property "LCSC" "C385977" (id 4) (at 237.49 71.12 0)
-      (effects (font (size 1.27 1.27)) hide)
-    )
-    (property "manf_num  " "HMK212BC7105KGHTE" (id 5) (at 237.49 71.12 0)
+    (property "Datasheet" "https://datasheet.lcsc.com/lcsc/1912111437_TDK-CGA4J3X7S2A105KT0Y0N_C338074.pdf" (id 3) (at 237.49 71.12 0)
+      (effects (font (size 1.27 1.27)) hide)
+    )
+    (property "LCSC" "C338074" (id 4) (at 237.49 71.12 0)
+      (effects (font (size 1.27 1.27)) hide)
+    )
+    (property "manf_num  " "CGA4J3X7S2A105KT0Y0N" (id 5) (at 237.49 71.12 0)
       (effects (font (size 1.27 1.27)) hide)
     )
@@
       (effects (font (size 1.27 1.27)) hide)
     )
-    (property "Datasheet" "https://datasheet.lcsc.com/lcsc/2105241210_Taiyo-Yuden-HMK212BC7105KGHTE_C385977.pdf" (id 3) (at 195.58 36.83 0)
-      (effects (font (size 1.27 1.27)) hide)
-    )
-    (property "LCSC" "C385977" (id 4) (at 195.58 36.83 0)
-      (effects (font (size 1.27 1.27)) hide)
-    )
-    (property "manf_num  " "HMK212BC7105KGHTE" (id 5) (at 195.58 36.83 0)
+    (property "Datasheet" "https://datasheet.lcsc.com/lcsc/1912111437_TDK-CGA4J3X7S2A105KT0Y0N_C338074.pdf" (id 3) (at 195.58 36.83 0)
+      (effects (font (size 1.27 1.27)) hide)
+    )
+    (property "LCSC" "C338074" (id 4) (at 195.58 36.83 0)
+      (effects (font (size 1.27 1.27)) hide)
+    )
+    (property "manf_num  " "CGA4J3X7S2A105KT0Y0N" (id 5) (at 195.58 36.83 0)
       (effects (font (size 1.27 1.27)) hide)
     )
@@
       (effects (font (size 1.27 1.27)) hide)
     )
-    (property "Datasheet" "https://datasheet.lcsc.com/lcsc/2105241210_Taiyo-Yuden-HMK212BC7105KGHTE_C385977.pdf" (id 3) (at 251.46 71.12 0)
-      (effects (font (size 1.27 1.27)) hide)
-    )
-    (property "LCSC" "C385977" (id 4) (at 251.46 71.12 0)
-      (effects (font (size 1.27 1.27)) hide)
-    )
-    (property "manf_num  " "HMK212BC7105KGHTE" (id 5) (at 251.46 71.12 0)
+    (property "Datasheet" "https://datasheet.lcsc.com/lcsc/1912111437_TDK-CGA4J3X7S2A105KT0Y0N_C338074.pdf" (id 3) (at 251.46 71.12 0)
+      (effects (font (size 1.27 1.27)) hide)
+    )
+    (property "LCSC" "C338074" (id 4) (at 251.46 71.12 0)
+      (effects (font (size 1.27 1.27)) hide)
+    )
+    (property "manf_num  " "CGA4J3X7S2A105KT0Y0N" (id 5) (at 251.46 71.12 0)
       (effects (font (size 1.27 1.27)) hide)
     )
@@
       (effects (font (size 1.27 1.27)) hide)
     )
-    (property "Datasheet" "https://datasheet.lcsc.com/lcsc/2105241210_Taiyo-Yuden-HMK212BC7105KGHTE_C385977.pdf" (id 3) (at 266.7 71.12 0)
-      (effects (font (size 1.27 1.27)) hide)
-    )
-    (property "LCSC" "C385977" (id 4) (at 266.7 71.12 0)
-      (effects (font (size 1.27 1.27)) hide)
-    )
-    (property "manf_num  " "HMK212BC7105KGHTE" (id 5) (at 266.7 71.12 0)
+    (property "Datasheet" "https://datasheet.lcsc.com/lcsc/1912111437_TDK-CGA4J3X7S2A105KT0Y0N_C338074.pdf" (id 3) (at 266.7 71.12 0)
+      (effects (font (size 1.27 1.27)) hide)
+    )
+    (property "LCSC" "C338074" (id 4) (at 266.7 71.12 0)
+      (effects (font (size 1.27 1.27)) hide)
+    )
+    (property "manf_num  " "CGA4J3X7S2A105KT0Y0N" (id 5) (at 266.7 71.12 0)
       (effects (font (size 1.27 1.27)) hide)
     )
@@
       (effects (font (size 1.27 1.27)) hide)
     )
-    (property "Datasheet" "https://datasheet.lcsc.com/lcsc/2105241210_Taiyo-Yuden-HMK212BC7105KGHTE_C385977.pdf" (id 3) (at 209.55 111.76 0)
-      (effects (font (size 1.27 1.27)) hide)
-    )
-    (property "LCSC" "C385977" (id 4) (at 209.55 111.76 0)
-      (effects (font (size 1.27 1.27)) hide)
-    )
-    (property "manf_num  " "HMK212BC7105KGHTE" (id 5) (at 209.55 111.76 0)
+    (property "Datasheet" "https://datasheet.lcsc.com/lcsc/1912111437_TDK-CGA4J3X7S2A105KT0Y0N_C338074.pdf" (id 3) (at 209.55 111.76 0)
+      (effects (font (size 1.27 1.27)) hide)
+    )
+    (property "LCSC" "C338074" (id 4) (at 209.55 111.76 0)
+      (effects (font (size 1.27 1.27)) hide)
+    )
+    (property "manf_num  " "CGA4J3X7S2A105KT0Y0N" (id 5) (at 209.55 111.76 0)
       (effects (font (size 1.27 1.27)) hide)
     )
@@
       (effects (font (size 1.27 1.27)) hide)
     )
-    (property "Datasheet" "https://datasheet.lcsc.com/lcsc/2105241210_Taiyo-Yuden-HMK212BC7105KGHTE_C385977.pdf" (id 3) (at 228.6 111.76 0)
-      (effects (font (size 1.27 1.27)) hide)
-    )
-    (property "LCSC" "C385977" (id 4) (at 228.6 111.76 0)
-      (effects (font (size 1.27 1.27)) hide)
-    )
-    (property "manf_num  " "HMK212BC7105KGHTE" (id 5) (at 228.6 111.76 0)
-      (effects (font (size 1.27 1.27)) hide)
-    )
+    (property "Datasheet" "https://datasheet.lcsc.com/lcsc/1912111437_TDK-CGA4J3X7S2A105KT0Y0N_C338074.pdf" (id 3) (at 228.6 111.76 0)
+      (effects (font (size 1.27 1.27)) hide)
+    )
+    (property "LCSC" "C338074" (id 4) (at 228.6 111.76 0)
+      (effects (font (size 1.27 1.27)) hide)
+    )
+    (property "manf_num  " "CGA4J3X7S2A105KT0Y0N" (id 5) (at 228.6 111.76 0)
+      (effects (font (size 1.27 1.27)) hide)
+    )
