File: opm-inline/source/Connectors.kicad_sch (KiCad schematic)
At the start: 32 parts, among them J1 Info, J2 VCC_IO, J3 PWMx6, J4 Fan, J6 Current Sensing, Q7 WSD90P06DN56, U2 TerminalBlock_2_P5.08mm, U3 TerminalBlock_3_P5.08mm

Commit message: fix red led
Parts:
- D2: LCSC C181863 -> C72044; manf_num 19-213/R6W-BP2Q2B/3T -> 19-217/R6C-AL1M2VY/3T
Changed lines of the file:
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@@
       (effects (font (size 1.27 1.27)) hide)
     )
-    (property "LCSC" "C181863" (id 5) (at 132.08 74.93 0)
+    (property "LCSC" "C72044" (id 5) (at 132.08 74.93 0)
       (effects (font (size 1.27 1.27)) hide)
     )
-    (property "manf_num" "19-213/R6W-BP2Q2B/3T" (id 6) (at 132.08 74.93 0)
+    (property "manf_num" "19-217/R6C-AL1M2VY/3T" (id 6) (at 132.08 74.93 0)
       (effects (font (size 1.27 1.27)) hide)
     )
