File: opm-lowside/source/Motor Driver.sch (KiCad schematic (older format))
At the start: 55 parts, among them IC301 TMC6100-LA, Q301 YJG95G06A, Q302 YJG95G06A, Q303 YJG95G06A, Q304 YJG95G06A, Q305 YJG95G06A, Q306 YJG95G06A, U1 INA180A3IDBVR, U2 INA180A3IDBVR, U3 INA180A3IDBVR

Commit message: cleanup
Parts:
- IC301: symbol opm-v1.2-rescue:TMC6100-LA -> opm-lowside-rescue:TMC6100-LA-opm-v1.2-rescue
- Q301, Q302, Q303, Q304, Q305, Q306: symbol opm-v1.1-rescue:YJG95G06A-Transistor_FET -> opm-lowside-rescue:YJG95G06A-Transistor_FET-opm-v1.1-rescue
Changed lines of the file:
@@
 $EndDescr
 $Comp
-L opm-v1.1-rescue:YJG95G06A-Transistor_FET Q301
+L opm-lowside-rescue:YJG95G06A-Transistor_FET-opm-v1.1-rescue Q301
 U 1 1 5D6B7163
 P 6800 800
@@
 $EndComp
 $Comp
-L opm-v1.1-rescue:YJG95G06A-Transistor_FET Q302
+L opm-lowside-rescue:YJG95G06A-Transistor_FET-opm-v1.1-rescue Q302
 U 1 1 5D6C3CF4
 P 6800 1400
@@
 	6000 1100 6900 1100
 $Comp
-L opm-v1.2-rescue:TMC6100-LA IC301
+L opm-lowside-rescue:TMC6100-LA-opm-v1.2-rescue IC301
 U 1 1 5D604226
 P 3950 3500
@@
 	6900 500  6900 600
 $Comp
-L opm-v1.1-rescue:YJG95G06A-Transistor_FET Q303
+L opm-lowside-rescue:YJG95G06A-Transistor_FET-opm-v1.1-rescue Q303
 U 1 1 5D88B06B
 P 6800 2750
@@
 $EndComp
 $Comp
-L opm-v1.1-rescue:YJG95G06A-Transistor_FET Q304
+L opm-lowside-rescue:YJG95G06A-Transistor_FET-opm-v1.1-rescue Q304
 U 1 1 5D88B088
 P 6800 3350
@@
 	6900 2450 6900 2550
 $Comp
-L opm-v1.1-rescue:YJG95G06A-Transistor_FET Q305
+L opm-lowside-rescue:YJG95G06A-Transistor_FET-opm-v1.1-rescue Q305
 U 1 1 5D8A0197
 P 6800 4750
@@
 $EndComp
 $Comp
-L opm-v1.1-rescue:YJG95G06A-Transistor_FET Q306
+L opm-lowside-rescue:YJG95G06A-Transistor_FET-opm-v1.1-rescue Q306
 U 1 1 5D8A01B4
 P 6800 5350

Commit message: update libs
Parts:
- C1, C2, C3: value 0.1uF -> 100nF/10V; LCSC (none) -> C14663; manf_num (none) -> CC0603KRX7R9BB104
- C303, C310: LCSC (none) -> C519409; alt (none) -> CC0603JRX7R7BB471; manf_num (none) -> CC0603KRX7R7BB471
- C305, C307: footprint Capacitor_SMD:C_0805_2012Metric -> Capacitor_SMD:C_0603_1608Metric; LCSC (none) -> C106243; manf_num (none) -> CC0805KKX7R0BB104
- C306: LCSC (none) -> C313105; manf_num (none) -> CC0603KRX7R0BB223
- C311: LCSC (none) -> C106243; manf_num (none) -> CC0805KKX7R0BB104
- C312: Field4 (none) -> C49217; alt (none) -> UMK212BB7225KG-T; manf_num (none) -> 0805F225M500NT
- C313: LCSC (none) -> C49217; alt (none) -> UMK212BB7225KG-T; manf_num (none) -> 0805F225M500NT
- C315: Field4 (none) -> C14663; Field5 (none) -> CC0603KRX7R9BB104
- C318: Field4 (none) -> C519409; Field5 (none) -> CC0603KRX7R7BB471; Field6 (none) -> CC0603JRX7R7BB471
- C5, C6: LCSC (none) -> C1613; manf_num (none) -> CL10B332KB8NNNC
- C7, C8, C9: value 1000pF -> 1nF/16V; LCSC (none) -> C1588; manf_num (none) -> CL10B102KB8NNNC
- R1, R2, R3, R4, R5, R6: LCSC (none) -> C22935; manf_num (none) -> 0603WAF1004T5E
- R10, R11, R12, R7, R9: LCSC (none) -> C22859; alt (none) -> AC0603FR-0710RL; manf_num (none) -> 0603WAF100JT5E
- R13, R14, R15: LCSC (none) -> C22775; manf_num (none) -> 0603WAF1000T5E
- R311, R314: LCSC (none) -> C21189; alt (none) -> RC0603FR-070RL; manf_num (none) -> 0603WAF0000T5E
- U1, U2, U3: LCSC (none) -> C122882; manf_num (none) -> INA180A3IDBVR

Commit message: cleanup
Parts:
- C7, C8, C9: LCSC C1588 -> C342905; manf_num CL10B102KB8NNNC -> CGA3E2X7R2A102KT0Y0N
Connections:
- net +5V: now also C9.2
Changed lines of the file:
@@
 F 1 "1nF/16V" H 10715 1905 50  0000 L CNN
 F 2 "Capacitor_SMD:C_0603_1608Metric" H 10638 1800 50  0001 C CNN
-F 3 "https://datasheet.lcsc.com/lcsc/1811071810_Samsung-Electro-Mechanics-CL10B102KB8NNNC_C1588.pdf" H 10600 1950 50  0001 C CNN
-F 4 "C1588" H 10600 1950 50  0001 C CNN "LCSC"
-F 5 "CL10B102KB8NNNC" H 10600 1950 50  0001 C CNN "manf_num"
+F 3 "https://datasheet.lcsc.com/lcsc/1912111437_TDK-CGA3E2X7R2A102KT0Y0N_C342905.pdf" H 10600 1950 50  0001 C CNN
+F 4 "C342905" H 10600 1950 50  0001 C CNN "LCSC"
+F 5 "CGA3E2X7R2A102KT0Y0N" H 10600 1950 50  0001 C CNN "manf_num"
 	1    10600 1950
 	1    0    0    -1
@@
 F 1 "1nF/16V" H 10715 3855 50  0000 L CNN
 F 2 "Capacitor_SMD:C_0603_1608Metric" H 10638 3750 50  0001 C CNN
-F 3 "https://datasheet.lcsc.com/lcsc/1811071810_Samsung-Electro-Mechanics-CL10B102KB8NNNC_C1588.pdf" H 10600 3900 50  0001 C CNN
-F 4 "C1588" H 10600 3900 50  0001 C CNN "LCSC"
-F 5 "CL10B102KB8NNNC" H 10600 3900 50  0001 C CNN "manf_num"
+F 3 "https://datasheet.lcsc.com/lcsc/1912111437_TDK-CGA3E2X7R2A102KT0Y0N_C342905.pdf" H 10600 3900 50  0001 C CNN
+F 4 "C342905" H 10600 3900 50  0001 C CNN "LCSC"
+F 5 "CGA3E2X7R2A102KT0Y0N" H 10600 3900 50  0001 C CNN "manf_num"
 	1    10600 3900
 	1    0    0    -1
@@
 F 1 "1nF/16V" H 10715 5855 50  0000 L CNN
 F 2 "Capacitor_SMD:C_0603_1608Metric" H 10638 5750 50  0001 C CNN
-F 3 "https://datasheet.lcsc.com/lcsc/1811071810_Samsung-Electro-Mechanics-CL10B102KB8NNNC_C1588.pdf" H 10600 5900 50  0001 C CNN
-F 4 "C1588" H 10600 5900 50  0001 C CNN "LCSC"
-F 5 "CL10B102KB8NNNC" H 10600 5900 50  0001 C CNN "manf_num"
+F 3 "https://datasheet.lcsc.com/lcsc/1912111437_TDK-CGA3E2X7R2A102KT0Y0N_C342905.pdf" H 10600 5900 50  0001 C CNN
+F 4 "C342905" H 10600 5900 50  0001 C CNN "LCSC"
+F 5 "CGA3E2X7R2A102KT0Y0N" H 10600 5900 50  0001 C CNN "manf_num"
 	1    10600 5900
 	1    0    0    -1
@@
 	1    0    0    -1
 $EndComp
+$Comp
+L power:GND #PWR?
+U 1 1 61BF211A
+P 10600 6150
+F 0 "#PWR?" H 10600 5900 50  0001 C CNN
+F 1 "GND" H 10605 5977 50  0000 C CNN
+F 2 "" H 10600 6150 50  0001 C CNN
+F 3 "" H 10600 6150 50  0001 C CNN
+	1    10600 6150
+	1    0    0    -1
+$EndComp
+Wire Wire Line
+	10600 6050 10600 6150
 $EndSCHEMATC
