File: opm-lowside/source/opm-lowside.kicad_pcb (KiCad board)
At the start: 2 copper layers, 58 x 40 mm, 84 parts, among them IC1 INA180A3IDBVR, IC2 INA180A3IDBVR, IC3 INA180A3IDBVR, IC4 QFN37_7X7_TRI, J1 Current Sensing, J2 SPI/Info, J3 VCC_IO, J4 PWMx6, J5 Temperature, M1 Fan, Q1 HYG025N06LS1C2, Q2 HYG025N06LS1C2, Q3 HYG025N06LS1C2, Q4 HYG025N06LS1C2, Q5 HYG025N06LS1C2, Q6 HYG025N06LS1C2, U1 TerminalBlock_2_P5.08mm, U2 TerminalBlock_3_P5.08mm

Commit message: upgrade to kicad6
Connections:
- net /~CS_DRIVER renamed /~{CS_DRIVER}
Other:
- net class Default removed
