File: opm-inline-mcu/source/MotorDriver.kicad_sch (KiCad schematic)
At the start: 44 parts, among them IC1 TMC6200-TA, Q1 HYG025N06LS1C2, Q2 HYG025N06LS1C2, Q3 HYG025N06LS1C2, Q4 HYG025N06LS1C2, Q5 HYG025N06LS1C2, Q6 HYG025N06LS1C2

Commit message: update mcu
Parts:
- IC1: value TMC6200-TA -> eTQFP48_9x9_TRI
Changed lines of the file:
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@@
       (effects (font (size 1.016 1.016)) (justify right))
     )
-    (property "Value" "TMC6200-TA" (id 1) (at 106.68 118.3132 0)
+    (property "Value" "eTQFP48_9x9_TRI" (id 1) (at 106.68 118.3132 0)
       (effects (font (size 1.016 1.016)) (justify right))
     )
