File: opm-inline-mcu/source/mcu.kicad_sch (KiCad schematic)
At the start: 1 part, among them U1 RP2040

Commit message: update mcu
Parts:
- U1: footprint IC57_RP2040 -> Libraries:RP2040
Connections:
- net ADC_I_u: now reaches U1.38 (GPIO26/ADC0)
- net ADC_I_v: now reaches U1.39 (GPIO27/ADC1)
- net ADC_I_w: now reaches U1.40 (GPIO28/ADC2)
- net TEMP: now reaches U1.41 (GPIO29/ADC3)
Changed lines of the file:
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@@
 (kicad_sch (version 20211123) (generator eeschema)
   (paper "A4")
+  (hierarchical_label "ADC_I_w" (shape input) (at 172.72 109.22 0)
+    (effects (font (size 1.27 1.27)) (justify left))
+  )
+  (hierarchical_label "TEMP" (shape input) (at 172.72 106.68 0)
+    (effects (font (size 1.27 1.27)) (justify left))
+  )
+  (hierarchical_label "ADC_I_u" (shape input) (at 172.72 114.3 0)
+    (effects (font (size 1.27 1.27)) (justify left))
+  )
+  (hierarchical_label "ADC_I_v" (shape input) (at 172.72 111.76 0)
+    (effects (font (size 1.27 1.27)) (justify left))
+  )
   (symbol (lib_id "rp2040:RP2040") (at 111.76 66.04 0) (unit 1)
     (in_bom yes) (on_board yes) (fields_autoplaced)
@@
       (effects (font (size 1.524 1.524)))
     )
-    (property "Footprint" "IC57_RP2040" (id 2) (at 142.24 59.944 0)
+    (property "Footprint" "Libraries:RP2040" (id 2) (at 142.24 59.944 0)
       (effects (font (size 1.524 1.524)) hide)
     )

Commit message: update for can
Connections:
- net TEMP renamed TEMP_PCB
Changed lines of the file:
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@@
     (effects (font (size 1.27 1.27)) (justify left))
   )
-  (hierarchical_label "TEMP" (shape input) (at 172.72 106.68 0)
+  (hierarchical_label "TEMP_PCB" (shape input) (at 172.72 106.68 0)
     (effects (font (size 1.27 1.27)) (justify left))
   )
