File: opm-inline-mcu/source/can.kicad_sch (KiCad schematic)
At the start: 34 parts, among them IC2 RP2040, IC3 RP2040, IC4 RP2040, IC5 MIC5219-3.3YM5-TR, IC6 MIC5219-5.0YM5-TR, IC7 TJA1051TK{slash}3, Q8 CSTCE8M00G55-R0

Commit message: update for can
Parts:
- renumbered R26 to R23, R27 to R24
Changed lines of the file:
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@@
   (symbol (lib_id "uc4h node v2100-eagle-import:R-EU_R0603") (at 121.92 99.06 90) (unit 1)
     (in_bom yes) (on_board yes)
-    (property "Reference" "R27" (id 0) (at 120.4214 102.87 0)
+    (property "Reference" "R24" (id 0) (at 120.4214 102.87 0)
       (effects (font (size 1.778 1.5113)) (justify left bottom))
     )
@@
   (symbol (lib_id "uc4h node v2100-eagle-import:R-EU_R0603") (at 50.8 119.38 90) (unit 1)
     (in_bom yes) (on_board yes)
-    (property "Reference" "R26" (id 0) (at 49.53 121.92 0)
-      (effects (font (size 1.778 1.5113)) (justify left bottom))
-    )
+    (property "Reference" "R23" (id 0) (at 49.53 121.92 0)
+      (effects (font (size 1.778 1.5113)) (justify left bottom))
+    )

Commit message: update for can
Parts:
- C28: footprint Resistor_SMD:R_0603_1608Metric -> Capacitor_SMD:C_0603_1608Metric
- C29, C30, C35: footprint uc4h node v2100:C0603K -> Capacitor_SMD:C_0603_1608Metric
- F1: footprint uc4h node v2100:FUSE-0805 -> uc4h node v2100.pretty:FUSE-0805
- IC5, IC6: footprint uc4h node v2100:SOT23-5 -> uc4h node v2100.pretty:SOT23-5
- IC7: footprint uc4h node v2100:HVSON8 -> uc4h node v2100.pretty:HVSON8
- JP2: footprint uc4h node v2100:1X01 -> uc4h node v2100.pretty:1X01
- JP3: footprint uc4h node v2100:1X02 -> uc4h node v2100.pretty:1X02
- JP4, JP5: footprint uc4h node v2100:SM04B-GHS-TB -> uc4h node v2100.pretty:SM04B-GHS-TB
- LED1, LED2: footprint uc4h node v2100:CHIPLED_0603 -> uc4h node v2100.pretty:CHIPLED_0603
- Q8: footprint uc4h node v2100:RESONATOR-SMD -> uc4h node v2100.pretty:RESONATOR-SMD
- R23, R29, R30, R31: footprint uc4h node v2100:R0603 -> Resistor_SMD:R_0603_1608Metric
- SJ1: footprint uc4h node v2100:SJ_2S-NO -> uc4h node v2100.pretty:SJ_2S-NO
Changed lines of the file:
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@@
       (effects (font (size 1.778 1.5113)) (justify left bottom))
     )
-    (property "Footprint" "uc4h node v2100:SJ_2S-NO" (id 2) (at 43.18 101.6 0)
+    (property "Footprint" "uc4h node v2100.pretty:SJ_2S-NO" (id 2) (at 43.18 101.6 0)
       (effects (font (size 1.27 1.27)) hide)
     )
@@
       (effects (font (size 1.778 1.5113)) (justify left bottom))
     )
-    (property "Footprint" "uc4h node v2100:1X02" (id 2) (at 182.88 124.46 0)
+    (property "Footprint" "uc4h node v2100.pretty:1X02" (id 2) (at 182.88 124.46 0)
       (effects (font (size 1.27 1.27)) hide)
     )
@@
       (effects (font (size 1.778 1.5113)) (justify right top))
     )
-    (property "Footprint" "uc4h node v2100:SM04B-GHS-TB" (id 2) (at 246.38 53.34 0)
+    (property "Footprint" "uc4h node v2100.pretty:SM04B-GHS-TB" (id 2) (at 246.38 53.34 0)
       (effects (font (size 1.27 1.27)) hide)
     )
@@
       (effects (font (size 1.778 1.5113)) (justify left bottom))
     )
-    (property "Footprint" "uc4h node v2100:C0603K" (id 2) (at 48.26 76.2 0)
+    (property "Footprint" "Capacitor_SMD:C_0603_1608Metric" (id 2) (at 48.26 76.2 0)
       (effects (font (size 1.27 1.27)) hide)
     )
@@
       (effects (font (size 1.778 1.5113)) (justify left bottom))
     )
-    (property "Footprint" "uc4h node v2100:CHIPLED_0603" (id 2) (at 259.08 137.16 0)
+    (property "Footprint" "uc4h node v2100.pretty:CHIPLED_0603" (id 2) (at 259.08 137.16 0)
       (effects (font (size 1.27 1.27)) hide)
     )
@@
       (effects (font (size 1.778 1.5113)) (justify left bottom))
     )
-    (property "Footprint" "uc4h node v2100:SOT23-5" (id 2) (at 104.14 170.18 0)
+    (property "Footprint" "uc4h node v2100.pretty:SOT23-5" (id 2) (at 104.14 170.18 0)
       (effects (font (size 1.27 1.27)) hide)
     )
@@
       (effects (font (size 1.778 1.5113)) (justify left bottom))
     )
-    (property "Footprint" "uc4h node v2100:R0603" (id 2) (at 205.74 93.98 0)
+    (property "Footprint" "Resistor_SMD:R_0603_1608Metric" (id 2) (at 205.74 93.98 0)
       (effects (font (size 1.27 1.27)) hide)
     )
@@
       (effects (font (size 1.778 1.5113)) (justify left bottom))
     )
-    (property "Footprint" "uc4h node v2100:RESONATOR-SMD" (id 2) (at 48.26 33.02 0)
+    (property "Footprint" "uc4h node v2100.pretty:RESONATOR-SMD" (id 2) (at 48.26 33.02 0)
       (effects (font (size 1.27 1.27)) hide)
     )
@@
       (effects (font (size 1.778 1.5113)) (justify left bottom))
     )
-    (property "Footprint" "uc4h node v2100:C0603K" (id 2) (at 40.64 111.76 0)
+    (property "Footprint" "Capacitor_SMD:C_0603_1608Metric" (id 2) (at 40.64 111.76 0)
       (effects (font (size 1.27 1.27)) hide)
     )
@@
       (effects (font (size 1.778 1.5113)) (justify left bottom))
     )
-    (property "Footprint" "uc4h node v2100:FUSE-0805" (id 2) (at 195.58 53.34 0)
+    (property "Footprint" "uc4h node v2100.pretty:FUSE-0805" (id 2) (at 195.58 53.34 0)
       (effects (font (size 1.27 1.27)) hide)
     )
@@
       (effects (font (size 1.778 1.5113)) (justify left bottom))
     )
-    (property "Footprint" "uc4h node v2100:CHIPLED_0603" (id 2) (at 259.08 152.4 0)
+    (property "Footprint" "uc4h node v2100.pretty:CHIPLED_0603" (id 2) (at 259.08 152.4 0)
       (effects (font (size 1.27 1.27)) hide)
     )
@@
       (effects (font (size 1.778 1.5113)) (justify left bottom))
     )
-    (property "Footprint" "uc4h node v2100:SOT23-5" (id 2) (at 109.22 134.62 0)
+    (property "Footprint" "uc4h node v2100.pretty:SOT23-5" (id 2) (at 109.22 134.62 0)
       (effects (font (size 1.27 1.27)) hide)
     )
@@
       (effects (font (size 1.778 1.5113)) (justify left bottom))
     )
-    (property "Footprint" "uc4h node v2100:C0603K" (id 2) (at 154.94 83.82 0)
+    (property "Footprint" "Capacitor_SMD:C_0603_1608Metric" (id 2) (at 154.94 83.82 0)
       (effects (font (size 1.27 1.27)) hide)
     )
@@
       (effects (font (size 1.778 1.5113)) (justify left bottom))
     )
-    (property "Footprint" "Resistor_SMD:R_0603_1608Metric" (id 2) (at 40.64 76.2 0)
+    (property "Footprint" "Capacitor_SMD:C_0603_1608Metric" (id 2) (at 40.64 76.2 0)
       (effects (font (size 1.27 1.27)) hide)
     )
@@
       (effects (font (size 1.778 1.5113)) (justify right top))
     )
-    (property "Footprint" "uc4h node v2100:SM04B-GHS-TB" (id 2) (at 246.38 73.66 0)
+    (property "Footprint" "uc4h node v2100.pretty:SM04B-GHS-TB" (id 2) (at 246.38 73.66 0)
       (effects (font (size 1.27 1.27)) hide)
     )
@@
       (effects (font (size 1.778 1.5113)) (justify left bottom))
     )
-    (property "Footprint" "uc4h node v2100:R0603" (id 2) (at 50.8 119.38 0)
+    (property "Footprint" "Resistor_SMD:R_0603_1608Metric" (id 2) (at 50.8 119.38 0)
       (effects (font (size 1.27 1.27)) hide)
     )
@@
       (effects (font (size 1.778 1.5113)) (justify left bottom))
     )
-    (property "Footprint" "uc4h node v2100:HVSON8" (id 2) (at 180.34 81.28 0)
+    (property "Footprint" "uc4h node v2100.pretty:HVSON8" (id 2) (at 180.34 81.28 0)
       (effects (font (size 1.27 1.27)) hide)
     )
@@
       (effects (font (size 1.778 1.5113)) (justify left bottom))
     )
-    (property "Value" "4.7k" (id 1) (at 245.11 140.462 0)
-      (effects (font (size 1.778 1.5113)) (justify left bottom))
-    )
-    (property "Footprint" "uc4h node v2100:R0603" (id 2) (at 248.92 137.16 0)
+    (property "Value" "4.7k" (id 1) (at 245.11 140.97 0)
+      (effects (font (size 1.778 1.5113)) (justify left bottom))
+    )
+    (property "Footprint" "Resistor_SMD:R_0603_1608Metric" (id 2) (at 248.92 137.16 0)
       (effects (font (size 1.27 1.27)) hide)
     )
@@
       (effects (font (size 1.778 1.5113)) (justify left bottom))
     )
-    (property "Value" "2.2k" (id 1) (at 245.11 155.702 0)
-      (effects (font (size 1.778 1.5113)) (justify left bottom))
-    )
-    (property "Footprint" "uc4h node v2100:R0603" (id 2) (at 248.92 152.4 0)
+    (property "Value" "2.2k" (id 1) (at 245.11 156.21 0)
+      (effects (font (size 1.778 1.5113)) (justify left bottom))
+    )
+    (property "Footprint" "Resistor_SMD:R_0603_1608Metric" (id 2) (at 248.92 152.4 0)
       (effects (font (size 1.27 1.27)) hide)
     )
@@
       (effects (font (size 1.778 1.5113)) (justify left bottom))
     )
-    (property "Footprint" "uc4h node v2100:1X01" (id 2) (at 182.88 114.3 0)
-      (effects (font (size 1.27 1.27)) hide)
-    )
+    (property "Footprint" "uc4h node v2100.pretty:1X01" (id 2) (at 182.88 114.3 0)
+      (effects (font (size 1.27 1.27)) hide)
+    )

Commit message: update for can
Parts:
- IC5: footprint uc4h node v2100.pretty:SOT23-5 -> Package_TO_SOT_SMD:SOT-23-5; LCSC (none) -> C29613; manf_num (none) -> MIC5219-3.3YM5-TR
- IC6: footprint uc4h node v2100.pretty:SOT23-5 -> Package_TO_SOT_SMD:SOT-23-5; LCSC (none) -> C144182; manf_num (none) -> MIC5219-5.0YM5-TR
- IC7: value TJA1051TK/3 -> TJA1051TK/3; footprint uc4h node v2100.pretty:HVSON8 -> Package_DFN_QFN:VDFN-8-1EP_2x2mm_P0.5mm_EP0.9x1.7mm; LCSC (none) -> C2875699; manf_num (none) -> TJA1051TK/3
Changed lines of the file:
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@@
       (effects (font (size 1.778 1.5113)) (justify left bottom))
     )
-    (property "Footprint" "uc4h node v2100.pretty:SOT23-5" (id 2) (at 104.14 170.18 0)
-      (effects (font (size 1.27 1.27)) hide)
-    )
-    (property "Datasheet" "" (id 3) (at 104.14 170.18 0)
+    (property "Footprint" "Package_TO_SOT_SMD:SOT-23-5" (id 2) (at 104.14 170.18 0)
+      (effects (font (size 1.27 1.27)) hide)
+    )
+    (property "Datasheet" "https://datasheet.lcsc.com/lcsc/1811132212_Microchip-Tech-MIC5219-3-3YM5-TR_C29613.pdf" (id 3) (at 104.14 170.18 0)
+      (effects (font (size 1.27 1.27)) hide)
+    )
+    (property "LCSC" "C29613" (id 4) (at 104.14 170.18 0)
+      (effects (font (size 1.27 1.27)) hide)
+    )
+    (property "manf_num" "MIC5219-3.3YM5-TR" (id 5) (at 104.14 170.18 0)
       (effects (font (size 1.27 1.27)) hide)
     )
@@
   (symbol (lib_id "uc4h node v2100-eagle-import:R-EU_R0603") (at 205.74 93.98 0) (unit 1)
     (in_bom yes) (on_board yes)
-    (property "Reference" "R29" (id 0) (at 201.93 92.4814 0)
-      (effects (font (size 1.778 1.5113)) (justify left bottom))
-    )
-    (property "Value" "120" (id 1) (at 201.93 97.282 0)
+    (property "Reference" "R29" (id 0) (at 203.2 92.71 0)
+      (effects (font (size 1.778 1.5113)) (justify left bottom))
+    )
+    (property "Value" "120" (id 1) (at 203.2 97.79 0)
       (effects (font (size 1.778 1.5113)) (justify left bottom))
     )
@@
       (effects (font (size 1.778 1.5113)) (justify left bottom))
     )
-    (property "Footprint" "uc4h node v2100.pretty:SOT23-5" (id 2) (at 109.22 134.62 0)
-      (effects (font (size 1.27 1.27)) hide)
-    )
-    (property "Datasheet" "" (id 3) (at 109.22 134.62 0)
+    (property "Footprint" "Package_TO_SOT_SMD:SOT-23-5" (id 2) (at 109.22 134.62 0)
+      (effects (font (size 1.27 1.27)) hide)
+    )
+    (property "Datasheet" "https://datasheet.lcsc.com/lcsc/1806090830_Microchip-Tech-MIC5219-5-0YM5-TR_C144182.pdf" (id 3) (at 109.22 134.62 0)
+      (effects (font (size 1.27 1.27)) hide)
+    )
+    (property "LCSC" "C144182" (id 4) (at 109.22 134.62 0)
+      (effects (font (size 1.27 1.27)) hide)
+    )
+    (property "manf_num" "MIC5219-5.0YM5-TR" (id 5) (at 109.22 134.62 0)
       (effects (font (size 1.27 1.27)) hide)
     )
@@
       (effects (font (size 1.778 1.5113)) (justify left bottom))
     )
-    (property "Value" "TJA1051TK{slash}3" (id 1) (at 170.18 96.52 0)
-      (effects (font (size 1.778 1.5113)) (justify left bottom))
-    )
-    (property "Footprint" "uc4h node v2100.pretty:HVSON8" (id 2) (at 180.34 81.28 0)
+    (property "Value" "TJA1051TK/3" (id 1) (at 170.18 96.52 0)
+      (effects (font (size 1.778 1.5113)) (justify left bottom))
+    )
+    (property "Footprint" "Package_DFN_QFN:VDFN-8-1EP_2x2mm_P0.5mm_EP0.9x1.7mm" (id 2) (at 180.34 81.28 0)
       (effects (font (size 1.27 1.27)) hide)
     )
@@
       (effects (font (size 1.27 1.27)) hide)
     )
+    (property "LCSC" "C2875699" (id 4) (at 180.34 81.28 0)
+      (effects (font (size 1.27 1.27)) hide)
+    )
+    (property "manf_num" "TJA1051TK/3" (id 5) (at 180.34 81.28 0)
+      (effects (font (size 1.27 1.27)) hide)
+    )

Commit message: update for can
Parts:
- R24, R28: footprint uc4h node v2100:R0603 -> Resistor_SMD:R_0603_1608Metric
Changed lines of the file:
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@@
       (effects (font (size 1.778 1.5113)) (justify left bottom))
     )
-    (property "Footprint" "uc4h node v2100:R0603" (id 2) (at 121.92 99.06 0)
-      (effects (font (size 1.27 1.27)) hide)
-    )
+    (property "Footprint" "Resistor_SMD:R_0603_1608Metric" (id 2) (at 121.92 99.06 0))
     (property "Datasheet" "" (id 3) (at 121.92 99.06 0)
       (effects (font (size 1.27 1.27)) hide)
@@
       (effects (font (size 1.778 1.5113)) (justify left bottom))
     )
-    (property "Footprint" "uc4h node v2100:R0603" (id 2) (at 129.54 99.06 0)
-      (effects (font (size 1.27 1.27)) hide)
-    )
+    (property "Footprint" "Resistor_SMD:R_0603_1608Metric" (id 2) (at 129.54 99.06 0)
+      (effects (font (size 1.27 1.27)) hide)
+    )

Commit message: add can
Parts:
- removed IC2, IC3, IC4: RP2040, uc4h node v2100:VFQFPN36, symbol uc4h node v2100-eagle-import:STM32F10XTXU6
- C32: footprint uc4h node v2100:C0603K -> Capacitor_SMD:C_0603_1608Metric
- C33: value 1u -> 1uF; footprint uc4h node v2100:C0603K -> Capacitor_SMD:C_0603_1608Metric
- C34: value 1u -> 1uF; footprint uc4h node v2100:C0603K -> Capacitor_SMD:C_0201_0603Metric
- R24, R28: value 10k -> 10KR/1%
- SJ2, SJ3: footprint uc4h node v2100:SJ_2S-NO -> uc4h node v2100.pretty:SJ_2S-NO
- SWD1: footprint uc4h node v2100:4X1_1P27_OCT_BILEX -> uc4h node v2100.pretty:4X1_1P27_OCT_BILEX
Connections:
- net BOOT0: now reaches R23.2, SJ1.2
- net PD0/OSC<=: now reaches Q8.1
- net PD1/OSC=>: now reaches Q8.3
- net NRST: now reaches C29.1
- net SCL/A2 renamed SCL/A2
- net SDA/A1 renamed SDA/A1
Other:
- note removed: "Uavcan 4 Hobbyists"
- note removed: "Uc4h All-In-One Node"
- note removed: "this is because TIM on Tx1 can't be used if Rx1 is used, STM errata"
- note removed: "this is to avoid DMA overlap"
- moved on the sheet: C29, C35, F1, IC7, JP4, JP5, R23, R24, R28, R29, SJ1, SJ2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
