File: opm-inline-mcu/source/opm-inline.kicad_pcb (KiCad board)
At the start: 4 copper layers, 58 x 40 mm, 76 parts, among them IC1 eTQFP48_9x9_TRI, J1 Info, J2 VCC_IO, J3 PWMx6, J4 Fan, J6 Current Sensing, Q1 HYG025N06LS1C2, Q2 HYG025N06LS1C2, Q3 HYG025N06LS1C2, Q4 HYG025N06LS1C2, Q5 HYG025N06LS1C2, Q6 HYG025N06LS1C2, Q7 WSD90P06DN56, U2 TerminalBlock_2_P5.08mm, U3 TerminalBlock_3_P5.08mm

Commit message: update mcu
Parts:
- removed D7: Val**, Libraries:NUP4114UCW1T2G
- removed J1: Info, Connector_JST:JST_PH_B3B-PH-K_1x03_P2.00mm_Vertical
- removed J6: Current Sensing, Connector_JST:JST_PH_B3B-PH-K_1x03_P2.00mm_Vertical
- added U1: RP2040, Libraries:RP2040, F.Cu at (140.5, 94.0)
- moved R26 3.59 mm to (148.5, 97.8), turned to 180 degrees
Connections:
- D5 pad 1: /FAULT -> unconnected-(D5-Pad1)
- D5 pad 4: /DRV_EN -> unconnected-(D5-Pad4)
- D5 pad 6: /TEMP_PCB -> unconnected-(D5-Pad6)
Routing:
- net /TEMP_PCB: track 42.5 -> 3.78 mm, vias 1 -> 0
- net /DRV_EN: track 37.9 -> 0.00 mm, vias 2 -> 0
- net /FAULT: track 63.0 -> 28.2 mm, vias 4 -> 2
- net /ADC_I_w: track 17.0 -> 0.00 mm
- net /ADC_I_v: track 16.5 -> 0.00 mm
- net /ADC_I_u: track 15.5 -> 0.00 mm
- net Net-(IC1-Pad24): track 6.59 -> 0.00 mm
- net GND: track 27.3 -> 26.5 mm, vias 46 -> 45
- net Net-(IC1-Pad46): vias 1 -> 0

Commit message: update for can
Parts:
- moved J4 11.2 mm to (140.3, 104.0), turned to 180 degrees
- moved U1 10.2 mm to (140.8, 83.8)
- moved HS1 8.52 mm to (148.2, 103.4)
- moved R22 6.77 mm to (148.2, 81.8), turned to 90 degrees
- moved R21 6.49 mm to (148.2, 84.8), turned to -90 degrees
- moved D3 5.80 mm to (140.1, 73.1)
- moved D5 5.77 mm to (136.5, 73.1)
- moved C10 5.60 mm to (151.1, 84.1)
- moved C20 5.60 mm to (149.6, 84.1)
- moved J2 5.48 mm to (132.7, 74.4)
Routing:
- net /+VCC_IO: track 52.5 -> 19.1 mm
- net /WL: track 34.2 -> 19.4 mm, vias 2 -> 1
- net /UL: track 27.4 -> 13.6 mm, vias 2 -> 1
- net /UH: track 27.1 -> 13.8 mm, vias 2 -> 1
- net /VH: track 28.6 -> 16.8 mm, vias 2 -> 1
- net GND: track 26.5 -> 20.2 mm, vias 45 -> 40
- net /WH: track 33.2 -> 27.2 mm, vias 3 -> 1
- net /Motor Driver/VOFS: track 4.15 -> 0.00 mm
- net /VL: track 32.1 -> 28.5 mm, vias 3 -> 1
- net /Connectors/VOFS: track 1.52 -> 0.00 mm

Commit message: update for can
Parts:
- removed D3: Val**, Libraries:NUP4114UCW1T2G
- removed J3: PWMx6, Connector_JST:JST_PH_B6B-PH-K_1x06_P2.00mm_Vertical
- added C27: 100n, Capacitor_SMD:C_0603_1608Metric, F.Cu at (137.6, 98.8)
- added C28: 100n, Resistor_SMD:R_0603_1608Metric, F.Cu at (137.9, 104.8)
- added C29: 100n, Capacitor_SMD:C_0603_1608Metric, F.Cu at (133.8, 99.1)
- added C30: 100n, Capacitor_SMD:C_0603_1608Metric, F.Cu at (133.7, 100.6)
- added C31: 10u/25V, Capacitor_SMD:C_0603_1608Metric, F.Cu at (137.9, 103.2)
- added C35: 100n, Capacitor_SMD:C_0603_1608Metric, F.Cu at (142.2, 73.5)
- added F1: 0ZCK0020FF2G, uc4h node v2100.pretty:FUSE-0805, F.Cu at (136.2, 76.6)
- added IC5: MIC5219-3.3YM5-TR, uc4h node v2100.pretty:SOT23-5, F.Cu at (140.9, 90.9)
- added IC6: MIC5219-5.0YM5-TR, uc4h node v2100.pretty:SOT23-5, F.Cu at (138.8, 74.7)
- added IC7: TJA1051TK/3, uc4h node v2100.pretty:HVSON8, F.Cu at (139.3, 94.7)
- added JP1: M04PTH, uc4h node v2100.pretty:1X04, F.Cu at (131.9, 76.2)
- added JP2: M01PTH, uc4h node v2100.pretty:1X01, F.Cu at (135.1, 73.4)
- added JP3: M02PTH, uc4h node v2100.pretty:1X02, F.Cu at (135.1, 70.9)
- added JP4: JST-GH-4, uc4h node v2100.pretty:SM04B-GHS-TB, F.Cu at (130.6, 84.0)
- added JP5: JST-GH-4, uc4h node v2100.pretty:SM04B-GHS-TB, F.Cu at (130.7, 93.6)
- added LED1: red, uc4h node v2100.pretty:CHIPLED_0603, F.Cu at (135.1, 103.3)
- added LED2: green, uc4h node v2100.pretty:CHIPLED_0603, F.Cu at (131.1, 99.5)
- added Q8: CSTCE8M00G55-R0, uc4h node v2100.pretty:RESONATOR-SMD, F.Cu at (144.5, 99.4)
- added R23: 10k, Resistor_SMD:R_0603_1608Metric, F.Cu at (137.6, 90.0)
- added R29: 120, Resistor_SMD:R_0603_1608Metric, F.Cu at (137.8, 101.6)
- added R30: 4.7k, Resistor_SMD:R_0603_1608Metric, F.Cu at (137.7, 97.2)
- added R31: 2.2k, Resistor_SMD:R_0603_1608Metric, F.Cu at (131.8, 103.0)
- added SJ1: BOOT0, uc4h node v2100.pretty:SJ_2S-NO, F.Cu at (137.4, 88.3)
- moved H202 28.3 mm to (157.1, 103.7)
- moved H201 17.7 mm to (150.9, 103.6)
- moved D5 9.26 mm to (145.6, 71.4)
- moved J2 8.89 mm to (139.7, 68.9), turned to 0 degrees
- moved J4 4.10 mm to (144.4, 104.0)
- moved U1 1.34 mm to (142.0, 83.2)
- moved R22 0.93 mm to (148.1, 80.9)
- moved R21 0.91 mm to (148.1, 83.9)
Connections:
- net /TEMP renamed /MCU/TEMP
- D5 pad 5: /WL -> unconnected-(D5-Pad5)
Routing:
- net /WH: track 27.2 -> 17.9 mm
- net /VL: track 28.5 -> 19.7 mm
- net /UL: track 13.6 -> 9.31 mm
- net GND: track 20.2 -> 23.1 mm
- net /VH: track 16.8 -> 15.5 mm
- net /WL: track 19.4 -> 18.1 mm

Commit message: update for can
Parts:
- moved J4 1.99 mm to (142.5, 103.4), turned to 0 degrees
Changed lines of the file:
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@@
   )
   (footprint "Connector_JST:JST_PH_B2B-PH-K_1x02_P2.00mm_Vertical" (layer "F.Cu")
-    (at 144.4 104 180)
+    (at 142.5 103.4)
     (descr "JST PH series connector, B2B-PH-K (http://www.jst-mfg.com/product/pdf/eng/ePH.pdf), generated with kicad-footprint-generator")
     (tags "connector JST PH side entry")
@@
     (fp_line (start -1.11 -2.11) (end -2.36 -2.11) (layer "F.Fab") (width 0.1))
     (fp_line (start 3.95 -1.7) (end -1.95 -1.7) (layer "F.Fab") (width 0.1))
-    (pad "1" thru_hole roundrect (at 0 0 180) (size 1.2 1.75) (drill 0.75) (layers *.Cu *.Mask) (roundrect_rratio 0.208333)
+    (pad "1" thru_hole roundrect (at 0 0) (size 1.2 1.75) (drill 0.75) (layers *.Cu *.Mask) (roundrect_rratio 0.208333)
       (net 49 "/+VCC_IO") (pinfunction "Pin_1") (pintype "passive"))
-    (pad "2" thru_hole oval (at 2 0 180) (size 1.2 1.75) (drill 0.75) (layers *.Cu *.Mask)
+    (pad "2" thru_hole oval (at 2 0) (size 1.2 1.75) (drill 0.75) (layers *.Cu *.Mask)
       (net 5 "GND") (pinfunction "Pin_2") (pintype "passive"))
     (model "${KICAD6_3DMODEL_DIR}/Connector_JST.3dshapes/JST_PH_B2B-PH-K_1x02_P2.00mm_Vertical.wrl"

Commit message: update for can
Parts:
- C28: footprint Resistor_SMD:R_0603_1608Metric -> Capacitor_SMD:C_0603_1608Metric
- IC5, IC6: footprint uc4h node v2100.pretty:SOT23-5 -> Package_TO_SOT_SMD:SOT-23-5
- IC7: footprint uc4h node v2100.pretty:HVSON8 -> Package_DFN_QFN:VDFN-8-1EP_2x2mm_P0.5mm_EP0.9x1.7mm
- U1: value RP2040 -> IC57_RP2040
Connections:
- U1 pad 41: /MCU/TEMP -> /TEMP_PCB
Routing:
- net /VL: track 19.7 -> 2.75 mm
- net /WL: track 18.1 -> 2.19 mm
- net /WH: track 17.9 -> 2.35 mm
- net /VH: track 15.5 -> 1.78 mm
- net /UH: track 13.8 -> 3.97 mm
- net /UL: track 9.31 -> 2.84 mm

Commit message: update for can
Parts:
- added R24: 10k, Resistor_SMD:R_0603_1608Metric, F.Cu at (140.0, 77.4)
- added R28: 10k, Resistor_SMD:R_0603_1608Metric, F.Cu at (144.0, 77.4)
- U1: value IC57_RP2040 -> RP2040
- moved Q8 0.10 mm to (144.5, 99.5)
Changed lines of the file:
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@@
       (net 114 "/CAN/CAN-PWR-IN") (pinfunction "2") (pintype "bidirectional") (solder_mask_margin 0.0635))
+  )
+  (footprint "Resistor_SMD:R_0603_1608Metric" (layer "F.Cu")
+    (at 140 77.4)
+    (descr "Resistor SMD 0603 (1608 Metric), square (rectangular) end terminal, IPC_7351 nominal, (Body size source: IPC-SM-782 page 72, https://www.pcb-3d.com/wordpress/wp-content/uploads/ipc-sm-782a_amendment_1_and_2.pdf), generated with kicad-footprint-generator")
+    (tags "resistor")
+    (property "Sheetfile" "can.kicad_sch")
+    (property "Sheetname" "CAN")
+    (attr smd)
+    (fp_text reference "R24" (at 0 -1.43) (layer "F.SilkS")
+      (effects (font (size 1 1) (thickness 0.15)))
+    )
+    (fp_text value "10k" (at 0 1.43) (layer "F.Fab")
+      (effects (font (size 1 1) (thickness 0.15)))
+    )
+    (fp_text user "${REFERENCE}" (at 0 0) (layer "F.Fab")
+      (effects (font (size 0.4 0.4) (thickness 0.06)))
+    )
+    (fp_line (start -0.237258 -0.5225) (end 0.237258 -0.5225) (layer "F.SilkS") (width 0.12))
+    (fp_line (start -0.237258 0.5225) (end 0.237258 0.5225) (layer "F.SilkS") (width 0.12))
+    (fp_line (start 1.48 -0.73) (end 1.48 0.73) (layer "F.CrtYd") (width 0.05))
+    (fp_line (start -1.48 0.73) (end -1.48 -0.73) (layer "F.CrtYd") (width 0.05))
+    (fp_line (start 1.48 0.73) (end -1.48 0.73) (layer "F.CrtYd") (width 0.05))
+    (fp_line (start -1.48 -0.73) (end 1.48 -0.73) (layer "F.CrtYd") (width 0.05))
+    (fp_line (start 0.8 0.4125) (end -0.8 0.4125) (layer "F.Fab") (width 0.1))
+    (fp_line (start -0.8 0.4125) (end -0.8 -0.4125) (layer "F.Fab") (width 0.1))
+    (fp_line (start 0.8 -0.4125) (end 0.8 0.4125) (layer "F.Fab") (width 0.1))
+    (fp_line (start -0.8 -0.4125) (end 0.8 -0.4125) (layer "F.Fab") (width 0.1))
+    (pad "1" smd roundrect (at -0.825 0) (size 0.8 0.95) (layers "F.Cu" "F.Paste" "F.Mask") (roundrect_rratio 0.25)
+      (net 122 "/CAN/SCL{slash}A2") (pinfunction "1") (pintype "passive"))
+    (pad "2" smd roundrect (at 0.825 0) (size 0.8 0.95) (layers "F.Cu" "F.Paste" "F.Mask") (roundrect_rratio 0.25)
+      (net 111 "3.3V") (pinfunction "2") (pintype "passive"))
+    (model "${KICAD6_3DMODEL_DIR}/Resistor_SMD.3dshapes/R_0603_1608Metric.wrl"
+      (offset (xyz 0 0 0))
+      (scale (xyz 1 1 1))
+      (rotate (xyz 0 0 0))
+    )
   )
   (footprint "Capacitor_SMD:C_0603_1608Metric" (layer "F.Cu")
@@
     )
   )
+  (footprint "Resistor_SMD:R_0603_1608Metric" (layer "F.Cu")
+    (at 144.01 77.4)
+    (descr "Resistor SMD 0603 (1608 Metric), square (rectangular) end terminal, IPC_7351 nominal, (Body size source: IPC-SM-782 page 72, https://www.pcb-3d.com/wordpress/wp-content/uploads/ipc-sm-782a_amendment_1_and_2.pdf), generated with kicad-footprint-generator")
+    (tags "resistor")
+    (property "Sheetfile" "can.kicad_sch")
+    (property "Sheetname" "CAN")
+    (attr smd)
+    (fp_text reference "R28" (at 0 -1.43) (layer "F.SilkS")
+      (effects (font (size 1 1) (thickness 0.15)))
+    )
+    (fp_text value "10k" (at 0 1.43) (layer "F.Fab")
+      (effects (font (size 1 1) (thickness 0.15)))
+    )
+    (fp_text user "${REFERENCE}" (at 0 0) (layer "F.Fab")
+      (effects (font (size 0.4 0.4) (thickness 0.06)))
+    )
+    (fp_line (start -0.237258 0.5225) (end 0.237258 0.5225) (layer "F.SilkS") (width 0.12))
+    (fp_line (start -0.237258 -0.5225) (end 0.237258 -0.5225) (layer "F.SilkS") (width 0.12))
+    (fp_line (start 1.48 -0.73) (end 1.48 0.73) (layer "F.CrtYd") (width 0.05))
+    (fp_line (start 1.48 0.73) (end -1.48 0.73) (layer "F.CrtYd") (width 0.05))
+    (fp_line (start -1.48 0.73) (end -1.48 -0.73) (layer "F.CrtYd") (width 0.05))
+    (fp_line (start -1.48 -0.73) (end 1.48 -0.73) (layer "F.CrtYd") (width 0.05))
+    (fp_line (start 0.8 0.4125) (end -0.8 0.4125) (layer "F.Fab") (width 0.1))
+    (fp_line (start 0.8 -0.4125) (end 0.8 0.4125) (layer "F.Fab") (width 0.1))
+    (fp_line (start -0.8 0.4125) (end -0.8 -0.4125) (layer "F.Fab") (width 0.1))
+    (fp_line (start -0.8 -0.4125) (end 0.8 -0.4125) (layer "F.Fab") (width 0.1))
+    (pad "1" smd roundrect (at -0.825 0) (size 0.8 0.95) (layers "F.Cu" "F.Paste" "F.Mask") (roundrect_rratio 0.25)
+      (net 123 "/CAN/SDA{slash}A1") (pinfunction "1") (pintype "passive"))
+    (pad "2" smd roundrect (at 0.825 0) (size 0.8 0.95) (layers "F.Cu" "F.Paste" "F.Mask") (roundrect_rratio 0.25)
+      (net 111 "3.3V") (pinfunction "2") (pintype "passive"))
+    (model "${KICAD6_3DMODEL_DIR}/Resistor_SMD.3dshapes/R_0603_1608Metric.wrl"
+      (offset (xyz 0 0 0))
+      (scale (xyz 1 1 1))
+      (rotate (xyz 0 0 0))
+    )
+  )
   (footprint "uc4h node v2100.pretty:RESONATOR-SMD" (layer "F.Cu")
-    (at 144.5 99.4)
+    (at 144.5 99.5)
     (property "Sheetfile" "can.kicad_sch")
     (property "Sheetname" "CAN")
@@
       (effects (font (size 1 1) (thickness 0.15)))
     )
-    (fp_text value "IC57_RP2040" (at 0 0) (layer "F.SilkS")
+    (fp_text value "RP2040" (at 0 0) (layer "F.SilkS")
       (effects (font (size 1 1) (thickness 0.15)))
     )

Commit message: add can
Parts:
- added C32: 100n, Capacitor_SMD:C_0603_1608Metric, F.Cu at (142.4, 74.7)
- added C33: 1uF, Capacitor_SMD:C_0603_1608Metric, F.Cu at (142.5, 73.0)
- added C34: 1uF, Capacitor_SMD:C_0201_0603Metric, F.Cu at (146.3, 74.6)
- added SJ2: SOLDERJUMPERNO, uc4h node v2100.pretty:SJ_2S-NO, F.Cu at (140.8, 100.3)
- added SJ3: SOLDERJUMPERNO, uc4h node v2100.pretty:SJ_2S-NO, F.Cu at (141.1, 98.7)
- added SWD1: PH4, uc4h node v2100.pretty:4X1_1P27_OCT_BILEX, F.Cu at (131.6, 78.7)
- R24, R28: value 10k -> 10KR/1%
- moved C35 3.68 mm to (145.9, 73.5)
- moved JP4 0.32 mm to (130.3, 84.0)
- moved JP5 0.32 mm to (130.4, 93.6)
Connections:
- net /CAN/LED renamed LED
- net /CAN/SCL/A2 renamed SCL/A2
- net /CAN/SDA/A1 renamed SDA/A1
- net Net-(R23-Pad2) renamed BOOT0
- C29 pad 1: unconnected-(C29-Pad1) -> NRST
- Q8 pad 1: unconnected-(Q8-Pad1) -> /CAN/PD0/OSC<=
- Q8 pad 3: unconnected-(Q8-Pad3) -> /CAN/PD1/OSC=>
