File: opm-inline-mcu/source/opm-inline.kicad_sch (KiCad schematic)
At the start: 0 parts

Commit message: update mcu
Other:
- sheet mcu ports: added ADC_I_u, ADC_I_v, ADC_I_w, TEMP; removed none
Changed lines of the file:
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@@
+    (stroke (width 0) (type default) (color 0 0 0 0))
+  )
+  (wire (pts (xy 110.49 88.9) (xy 107.95 88.9))
     (stroke (width 0) (type default) (color 0 0 0 0))
   )
@@
     (stroke (width 0) (type default) (color 0 0 0 0))
   )
+  (wire (pts (xy 107.95 83.82) (xy 110.49 83.82))
+    (stroke (width 0) (type default) (color 0 0 0 0))
+  )
+  (wire (pts (xy 107.95 86.36) (xy 110.49 86.36))
+    (stroke (width 0) (type default) (color 0 0 0 0))
+  )
   (wire (pts (xy 234.95 87.63) (xy 232.41 87.63))
     (stroke (width 0) (type default) (color 0 0 0 0))
@@
     (stroke (width 0) (type default) (color 0 0 0 0))
   )
+  (wire (pts (xy 107.95 81.28) (xy 110.49 81.28))
+    (stroke (width 0) (type default) (color 0 0 0 0))
+  )
   (wire (pts (xy 171.45 74.93) (xy 168.91 74.93))
     (stroke (width 0) (type default) (color 0 0 0 0))
@@
     (effects (font (size 0.9906 0.9906)) (justify left bottom))
   )
+  (label "ADC_I_w" (at 110.49 88.9 0)
+    (effects (font (size 0.9906 0.9906)) (justify left bottom))
+  )
   (label "5Vout" (at 171.45 102.87 0)
     (effects (font (size 0.9906 0.9906)) (justify left bottom))
@@
     (effects (font (size 0.9906 0.9906)) (justify left bottom))
   )
+  (label "TEMP" (at 110.49 81.28 0)
+    (effects (font (size 0.9906 0.9906)) (justify left bottom))
+  )
   (label "DRV_EN" (at 140.97 82.55 180)
     (effects (font (size 0.9906 0.9906)) (justify right bottom))
@@
     (effects (font (size 0.9906 0.9906)) (justify right bottom))
   )
+  (label "ADC_I_v" (at 110.49 86.36 0)
+    (effects (font (size 0.9906 0.9906)) (justify left bottom))
+  )
   (label "VH" (at 140.97 100.33 180)
     (effects (font (size 0.9906 0.9906)) (justify right bottom))
@@
   )
   (label "DRV_EN" (at 234.95 100.33 0)
+    (effects (font (size 0.9906 0.9906)) (justify left bottom))
+  )
+  (label "ADC_I_u" (at 110.49 83.82 0)
     (effects (font (size 0.9906 0.9906)) (justify left bottom))
   )
@@
       (effects (font (size 1.27 1.27)) (justify left top))
     )
+    (pin "ADC_I_w" input (at 107.95 88.9 0)
+      (effects (font (size 1.27 1.27)) (justify right))
+    )
+    (pin "ADC_I_v" input (at 107.95 86.36 0)
+      (effects (font (size 1.27 1.27)) (justify right))
+    )
+    (pin "ADC_I_u" input (at 107.95 83.82 0)
+      (effects (font (size 1.27 1.27)) (justify right))
+    )
+    (pin "TEMP" input (at 107.95 81.28 0)
+      (effects (font (size 1.27 1.27)) (justify right))
+    )
   )
   (sheet_instances
@@
       (reference "#PWR011") (unit 1) (value "GND") (footprint "")
     )
-    (path "/00000000-0000-0000-0000-00005ba8c4e4/00000000-0000-0000-0000-000062254bf0"
-      (reference "#PWR012") (unit 1) (value "GND") (footprint "")
-    )
     (path "/00000000-0000-0000-0000-00005ba8c4e4/00000000-0000-0000-0000-000061bf9a67"
       (reference "#PWR0101") (unit 1) (value "GND") (footprint "")
@@
       (reference "D6") (unit 1) (value "TVS DIODE") (footprint "Diode_SMD:D_SMA")
     )
-    (path "/00000000-0000-0000-0000-00005ba8c4e4/00000000-0000-0000-0000-000062246232"
-      (reference "D7") (unit 1) (value "Val**") (footprint "Libraries:NUP4114UCW1T2G")
-    )
     (path "/00000000-0000-0000-0000-00005ba8c4e4/00000000-0000-0000-0000-00005c33535a"
       (reference "H201") (unit 1) (value "MountingHole") (footprint "MountingHole:MountingHole_2.2mm_M2_Pad_Via")
@@
       (reference "IC1") (unit 1) (value "eTQFP48_9x9_TRI") (footprint "Libraries:TMC6200-TA")
     )
-    (path "/00000000-0000-0000-0000-00005ba8c4e4/00000000-0000-0000-0000-000061c4dafd"
-      (reference "J1") (unit 1) (value "Info") (footprint "Connector_JST:JST_PH_B3B-PH-K_1x03_P2.00mm_Vertical")
-    )
     (path "/00000000-0000-0000-0000-00005ba8c4e4/00000000-0000-0000-0000-000061c15679"
       (reference "J2") (unit 1) (value "VCC_IO") (footprint "Connector_JST:JST_PH_B2B-PH-K_1x02_P2.00mm_Vertical")
@@
       (reference "J4") (unit 1) (value "Fan") (footprint "Connector_JST:JST_PH_B2B-PH-K_1x02_P2.00mm_Vertical")
     )
-    (path "/00000000-0000-0000-0000-00005ba8c4e4/00000000-0000-0000-0000-000061c68d2f"
-      (reference "J6") (unit 1) (value "Current Sensing") (footprint "Connector_JST:JST_PH_B3B-PH-K_1x03_P2.00mm_Vertical")
-    )
     (path "/00000000-0000-0000-0000-00005d5fdd98/00000000-0000-0000-0000-000061cdf1c7"
       (reference "Q1") (unit 1) (value "HYG025N06LS1C2") (footprint "Libraries:PDFN-8")
@@
     )
     (path "/3a8d36b7-ae2b-4099-920c-31906ad65e30/78722155-0322-4653-b298-06aa3dc96ced"
-      (reference "U1") (unit 1) (value "RP2040") (footprint "IC57_RP2040")
+      (reference "U1") (unit 1) (value "RP2040") (footprint "Libraries:RP2040")
     )
     (path "/00000000-0000-0000-0000-00005ba8c4e4/00000000-0000-0000-0000-000061bff192"

Commit message: update for can
Other:
- added sheet CAN (can.kicad_sch)

Commit message: update for can
Other:
- sheet mcu renamed MCU
- sheet MCU ports: added TEMP_PCB; removed TEMP
